File: Toyota Satoshi Emblem/Toyota Satoshi Emblem.kicad_sch (KiCad schematic)
At the start: 293 parts

Commit message: v1.1
Parts:
- removed D? (x58): W_LED, symbol Device:LED
- removed J?: Conn_01x20_Male, symbol Connector:Conn_01x20_Male
- removed Q? (x6): BC337, Package_TO_SOT_THT:TO-92_Inline, symbol Transistor_BJT:BC337
- removed Q? (x12): BC327, Package_TO_SOT_THT:TO-92_Inline, symbol Transistor_BJT:BC327
- removed R? (x29): 10Ω, symbol Device:R
- removed R? (x12): 10KΩ, symbol Device:R
- removed R? (x12): 200Ω, symbol Device:R
- added D? (x86): A_LED, symbol Device:LED
- added Q? (x6): BC327, Package_TO_SOT_THT:TO-92_Inline, symbol Transistor_BJT:BC327
- added Q? (x12): S8550, Package_TO_SOT_THT:TO-92_Inline, symbol Transistor_BJT:S8550
- added R? (x86): 9Ω, symbol Device:R
- added R? (x12): 200Ω, symbol Device:R
- added R? (x12): 10KΩ, symbol Device:R
- added U? (x7): 74HC04, symbol 74xx:74HC04
- R?: value 200Ω -> 7.5k
Connections:
- net +5V: now also R?.2, R?.2, R?.2, R?.2, R?.2, R?.2, R?.2, R?.2, R?.2, R?.2, R?.2, R?.2
- net BUCK_A: now also Q?.3 (E), Q?.3 (E), Q?.3 (E)
- net BUCK_B: now also Q?.3 (E), Q?.3 (E), Q?.3 (E)
- net GND: now also D?.1 (K), D?.1 (K), D?.1 (K), D?.1 (K), D?.1 (K), D?.1 (K), D?.1 (K), D?.1 (K), D?.1 (K), D?.1 (K), D?.1 (K), D?.1 (K), D?.1 (K), D?.1 (K), D?.1 (K), D?.1 (K), D?.1 (K), D?.1 (K), D?.1 (K), D?.1 (K), D?.1 (K), D?.1 (K), D?.1 (K), D?.1 (K), D?.1 (K), D?.1 (K), D?.1 (K), D?.1 (K), D?.1 (K), D?.1 (K), D?.1 (K), D?.1 (K), D?.1 (K), D?.1 (K), D?.1 (K), D?.1 (K), D?.1 (K), D?.1 (K), D?.1 (K), D?.1 (K), D?.1 (K), D?.1 (K), D?.1 (K), D?.1 (K), D?.1 (K), D?.1 (K), D?.1 (K), D?.1 (K), D?.1 (K), D?.1 (K), D?.1 (K), D?.1 (K), D?.1 (K), D?.1 (K), D?.1 (K), D?.1 (K), D?.1 (K), D?.1 (K), D?.1 (K), D?.1 (K), D?.1 (K), D?.1 (K), D?.1 (K), D?.1 (K), D?.1 (K), D?.1 (K), D?.1 (K), D?.1 (K), D?.1 (K), D?.1 (K), D?.1 (K), D?.1 (K), R?.1, R?.1, R?.1, R?.1, R?.1, R?.1; no longer R?.2, R?.2, R?.2, R?.2, R?.2, R?.2
- net at R?.1, R?.1, R?.1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: now also Q?.3 (C)
- net at R?.2: now also U?.4
- net at R?.1, R?.1, R?.1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: now also Q?.3 (C) (x2)
- net at R?.1, R?.1: now also Q?.2 (B) (x6)
- net at R?.1, R?.1, R?.1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: now also Q?.3 (C), R?.1
- net at R?.1, R?.1, R?.1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: now also Q?.3 (C), R?.1, R?.1 (x2)
- net at R?.2: now also U?.6
- net at R?.2: now also U?.8
- net at R?.2: now also U?.2
- net at R?.2: now also U?.12
- net at R?.2: now also U?.10
- new net: D?.1 (K), D?.2 (A) (x43)
- new net: D?.2 (A), R?.2 (x43)
- new net: R?.2, U?.3
- new net: R?.1, R?.2 (x43)
- new net: Q?.2 (B), R?.2, R?.2 (x6)
- new net: Q?.1 (E), Q?.1 (E) (x6)
- new net: Q?.2 (B), R?.1, R?.1 (x6)
- new net: Q?.3 (C), R?.1, R?.1, R?.1, R?.1, R?.1, R?.1 (x5)
- new net: R?.2, U?.9
- new net: R?.2, U?.1
- new net: R?.2, U?.11
- new net: R?.2, U?.5
- new net: Q?.3 (C), R?.1, R?.1, R?.1, R?.1
- new net: R?.2, U?.13
Other:
- note removed: "WHITE"
- note removed: "WHITE TOGGLE"
- moved on the sheet: D?, R?

Commit message: v1.2
Parts:
- removed Q? (x6): BC327, Package_TO_SOT_THT:TO-92_Inline, symbol Transistor_BJT:BC327
- removed Q? (x12): S8550, Package_TO_SOT_THT:TO-92_Inline, symbol Transistor_BJT:S8550
- removed R? (x17): 200Ω, symbol Device:R
- removed R? (x36): 9Ω, symbol Device:R
- removed R? (x18): 10KΩ, symbol Device:R
- removed R?: 7.5k, symbol Device:R
- removed U? (x7): 74HC04, symbol 74xx:74HC04
- added Q? (x6): 2N3904, Package_TO_SOT_THT:TO-92_Inline, symbol Transistor_BJT:2N3904
- added Q? (x18): IRLZ44N, Package_TO_SOT_THT:TO-220-3_Vertical, symbol Transistor_FET:IRLZ44N
- added R? (x12): 10K, symbol Device:R
- added R? (x6): 200, symbol Device:R
Connections:
- net at R?.1, R?.1, R?.1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: now also R?.1, R?.1, Q?.2 (D) (x2)
- net at R?.2: now also D?.2 (A) (x26)
- net at D?.2 (A): now also R?.2 (x10)
- net at R?.1, R?.1, R?.1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: now also Q?.2 (D) (x10)
- new net: Q?.1 (G), Q?.3 (C), R?.1 (x6)
- new net: R?.2, R?.2 (x3)
- new net: Q?.1 (E), Q?.3 (S), R?.2 (x6)
- new net: Q?.2 (B), R?.1 (x6)
- new net: Q?.2 (D), Q?.3 (S), Q?.3 (S) (x6)
- new net: Q?.1 (G), R?.1, R?.2 (x6)
Other:
- note removed: "AMBER TOGGLE"
- note removed: "LETTER INTENSITY"
- moved on the sheet: D?, R?

Commit message: v1.3
Parts:
- removed D? (x120): A_LED, symbol Device:LED
- removed J?: Conn_01x20_Female, symbol Connector:Conn_01x20_Female
- removed R? (x90): 9Ω, symbol Device:R
- added C?: 200uF, symbol Device:C_Polarized
- added C?: 100uF, symbol Device:C_Polarized
- added D? (x120): A_LED, symbol Device:LED
- added D?: 1N5822, Diode_THT:D_DO-201AD_P15.24mm_Horizontal, symbol Diode:1N5822
- added J? (x6): Conn_01x03_Male, symbol Connector:Conn_01x03_Male
- added J? (x6): Letter Terminal, symbol Connector:Conn_01x03_Female
- added L?: 68uH, symbol Device:L
- added R? (x2): R, symbol Device:R
- added R? (x90): 9Ω, symbol Device:R
- added U?: LM2596S-ADJ, Package_TO_SOT_SMD:TO-263-5_TabPin3, symbol Regulator_Switching:LM2596S-ADJ
Connections:
- net BUCK_A: now also R?.2, R?.2, J?.2 (Pin_2), J?.2 (Pin_2)
- net BUCK_B: now also R?.2, R?.2, J?.2 (Pin_2), J?.2 (Pin_2)
- net GND: now also Q?.1 (E), Q?.1 (E), Q?.1 (E), Q?.1 (E), Q?.1 (E), Q?.1 (E), Q?.3 (S), Q?.3 (S), Q?.3 (S), Q?.3 (S), Q?.3 (S), Q?.3 (S), R?.2, R?.2, R?.2, R?.2, R?.2, R?.2, C?.2, C?.2, D?.2 (A), R?.1, U?.3 (GND); no longer A?.4 (GND), D?.1 (K), D?.1 (K), D?.1 (K), D?.1 (K), D?.1 (K), D?.1 (K), D?.1 (K), D?.1 (K), D?.1 (K), D?.1 (K), D?.1 (K), D?.1 (K)
- net VDD: now also C?.1, U?.1 (VIN)
- net at Q?.2 (D): now also J?.1 (Pin_1) (x5)
- net BUCK_C: now reaches R?.2, R?.2
- net BUCK_C: now also C?.1, J?.2 (Pin_2), J?.2 (Pin_2), L?.2, R?.1
- net at Q?.1 (G): now also A?.13 (D10)
- net at Q?.1 (G), R?.1, R?.2: now also A?.11 (D8)
- net at R?.1, R?.1, R?.1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: now also R?.1, R?.1, R?.1, R?.1, R?.1, R?.1, J?.2 (Pin_2); no longer Q?.2 (D)
- net at Q?.1 (G), R?.1, R?.2: now also A?.5 (D2)
- net at Q?.2 (D): now also J?.3 (Pin_3) (x5)
- net at Q?.1 (G): now also A?.6 (D3)
- net at A?.15 (D12): now also Q?.1 (G), R?.1, R?.2
- net at A?.16 (D13): now also Q?.1 (G), R?.1, R?.2
- net at A?.8 (D5): now also Q?.1 (G)
- net at A?.9 (D6): now also Q?.1 (G)
- net at A?.12 (D9): now also Q?.1 (G)
- net at A?.14 (D11): now also Q?.1 (G)
- net at A?.7 (D4): now also Q?.1 (G), R?.1, R?.2
- net at A?.10 (D7): now also Q?.1 (G), R?.1, R?.2
- new net: D?.1 (K), D?.2 (A) (x60)
- new net: D?.2 (A), R?.2 (x60)
- new net: D?.1 (K), D?.1 (K), D?.1 (K), D?.1 (K), D?.1 (K), D?.1 (K), J?.1 (Pin_1) (x6)
- new net: J?.2 (Pin_2), R?.1, R?.1, R?.1, R?.1, R?.1, R?.1, R?.1, R?.1, R?.1, R?.1, R?.1, R?.1 (x5)
- new net: D?.1 (K), D?.1 (K), D?.1 (K), D?.1 (K), D?.1 (K), D?.1 (K), J?.3 (Pin_3) (x6)
- new net: R?.2, R?.2, U?.4 (FB)
- new net: R?.1, R?.2 (x30)
- new net: J?.1 (Pin_1), Q?.2 (D)
- new net: J?.3 (Pin_3), Q?.2 (D)
- new net: D?.1 (K), L?.1, U?.2 (OUT)
Other:
- note removed: "AMBER"
- moved on the sheet: 5A, 6A10, A?, C?, D?, L?, Q?, R?, U?

Commit message: v1.4
Parts:
- removed Q?: BC327, Package_TO_SOT_THT:TO-92_Inline, symbol Transistor_BJT:BC327
- removed R? (x60): 9Ω, symbol Device:R
- added C?: 0.22u, symbol Device:C
- added D? (x4): 1N47xxA, Diode_THT:D_DO-41_SOD81_P10.16mm_Horizontal, symbol Diode:1N47xxA
- added J?: Power Port Terminal, symbol Connector_Generic:Conn_02x04_Counter_Clockwise
- added J? (x2): Serial Terminal, symbol Connector:Conn_01x02_Male
- added J?: Ambient Harness, symbol Connector:Conn_01x02_Female
- added K?: FINDER-40.51, Relay_THT:Relay_SPDT_Finder_40.51, symbol Relay:FINDER-40.51
- added Q?: BC337, Package_TO_SOT_THT:TO-92_Inline, symbol Transistor_BJT:BC337
- added R? (x60): 8.2, symbol Device:R
- added R? (x7): 10K, symbol Device:R
- added R?: R_Photo, symbol Device:R_Photo
- added R? (x4): 1K, symbol Device:R
- C?: value C_Polarized -> 10u
- C?: value C_Polarized -> 4.7u
- C?: value C -> 0.1u
- D?: value 5KPxxA -> 5KP16A
- F?: renamed from 5A; value Fuse -> 7.5A
- L? (x3): value 68uH -> 47uH
- R? (x12): value 9Ω -> 8.2
- R? (x36): value 9Ω -> 3.3
- R?: value R -> 1K
- R? (x6): value 200 -> 1K
- R? (x2): value R -> 3.3K
- R?: value R -> 4.7K
- R? (x2): value R -> 1.5K
- R?: value R -> 10K
Connections:
- net +5VD is gone; now on net +5V: C?.1, C?.1, U?.3 (OUT)
- net VDD is gone; now on net +12V: C?.1, C?.1, C?.1, U?.1 (VIN), U?.1 (VIN), U?.1 (VIN)
- net BUCK_A: now also J?.1 (Pin_1), R?.2, R?.2
- net BUCK_B: now also J?.2 (Pin_2), R?.2, R?.2
- net BUCK_C: now also J?.8 (Pin_8), R?.2, R?.2
- net GND: now also A?.29 (GND), C?.2, D?.2 (A), D?.2 (A), D?.2 (A), D?.2 (A), J?.1 (Pin_1), J?.4 (Pin_4), J?.5 (Pin_5), K?.A1
- net at D?.2 (A): now also R?.2 (x30)
- net at J?.2 (Pin_2), R?.1, R?.1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: now also R?.1, R?.1, R?.1, R?.1, R?.1, R?.1 (x5)
- net at A?.13 (D10), Q?.1 (G): now also R?.1
- net at 6A10.1 (K), C?.1, D?.1 (A1)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: now also C?.1, Q?.1 (C)
- net at A?.6 (D3), Q?.1 (G): now also R?.1
- net at F?.1: now also 6A10.2 (A)
- net at F?.2: now also K?.14; no longer 6A10.2 (A)
- net at A?.12 (D9), Q?.1 (G): now also R?.1
- net at R?.2: now also Q?.2 (B)
- net at D?.2 (A): now also Q?.3 (E)
- net at A?.9 (D6), Q?.1 (G): now also R?.1
- net at A?.1 (D1/TX): now also J?.2 (Pin_2)
- net at A?.14 (D11), Q?.1 (G): now also R?.1
- net at A?.2 (D0/RX): now also D?.1 (K), R?.1
- net at A?.23 (A4): now also D?.1 (K), R?.2
- net at A?.24 (A5): now also D?.1 (K), R?.2
- net at A?.25 (A6): now also D?.1 (K), R?.2
- net at A?.26 (A7): now also J?.2 (Pin_2), R?.2
- net +5V: now reaches A?.27 (+5V)
- net +5V: now also J?.7 (Pin_7), R?.1
- net at A?.8 (D5), Q?.1 (G): now also R?.1
- net VD renamed +12V
- net +12V: now also J?.3 (Pin_3), J?.6 (Pin_6)
- new net: R?.1, R?.2 (x30)
- new net: J?.1 (Pin_1), R?.1
- new net: J?.2 (Pin_2), R?.2
- new net: J?.1 (Pin_1), R?.2
- new net BAT +12V: K?.11
- new net HEAD RLY (R-B): K?.A2
- new net L Turn Sig: R?.1
- new net R Turn Sig: R?.1
Other:
- note added: "VEHICLE POWER ----->"
- moved on the sheet: 6A10, A?, C?, D?, F?, J?, L?, Q?, R?, U?

Commit message: v1.5
Parts:
- removed C? (x3): 200uF, symbol Device:C_Polarized
- removed C? (x3): 100uF, symbol Device:C_Polarized
- removed D?: 1N47xxA, Diode_THT:D_DO-41_SOD81_P10.16mm_Horizontal, symbol Diode:1N47xxA
- removed D? (x3): 1N5822, Diode_THT:D_DO-201AD_P15.24mm_Horizontal, symbol Diode:1N5822
- removed L? (x3): 47uH, symbol Device:L
- removed R? (x4): R, symbol Device:R
- removed R? (x2): 1K, symbol Device:R
- removed R?: 4.7K, symbol Device:R
- removed U? (x3): LM2596S-ADJ, Package_TO_SOT_SMD:TO-263-5_TabPin3, symbol Regulator_Switching:LM2596S-ADJ
- added C? (x4): 200uF, symbol Device:C_Polarized
- added C? (x4): 100uF, symbol Device:C_Polarized
- added D? (x48): A_LED, symbol Device:LED
- added D? (x4): 1N5822, Diode_THT:D_DO-201AD_P15.24mm_Horizontal, symbol Diode:1N5822
- added J?: Conn_01x09_Male, symbol Connector:Conn_01x09_Male
- added J?: Conn_01x09_Female, symbol Connector:Conn_01x09_Female
- added L? (x4): 47uH, symbol Device:L
- added Q?: 2N3904, Package_TO_SOT_THT:TO-92_Inline, symbol Transistor_BJT:2N3904
- added Q? (x10): IRLZ44N, Package_TO_SOT_THT:TO-220-3_Vertical, symbol Transistor_FET:IRLZ44N
- added R? (x24): 8.2, symbol Device:R
- added R? (x12): 3.3, symbol Device:R
- added R?: 10K, symbol Device:R
- added R? (x5): 1K, symbol Device:R
- added R?: R, symbol Device:R
- added R? (x4): 4.7K, symbol Device:R
- added U? (x4): LM2596S-ADJ, Package_TO_SOT_SMD:TO-263-5_TabPin3, symbol Regulator_Switching:LM2596S-ADJ
Connections:
- net +12V: now also C?.1, C?.1, C?.1, C?.1, U?.1 (VIN), U?.1 (VIN), U?.1 (VIN), U?.1 (VIN)
- net BUCK_A: now also C?.1, C?.1, C?.1, C?.1, L?.2, L?.2, L?.2, L?.2, R?.2, R?.2, R?.2, R?.2
- net GND: now also A?.4 (GND), J?.2 (Pin_2), C?.2, C?.2, C?.2, C?.2, C?.2, C?.2, C?.2, C?.2, D?.2 (A), D?.2 (A), D?.2 (A), D?.2 (A), Q?.1 (E), Q?.2 (D), Q?.2 (D), R?.1, R?.1, R?.1, R?.1, R?.1, U?.3 (GND), U?.3 (GND), U?.3 (GND), U?.3 (GND), U?.5 (~{ON}/OFF), U?.5 (~{ON}/OFF), U?.5 (~{ON}/OFF), U?.5 (~{ON}/OFF); no longer A?.29 (GND), J?.1 (Pin_1)
- net at A?.23 (A4): now also Q?.1 (G), R?.1, R?.2
- net at A?.26 (A7), R?.2: now also J?.1 (Pin_1); no longer J?.2 (Pin_2)
- net at A?.19 (A0): now also Q?.1 (G), Q?.1 (G)
- net at A?.20 (A1): now also Q?.1 (G), Q?.1 (G)
- net at A?.21 (A2): now also Q?.1 (G), Q?.1 (G)
- net at A?.22 (A3): now also Q?.1 (G), Q?.1 (G)
- new net: R?.1, R?.2 (x12)
- new net: D?.2 (A), R?.2 (x24)
- new net: D?.1 (K), L?.1, U?.2 (OUT) (x4)
- new net: R?.1, R?.2, U?.4 (FB) (x4)
- new net: D?.1 (K), D?.1 (K), D?.1 (K), J?.1 (Pin_1)
- new net: D?.1 (K), D?.2 (A) (x24)
- new net: J?.5 (Pin_5), R?.1, R?.1, R?.1, R?.1, R?.1, R?.1, R?.1, R?.1, R?.1, R?.1, R?.1, R?.1, R?.1, R?.1, R?.1, R?.1, R?.1, R?.1, R?.1, R?.1, R?.1, R?.1, R?.1, R?.1
- new net: D?.1 (K), D?.1 (K), D?.1 (K), J?.2 (Pin_2)
- new net: D?.1 (K), D?.1 (K), D?.1 (K), J?.3 (Pin_3)
- new net: D?.1 (K), D?.1 (K), D?.1 (K), J?.4 (Pin_4)
- new net: D?.1 (K), D?.1 (K), D?.1 (K), J?.6 (Pin_6)
- new net: D?.1 (K), D?.1 (K), D?.1 (K), J?.7 (Pin_7)
- new net: D?.1 (K), D?.1 (K), D?.1 (K), J?.8 (Pin_8)
- new net: D?.1 (K), D?.1 (K), D?.1 (K), J?.9 (Pin_9)
- new net: Q?.1 (G), Q?.3 (C), R?.2
- new net: Q?.2 (B), R?.2
- new net: Q?.2 (D), Q?.2 (D), Q?.2 (D), Q?.2 (D), Q?.3 (S) (x2)
- new net: J?.7 (Pin_7), Q?.3 (S)
- new net: J?.1 (Pin_1), Q?.3 (S)
- new net: J?.3 (Pin_3), Q?.3 (S)
- new net: J?.8 (Pin_8), Q?.3 (S)
- new net: J?.4 (Pin_4), Q?.3 (S)
- new net: J?.2 (Pin_2), Q?.3 (S)
- new net: J?.9 (Pin_9), Q?.3 (S)
- new net: J?.6 (Pin_6), Q?.3 (S)
- new net BUCK_D: J?.5 (Pin_5), R?.1
Other:
- moved on the sheet: 6A10, C?, D?, F?, J?, K?, Q?, R?, U?

Commit message: v1.6
Parts:
- added R157, R158, R161, R162: 10K, symbol Device:R
- A1: renamed from A?; footprint Module:Arduino_Nano -> (none)
- D1, D10, D100, D101, D102, D103, D104, D105, D106, D107, D108, D11, D12, D121, D122, D123, D124, D125, D126, D127, D128, D129, D130, D131, D132, D145, D146, D147, D148, D149, D150, D151, D152, D153, D154, D155, D156, D157, D158, D159, D160, D161, D162, D163, D164, D165, D166, D167, D168, D2, D25, D26, D27, D28, D29, D3, D30, D31, D32, D33, D34, D35, D36, D4, D49, D5, D50, D51, D52, D53, D54, D55, D56, D57, D58, D59, D6, D60, D7, D73, D74, D75, D76, D77, D78, D79, D8, D80, D81, D82, D83, D84, D9, D97, D98, D99: renamed from D?; value A_LED -> W_LED; footprint (none) -> afootprints:5730 LED W
- D109, D110, D111, D112, D113, D114, D115, D116, D117, D118, D119, D120, D13, D133, D134, D135, D136, D137, D138, D139, D14, D140, D141, D142, D143, D144, D15, D16, D169, D17, D170, D171, D172, D173, D174, D175, D176, D177, D178, D179, D18, D180, D181, D182, D183, D184, D185, D186, D187, D188, D189, D19, D190, D191, D192, D20, D21, D22, D23, D24, D37, D38, D39, D40, D41, D42, D43, D44, D45, D46, D47, D48, D61, D62, D63, D64, D65, D66, D67, D68, D69, D70, D71, D72, D85, D86, D87, D88, D89, D90, D91, D92, D93, D94, D95, D96: renamed from D?; footprint (none) -> afootprints:5730 LED A
- D193: renamed from D?; footprint Diode_THT:D_P600_R-6_P20.00mm_Horizontal -> (none)
- D194, D195, D196, D197, D200, D201, D204: renamed from D?; footprint Diode_THT:D_DO-41_SOD81_P10.16mm_Horizontal -> (none)
- D198, D199, D202, D203: renamed from D?; footprint Diode_THT:D_DO-201AD_P15.24mm_Horizontal -> (none)
- K1: renamed from K?; footprint Relay_THT:Relay_SPDT_Finder_40.51 -> (none)
- Q1, Q10, Q2, Q21, Q22, Q23, Q24, Q25, Q26: renamed from Q?; footprint Package_TO_SOT_THT:TO-92_Inline -> (none)
- Q11, Q12, Q13, Q14, Q15, Q16, Q17, Q18, Q19, Q20, Q27, Q28, Q29, Q3, Q30, Q31, Q32, Q33, Q34, Q35, Q36, Q37, Q38, Q4, Q5, Q6, Q7, Q8, Q9: renamed from Q?; footprint Package_TO_SOT_THT:TO-220-3_Vertical -> (none)
- R1, R10, R100, R101, R102, R103, R104, R105, R106, R107, R108, R109, R11, R110, R111, R112, R113, R114, R115, R116, R117, R118, R119, R12, R120, R121, R122, R123, R124, R125, R126, R127, R128, R129, R13, R130, R131, R132, R133, R134, R135, R136, R137, R138, R139, R14, R140, R141, R142, R143, R144, R15, R16, R17, R18, R19, R2, R20, R21, R22, R23, R24, R25, R26, R27, R28, R29, R3, R30, R31, R32, R33, R34, R35, R36, R37, R38, R39, R4, R40, R41, R42, R43, R44, R45, R46, R47, R48, R49, R5, R50, R51, R52, R53, R54, R55, R56, R57, R58, R59, R6, R60, R61, R62, R63, R64, R65, R66, R67, R68, R69, R7, R70, R71, R72, R73, R74, R75, R76, R77, R78, R79, R8, R80, R81, R82, R83, R84, R85, R86, R87, R88, R89, R9, R90, R91, R92, R93, R94, R95, R96, R97, R98, R99: renamed from R?; footprint (none) -> afootprints:1206 R
- U1, U2, U4, U5: renamed from U?; footprint Package_TO_SOT_SMD:TO-263-5_TabPin3 -> (none)
- gave numbers to parts that had none: 81
- renumbered 6A10 to 6A1
Connections:
- net BUCK_D: now also R157.1, R158.1, R161.1, R162.1
- net at A1.20 (A1), Q13.1 (G), Q7.1 (G): now also R157.2
- net at A1.19 (A0), Q14.1 (G), Q8.1 (G): now also R161.2
- net at A1.21 (A2), Q11.1 (G), Q5.1 (G): now also R162.2
- net at A1.22 (A3), Q4.1 (G), Q9.1 (G): now also R158.2
Other:
- moved on the sheet: J10, R168
