File: Toyota Satoshi Emblem/Toyota Satoshi Emblem.kicad_sch (KiCad schematic)
At the start: 263 parts, among them J1 Conn_01x03_Male, J10 Ambient Harness, J11 Letter Terminal, J12 Letter Terminal, J13 Letter Terminal, J14 Letter Terminal, J15 Letter Terminal, J16 Letter Terminal, J17 Serial Terminal, J18 Power Port Terminal, J7 Conn_01x09_Male, J8 Conn_01x09_Female, J9 Serial Terminal, K1 FINDER-40.51, Q1 BC327, Q10 2N3904, Q11 IRLZ44N, Q12 IRLZ44N, Q13 IRLZ44N, Q14 IRLZ44N, Q15 IRLZ44N, Q16 IRLZ44N, Q17 IRLZ44N, Q18 IRLZ44N, Q19 IRLZ44N, Q2 BC337, Q20 IRLZ44N, Q21 2N3904, Q22 2N3904, Q23 2N3904, Q24 2N3904, Q25 2N3904, Q26 2N3904, Q27 IRLZ44N, Q28 IRLZ44N, Q29 IRLZ44N, Q3 IRF4905, Q30 IRLZ44N, Q31 IRLZ44N, Q32 IRLZ44N, Q33 IRLZ44N, Q34 IRLZ44N, Q35 IRLZ44N, Q36 IRLZ44N, Q37 IRLZ44N, Q38 IRLZ44N, Q4 IRLZ44N, Q5 IRLZ44N, Q6 IRLZ44N, Q7 IRLZ44N, Q8 IRLZ44N, Q9 IRLZ44N, U1 LM2596S-ADJ, U2 LM2596S-ADJ, U3 L7805, U4 LM2596S-ADJ, U5 LM2596S-ADJ

Commit message: v1.9
Letter O and A are now complete
Parts:
- added D31, D32, D33, D34, D35, D36, D37, D38, D39, D40, D41, D42, D61, D62, D63, D64, D65, D66, D67, D68, D69, D70, D71, D72: WLED, afootprints:5730 LED W, symbol Device:LED
- added D43, D44, D45, D46, D47, D48, D49, D50, D51, D52, D53, D54, D55, D56, D57, D58, D59, D60, D73, D74, D75, D76, D77, D78, D79, D80, D81, D82, D83, D84, D85, D86, D87, D88, D89, D90: ALED, afootprints:5730 LED A, symbol Device:LED
- added J2, J3: Conn_01x03_Male, symbol Connector:Conn_01x03_Male
- added R13, R14, R16, R17, R18, R19, R20, R21, R22, R23, R24, R25, R26, R28, R29, R30, R31, R32, R33, R34, R35, R36: 4.7, afootprints:1206 R, symbol Device:R
- added R15, R27: 4,7, afootprints:1206 R, symbol Device:R
- renumbered C3 to C1, C2 to C10, C5 to C11, C6 to C12, C9 to C2, C7 to C3, C11 to C4, C4 to C5, C10 to C6, C8 to C7, C12 to C8, C1 to C9, D202 to D100, D39 to D101, D40 to D102, D41 to D103, D42 to D104, D43 to D105, D44 to D106, D45 to D107, D46 to D108, D47 to D109, D48 to D110, D49 to D111, D50 to D112, D51 to D113, D52 to D114, D53 to D115, D54 to D116, D199 to D117, D203 to D118, D55 to D119, D56 to D120, D57 to D121, D58 to D122, D59 to D123, D60 to D124, D61 to D125, D62 to D126, D63 to D127, D64 to D128, D65 to D129, D66 to D130, D67 to D131, D68 to D132, D69 to D133, D70 to D134, D71 to D135, D72 to D136, D73 to D137, D74 to D138, D75 to D139, D76 to D140, D77 to D141, D78 to D142, D204 to D143, D196 to D144, D193 to D145, D197 to D146, D200 to D147, D201 to D148, D194 to D149, D195 to D150, D31 to D91, D32 to D92, D33 to D93, D34 to D94, D35 to D95, D36 to D96, D37 to D97, D38 to D98, D198 to D99, J18 to J11, J8 to J12, J17 to J13, J7 to J14, J9 to J15, J11 to J4, J12 to J5, J13 to J6, J14 to J7, J15 to J8, J16 to J9, L3 to L2, L2 to L3, Q15 to Q1, Q35 to Q10, Q29 to Q11, Q23 to Q12, Q18 to Q13, Q36 to Q14, Q30 to Q15, Q24 to Q16, Q19 to Q17, Q37 to Q18, Q31 to Q19, Q33 to Q2, Q25 to Q20, Q20 to Q21, Q38 to Q22, Q32 to Q23, Q26 to Q24, Q4 to Q25, Q5 to Q26, Q7 to Q27, Q8 to Q28, Q9 to Q29, Q27 to Q3, Q11 to Q30, Q13 to Q31, Q14 to Q32, Q6 to Q33, Q10 to Q34, Q12 to Q35, Q3 to Q36, Q1 to Q37, Q2 to Q38, Q21 to Q4, Q16 to Q5, Q34 to Q6, Q28 to Q7, Q22 to Q8, Q17 to Q9, R43 to R100, R44 to R101, R45 to R102, R46 to R103, R47 to R104, R48 to R105, R155 to R106, R169 to R107, R156 to R108, R150 to R109, R161 to R110, R157 to R111, R162 to R112, R158 to R113, R159 to R114, R160 to R115, R145 to R116, R146 to R117, R147 to R118, R148 to R119, R163 to R120, R149 to R121, R170 to R37, R176 to R38, R188 to R39, R182 to R40, R171 to R41, R177 to R42, R189 to R43, R183 to R44, R172 to R45, R178 to R46, R190 to R47, R184 to R48, R173 to R49, R179 to R50, R191 to R51, R185 to R52, R174 to R53, R180 to R54, R13 to R55, R14 to R56, R15 to R57, R153 to R58, R166 to R59, R192 to R60, R16 to R61, R17 to R62, R18 to R63, R186 to R64, R151 to R65, R164 to R66, R19 to R67, R20 to R68, R21 to R69, R22 to R70, R23 to R71, R24 to R72, R175 to R73, R181 to R74, R25 to R75, R26 to R76, R27 to R77, R154 to R78, R167 to R79, R193 to R80, R187 to R81, R28 to R82, R29 to R83, R30 to R84, R152 to R85, R165 to R86, R31 to R87, R32 to R88, R33 to R89, R34 to R90, R35 to R91, R36 to R92, R37 to R93, R38 to R94, R39 to R95, R168 to R96, R40 to R97, R41 to R98, R42 to R99, U4 to U2, U2 to U3, U5 to U4, U3 to U5
Connections:
- new net: D75.1 (K), D78.1 (K), D81.1 (K), D84.1 (K), D87.1 (K), D90.1 (K), J3.3 (Pin_3)
- new net: D77.1 (K), D78.2 (A)
- new net: D45.1 (K), D48.1 (K), D51.1 (K), D54.1 (K), D57.1 (K), D60.1 (K), J2.3 (Pin_3)
- new net: D50.1 (K), D51.2 (A)
- new net: D31.2 (A), D32.1 (K)
- new net: D32.2 (A), R13.2
- new net: D56.1 (K), D57.2 (A)
- new net: D33.2 (A), D34.1 (K)
- new net: D34.2 (A), R14.2
- new net: J2.2 (Pin_2), R13.1, R14.1, R15.1, R16.1, R17.1, R18.1, R19.1, R20.1, R21.1, R22.1, R23.1, R24.1
- new net: D43.2 (A), R19.2
- new net: D61.2 (A), D62.1 (K)
- new net: D62.2 (A), R25.2
- new net: J3.2 (Pin_2), R25.1, R26.1, R27.1, R28.1, R29.1, R30.1, R31.1, R32.1, R33.1, R34.1, R35.1, R36.1
- new net: D68.2 (A), R28.2
- new net: D31.1 (K), D33.1 (K), D35.1 (K), D37.1 (K), D39.1 (K), D41.1 (K), J2.1 (Pin_1)
- new net: D37.2 (A), D38.1 (K)
- new net: D52.2 (A), R22.2
- new net: D49.1 (K), D50.2 (A)
- new net: D49.2 (A), R21.2
- new net: D41.2 (A), D42.1 (K)
- new net: D42.2 (A), R18.2
- new net: D88.2 (A), R36.2
- new net: D74.1 (K), D75.2 (A)
- new net: D73.1 (K), D74.2 (A)
- new net: D55.1 (K), D56.2 (A)
- new net: D55.2 (A), R23.2
- new net: D61.1 (K), D63.1 (K), D65.1 (K), D67.1 (K), D69.1 (K), D71.1 (K), J3.1 (Pin_1)
- new net: D63.2 (A), D64.1 (K)
- new net: D64.2 (A), R26.2
- new net: D80.1 (K), D81.2 (A)
- new net: D86.1 (K), D87.2 (A)
- new net: D46.1 (K), D47.2 (A)
- new net: D46.2 (A), R20.2
- new net: D70.2 (A), R29.2
- new net: D82.2 (A), R34.2
- new net: D79.1 (K), D80.2 (A)
- new net: D79.2 (A), R33.2
- new net: D69.2 (A), D70.1 (K)
- new net: D73.2 (A), R31.2
- new net: D47.1 (K), D48.2 (A)
- new net: D43.1 (K), D44.2 (A)
- new net: D59.1 (K), D60.2 (A)
- new net: D83.1 (K), D84.2 (A)
- new net: D82.1 (K), D83.2 (A)
- new net: D58.1 (K), D59.2 (A)
- new net: D71.2 (A), D72.1 (K)
- new net: D72.2 (A), R30.2
- new net: D44.1 (K), D45.2 (A)
- new net: D89.1 (K), D90.2 (A)
- new net: D88.1 (K), D89.2 (A)
- new net: D76.1 (K), D77.2 (A)
- new net: D76.2 (A), R32.2
- new net: D67.2 (A), D68.1 (K)
- new net: D38.2 (A), R16.2
- new net: D39.2 (A), D40.1 (K)
- new net: D40.2 (A), R17.2
- new net: D58.2 (A), R24.2
- new net: D85.1 (K), D86.2 (A)
- new net: D85.2 (A), R35.2
- new net: D65.2 (A), D66.1 (K)
- new net: D53.1 (K), D54.2 (A)
- new net: D52.1 (K), D53.2 (A)
- new net: D66.2 (A), R27.2
- new net: D35.2 (A), D36.1 (K)
- new net: D36.2 (A), R15.2

Commit message: v1.10
Second letter O added
Parts:
- added D100, D101, D102, D121, D122, D123, D124, D125, D126, D127, D128, D129, D130, D131, D132, D91, D92, D93, D94, D95, D96, D97, D98, D99: WLED, afootprints:5730 LED W, symbol Device:LED
- added D103, D104, D105, D106, D107, D108, D109, D110, D111, D112, D113, D114, D115, D116, D117, D118, D119, D120, D133, D134, D135, D136, D137, D138, D139, D140, D141, D142, D143, D144, D145, D146, D147, D148, D149, D150: ALED, afootprints:5730 LED A, symbol Device:LED
- added J8, J9: Conn_01x03_Male, symbol Connector:Conn_01x03_Male
- added R37, R38, R40, R41, R42, R43, R44, R45, R46, R47, R48, R49, R50, R52, R53, R54, R55, R56, R57, R58, R59, R60: 4.7, afootprints:1206 R, symbol Device:R
- added R39, R51: 4,7, afootprints:1206 R, symbol Device:R
- renumbered D91 to D151, D92 to D152, D93 to D153, D94 to D154, D95 to D155, D96 to D156, D97 to D157, D98 to D158, D99 to D159, D100 to D160, D101 to D161, D102 to D162, D103 to D163, D104 to D164, D105 to D165, D106 to D166, D107 to D167, D108 to D168, D109 to D169, D110 to D170, D111 to D171, D112 to D172, D113 to D173, D114 to D174, D115 to D175, D116 to D176, D117 to D177, D118 to D178, D119 to D179, D120 to D180, D121 to D181, D122 to D182, D123 to D183, D124 to D184, D125 to D185, D126 to D186, D127 to D187, D128 to D188, D129 to D189, D130 to D190, D131 to D191, D132 to D192, D133 to D193, D134 to D194, D135 to D195, D136 to D196, D137 to D197, D138 to D198, D139 to D199, D140 to D200, D141 to D201, D142 to D202, D143 to D203, D144 to D204, D145 to D205, D146 to D206, D147 to D207, D148 to D208, D149 to D209, D150 to D210, J8 to J10, J9 to J11, J10 to J12, J11 to J13, J12 to J14, J13 to J15, J14 to J16, J15 to J17, R76 to R100, R77 to R101, R78 to R102, R79 to R103, R80 to R104, R81 to R105, R82 to R106, R83 to R107, R84 to R108, R85 to R109, R86 to R110, R87 to R111, R88 to R112, R89 to R113, R90 to R114, R91 to R115, R92 to R116, R93 to R117, R94 to R118, R95 to R119, R96 to R120, R97 to R121, R98 to R122, R99 to R123, R100 to R124, R101 to R125, R102 to R126, R103 to R127, R104 to R128, R105 to R129, R106 to R130, R107 to R131, R108 to R132, R109 to R133, R110 to R134, R111 to R135, R112 to R136, R113 to R137, R114 to R138, R115 to R139, R116 to R140, R117 to R141, R118 to R142, R119 to R143, R120 to R144, R121 to R145, R37 to R61, R38 to R62, R39 to R63, R40 to R64, R41 to R65, R42 to R66, R43 to R67, R44 to R68, R45 to R69, R46 to R70, R47 to R71, R48 to R72, R49 to R73, R50 to R74, R51 to R75, R52 to R76, R53 to R77, R54 to R78, R55 to R79, R56 to R80, R57 to R81, R58 to R82, R59 to R83, R60 to R84, R61 to R85, R62 to R86, R63 to R87, R64 to R88, R65 to R89, R66 to R90, R67 to R91, R68 to R92, R69 to R93, R70 to R94, R71 to R95, R72 to R96, R73 to R97, R74 to R98, R75 to R99
Connections:
- new net: D135.1 (K), D138.1 (K), D141.1 (K), D144.1 (K), D147.1 (K), D150.1 (K), J9.3 (Pin_3)
- new net: D149.1 (K), D150.2 (A)
- new net: D105.1 (K), D108.1 (K), D111.1 (K), D114.1 (K), D117.1 (K), D120.1 (K), J8.3 (Pin_3)
- new net: D107.1 (K), D108.2 (A)
- new net: D123.2 (A), D124.1 (K)
- new net: D124.2 (A), R50.2
- new net: D91.2 (A), D92.1 (K)
- new net: D92.2 (A), R37.2
- new net: D145.1 (K), D146.2 (A)
- new net: D145.2 (A), R59.2
- new net: D115.1 (K), D116.2 (A)
- new net: D115.2 (A), R47.2
- new net: D121.1 (K), D123.1 (K), D125.1 (K), D127.1 (K), D129.1 (K), D131.1 (K), J9.1 (Pin_1)
- new net: D131.2 (A), D132.1 (K)
- new net: J8.2 (Pin_2), R37.1, R38.1, R39.1, R40.1, R41.1, R42.1, R43.1, R44.1, R45.1, R46.1, R47.1, R48.1
- new net: D112.2 (A), R46.2
- new net: D93.2 (A), D94.1 (K)
- new net: D94.2 (A), R38.2
- new net: D127.2 (A), D128.1 (K)
- new net: J9.2 (Pin_2), R49.1, R50.1, R51.1, R52.1, R53.1, R54.1, R55.1, R56.1, R57.1, R58.1, R59.1, R60.1
- new net: D132.2 (A), R54.2
- new net: D101.1 (K), D91.1 (K), D93.1 (K), D95.1 (K), D97.1 (K), D99.1 (K), J8.1 (Pin_1)
- new net: D101.2 (A), D102.1 (K)
- new net: D139.1 (K), D140.2 (A)
- new net: D139.2 (A), R57.2
- new net: D134.1 (K), D135.2 (A)
- new net: D125.2 (A), D126.1 (K)
- new net: D126.2 (A), R51.2
- new net: D137.1 (K), D138.2 (A)
- new net: D128.2 (A), R52.2
- new net: D121.2 (A), D122.1 (K)
- new net: D113.1 (K), D114.2 (A)
- new net: D122.2 (A), R49.2
- new net: D110.1 (K), D111.2 (A)
- new net: D109.1 (K), D110.2 (A)
- new net: D148.1 (K), D149.2 (A)
- new net: D146.1 (K), D147.2 (A)
- new net: D95.2 (A), D96.1 (K)
- new net: D96.2 (A), R39.2
- new net: D97.2 (A), D98.1 (K)
- new net: D104.1 (K), D105.2 (A)
- new net: D103.1 (K), D104.2 (A)
- new net: D143.1 (K), D144.2 (A)
- new net: D142.1 (K), D143.2 (A)
- new net: D103.2 (A), R43.2
- new net: D136.1 (K), D137.2 (A)
- new net: D136.2 (A), R56.2
- new net: D106.2 (A), R44.2
- new net: D98.2 (A), R40.2
- new net: D119.1 (K), D120.2 (A)
- new net: D102.2 (A), R42.2
- new net: D106.1 (K), D107.2 (A)
- new net: D112.1 (K), D113.2 (A)
- new net: D133.1 (K), D134.2 (A)
- new net: D133.2 (A), R55.2
- new net: D116.1 (K), D117.2 (A)
- new net: D118.1 (K), D119.2 (A)
- new net: D118.2 (A), R48.2
- new net: D109.2 (A), R45.2
- new net: D129.2 (A), D130.1 (K)
- new net: D130.2 (A), R53.2
- new net: D142.2 (A), R58.2
- new net: D100.1 (K), D99.2 (A)
- new net: D100.2 (A), R41.2
- new net: D148.2 (A), R60.2
- new net: D140.1 (K), D141.2 (A)

Commit message: v1.11
All letters and raptor lights are complete. LED board is nearing completion. Photosensor board is remaining.
Parts:
- removed J16: Conn_01x09_Male, symbol Connector:Conn_01x09_Male
- removed R101, R108, R113, R116, R119, R123, R126, R129, R81, R87, R93, R96: 8.2, symbol Device:R
- added D151, D152, D153, D154, D155, D156, D157, D158, D159, D160, D161, D162: WLED, afootprints:5730 LED W, symbol Device:LED
- added D163, D164, D165, D166, D167, D168, D169, D170, D171, D172, D173, D174, D175, D176, D177, D178, D179, D180, D187, D190, D193, D202, D205, D208: ALED, afootprints:5730 LED A, symbol Device:LED
- added D217, D220, D223, D232, D235, D238: ALED, symbol Device:LED
- added J10, J17, J19, J20, J21: Conn_01x03_Male, symbol Connector:Conn_01x03_Male
- added R61, R62, R64, R65, R66, R67, R68, R69, R70, R71, R72: 4.7, afootprints:1206 R, symbol Device:R
- added R63: 4,7, afootprints:1206 R, symbol Device:R
- D181: renamed from D151; value W_LED -> WLED; footprint (none) -> afootprints:5730 LED W
- D182: renamed from D152; value W_LED -> WLED; footprint (none) -> afootprints:5730 LED W
- D183: renamed from D155; value W_LED -> WLED; footprint (none) -> afootprints:5730 LED W
- D184: renamed from D156; value W_LED -> WLED; footprint (none) -> afootprints:5730 LED W
- D185: renamed from D161; value W_LED -> WLED; footprint (none) -> afootprints:5730 LED W
- D186: renamed from D162; value W_LED -> WLED; footprint (none) -> afootprints:5730 LED W
- D188: renamed from D153; value A_LED -> ALED; footprint (none) -> afootprints:5730 LED A
- D189: renamed from D154; value A_LED -> ALED; footprint (none) -> afootprints:5730 LED A
- D191: renamed from D157; value A_LED -> ALED; footprint (none) -> afootprints:5730 LED A
- D192: renamed from D158; value A_LED -> ALED; footprint (none) -> afootprints:5730 LED A
- D194: renamed from D163; value A_LED -> ALED; footprint (none) -> afootprints:5730 LED A
- D195: renamed from D164; value A_LED -> ALED; footprint (none) -> afootprints:5730 LED A
- D196: renamed from D165; value W_LED -> WLED; footprint (none) -> afootprints:5730 LED W
- D197: renamed from D166; value W_LED -> WLED; footprint (none) -> afootprints:5730 LED W
- D198: renamed from D169; value W_LED -> WLED; footprint (none) -> afootprints:5730 LED W
- D199: renamed from D170; value W_LED -> WLED; footprint (none) -> afootprints:5730 LED W
- D200: renamed from D173; value W_LED -> WLED; footprint (none) -> afootprints:5730 LED W
- D201: renamed from D174; value W_LED -> WLED; footprint (none) -> afootprints:5730 LED W
- D203: renamed from D167; value A_LED -> ALED; footprint (none) -> afootprints:5730 LED A
- D204: renamed from D168; value A_LED -> ALED; footprint (none) -> afootprints:5730 LED A
- D206: renamed from D171; value A_LED -> ALED; footprint (none) -> afootprints:5730 LED A
- D207: renamed from D172; value A_LED -> ALED; footprint (none) -> afootprints:5730 LED A
- D209: renamed from D175; value A_LED -> ALED; footprint (none) -> afootprints:5730 LED A
- D210: renamed from D176; value A_LED -> ALED; footprint (none) -> afootprints:5730 LED A
- D211: renamed from D179; value W_LED -> WLED
- D212: renamed from D180; value W_LED -> WLED
- D213: renamed from D183; value W_LED -> WLED
- D214: renamed from D184; value W_LED -> WLED
- D215: renamed from D187; value W_LED -> WLED
- D216: renamed from D188; value W_LED -> WLED
- D218: renamed from D181; value A_LED -> ALED
- D219: renamed from D182; value A_LED -> ALED
- D221: renamed from D185; value A_LED -> ALED
- D222: renamed from D186; value A_LED -> ALED
- D224: renamed from D189; value A_LED -> ALED
- D225: renamed from D190; value A_LED -> ALED
- D226: renamed from D191; value W_LED -> WLED
- D227: renamed from D192; value W_LED -> WLED
- D228: renamed from D195; value W_LED -> WLED
- D229: renamed from D196; value W_LED -> WLED
- D230: renamed from D199; value W_LED -> WLED
- D231: renamed from D200; value W_LED -> WLED
- D233: renamed from D193; value A_LED -> ALED
- D234: renamed from D194; value A_LED -> ALED
- D236: renamed from D197; value A_LED -> ALED
- D237: renamed from D198; value A_LED -> ALED
- D239: renamed from D201; value A_LED -> ALED
- D240: renamed from D202; value A_LED -> ALED
- R73: renamed from R79; value 3.3 -> 4.7; footprint (none) -> afootprints:1206 R
- R74: renamed from R85; value 3.3 -> 4.7; footprint (none) -> afootprints:1206 R
- R75: renamed from R91; value 3.3 -> 4.7; footprint (none) -> afootprints:1206 R
- R76: renamed from R80; value 8.2 -> 4.7; footprint (none) -> afootprints:1206 R
- R77: renamed from R86; value 8.2 -> 4.7; footprint (none) -> afootprints:1206 R
- R78: renamed from R92; value 8.2 -> 4.7; footprint (none) -> afootprints:1206 R
- R79: renamed from R94; value 3.3 -> 4.7; footprint (none) -> afootprints:1206 R
- R80: renamed from R99; value 3.3 -> 4.7; footprint (none) -> afootprints:1206 R
- R81: renamed from R106; value 3.3 -> 4.7; footprint (none) -> afootprints:1206 R
- R82: renamed from R95; value 8.2 -> 4.7; footprint (none) -> afootprints:1206 R
- R83: renamed from R100; value 8.2 -> 4.7; footprint (none) -> afootprints:1206 R
- R84: renamed from R107; value 8.2 -> 4.7; footprint (none) -> afootprints:1206 R
- R85: renamed from R111; value 3.3 -> 4.7
- R86: renamed from R114; value 3.3 -> 4.7
- R87: renamed from R117; value 3.3 -> 4.7
- R88: renamed from R112; value 8.2 -> 4.7
- R89: renamed from R115; value 8.2 -> 4.7
- R90: renamed from R118; value 8.2 -> 4.7
- R91: renamed from R121; value 3.3 -> 4.7
- R92: renamed from R124; value 3.3 -> 4.7
- R93: renamed from R127; value 3.3 -> 4.7
- R94: renamed from R122; value 8.2 -> 4.7
- R95: renamed from R125; value 8.2 -> 4.7
- R96: renamed from R128; value 8.2 -> 4.7
- renumbered D159 to D241, D160 to D242, D177 to D243, D178 to D244, D203 to D245, D204 to D246, D205 to D247, D206 to D248, D207 to D249, D208 to D250, D209 to D251, D210 to D252, J10 to J11, J11 to J12, J12 to J13, J13 to J14, J14 to J15, J15 to J16, J17 to J18, R64 to R100, R65 to R101, R66 to R102, R67 to R103, R68 to R104, R69 to R105, R70 to R106, R71 to R107, R72 to R108, R73 to R109, R74 to R110, R75 to R111, R76 to R112, R77 to R113, R78 to R114, R82 to R115, R83 to R116, R84 to R117, R88 to R118, R89 to R119, R90 to R120, R97 to R121, R98 to R122, R102 to R123, R103 to R124, R104 to R125, R105 to R126, R109 to R127, R110 to R128, R120 to R129, R61 to R97, R62 to R98, R63 to R99
Connections:
- net at R90.2: now also D223.2 (A)
- net at D224.2 (A): now also D223.1 (K)
- net at R84.2: now also D208.2 (A)
- net at D209.2 (A): now also D208.1 (K)
- net at D181.1 (K), D183.1 (K), D185.1 (K): now also J17.1 (Pin_1)
- net at R77.2: now also D190.2 (A)
- net at D196.1 (K), D198.1 (K), D200.1 (K): now also J19.1 (Pin_1)
- net at D211.1 (K), D213.1 (K), D215.1 (K): now also J20.1 (Pin_1)
- net at D226.1 (K), D228.1 (K), D230.1 (K): now also J21.1 (Pin_1)
- net at D234.1 (K), D237.1 (K), D240.1 (K): now also J21.3 (Pin_3)
- net at D219.1 (K), D222.1 (K), D225.1 (K): now also J20.3 (Pin_3)
- net at D204.1 (K), D207.1 (K), D210.1 (K): now also J19.3 (Pin_3)
- net at D189.1 (K), D192.1 (K), D195.1 (K): now also J17.3 (Pin_3)
- net at D221.2 (A): now also D220.1 (K)
- net at D236.2 (A): now also D235.1 (K)
- net at R83.2: now also D205.2 (A)
- net at R89.2: now also D220.2 (A)
- net at D188.2 (A): now also D187.1 (K)
- net at R76.2: now also D187.2 (A)
- net at D203.2 (A): now also D202.1 (K)
- net at D191.2 (A): now also D190.1 (K)
- net at R88.2: now also D217.2 (A)
- net at D218.2 (A): now also D217.1 (K)
- net at D206.2 (A): now also D205.1 (K)
- net at R78.2: now also D193.2 (A)
- net at D194.2 (A): now also D193.1 (K)
- net at R95.2: now also D235.2 (A)
- net at R82.2: now also D202.2 (A)
- net at R94.2: now also D232.2 (A)
- net at D233.2 (A): now also D232.1 (K)
- net at R96.2: now also D238.2 (A)
- net at D239.2 (A): now also D238.1 (K)
- new net: J21.2 (Pin_2), R91.1, R92.1, R93.1, R94.1, R95.1, R96.1
- new net: J17.2 (Pin_2), R73.1, R74.1, R75.1, R76.1, R77.1, R78.1
- new net: D151.1 (K), D153.1 (K), D155.1 (K), D157.1 (K), D159.1 (K), D161.1 (K), J10.1 (Pin_1)
- new net: J10.2 (Pin_2), R61.1, R62.1, R63.1, R64.1, R65.1, R66.1, R67.1, R68.1, R69.1, R70.1, R71.1, R72.1
- new net: D165.1 (K), D168.1 (K), D171.1 (K), D174.1 (K), D177.1 (K), D180.1 (K), J10.3 (Pin_3)
- new net: J20.2 (Pin_2), R85.1, R86.1, R87.1, R88.1, R89.1, R90.1
- new net: J19.2 (Pin_2), R79.1, R80.1, R81.1, R82.1, R83.1, R84.1
- new net: D179.1 (K), D180.2 (A)
- new net: D155.2 (A), D156.1 (K)
- new net: D156.2 (A), R63.2
- new net: D170.1 (K), D171.2 (A)
- new net: D169.1 (K), D170.2 (A)
- new net: D153.2 (A), D154.1 (K)
- new net: D154.2 (A), R62.2
- new net: D164.1 (K), D165.2 (A)
- new net: D167.1 (K), D168.2 (A)
- new net: D166.1 (K), D167.2 (A)
- new net: D169.2 (A), R69.2
- new net: D151.2 (A), D152.1 (K)
- new net: D152.2 (A), R61.2
- new net: D173.1 (K), D174.2 (A)
- new net: D172.1 (K), D173.2 (A)
- new net: D163.1 (K), D164.2 (A)
- new net: D166.2 (A), R68.2
- new net: D163.2 (A), R67.2
- new net: D159.2 (A), D160.1 (K)
- new net: D160.2 (A), R65.2
- new net: D161.2 (A), D162.1 (K)
- new net: D162.2 (A), R66.2
- new net: D157.2 (A), D158.1 (K)
- new net: D178.2 (A), R72.2
- new net: D175.2 (A), R71.2
- new net: D178.1 (K), D179.2 (A)
- new net: D176.1 (K), D177.2 (A)
- new net: D175.1 (K), D176.2 (A)
- new net: D172.2 (A), R70.2
- new net: D158.2 (A), R64.2

Commit message: v1.12
many changes
Parts:
- removed J13: Ambient Harness, symbol Connector:Conn_01x02_Female
- removed J15: Conn_01x09_Female, symbol Connector:Conn_01x09_Female
- removed J18: Serial Terminal, symbol Connector:Conn_01x02_Male
- removed Q1, Q10, Q11, Q13, Q14, Q15, Q17, Q18, Q19, Q2, Q21, Q22, Q23, Q25, Q26, Q27, Q28, Q29, Q3, Q30, Q31, Q33, Q35, Q5, Q6, Q7, Q9: IRLZ44N, symbol Transistor_FET:IRLZ44N
- removed R129: R_Photo, symbol Device:R_Photo
- removed R144: 10K, symbol Device:R
- added J15, J22, J23, J24: Raptor Term, symbol Connector:Conn_01x03_Female
- added Q1, Q10, Q11, Q13, Q14, Q15, Q17, Q18, Q19, Q2, Q21, Q22, Q23, Q25, Q26, Q27, Q28, Q29, Q3, Q30, Q31, Q33, Q35, Q5, Q6, Q7, Q9: IRLR7843, symbol asymbols:IRLR7843
- D211, D212, D213, D214, D215, D216, D226, D227, D228, D229, D230, D231: footprint (none) -> afootprints:5730 LED W
- D217, D218, D219, D220, D221, D222, D223, D224, D225, D232, D233, D234, D235, D236, D237, D238, D239, D240: footprint (none) -> afootprints:5730 LED A
- D249, D250: value 1N47xxA -> 1N4733A
- D251: value 1N47xxA -> 1N4746A
- D252: value 1N47xxA -> 1N4739A
- F1: value 7.5A -> 10A
- J17, J19, J20, J21: value Conn_01x03_Male -> S-Pads
- R133: value R -> 10K
Connections:
- net +12V: no longer J14.6 (Pin_6)
- net +5V: now also J14.6 (Pin_6), R134.1, R135.1, R136.1, R137.1; no longer J14.7 (Pin_7)
- net BUCK_A: no longer C4.1, C7.1, C8.1, L2.2, L3.2, L4.2, R116.2, R123.2, R124.2
- net BUCK_B: now also C7.1, L3.2, R123.2
- net BUCK_C: now also C4.1, L2.2, R116.2
- net BUCK_D: now also C8.1, J14.7 (Pin_7), L4.2, R124.2, J15.2 (Pin_2), J22.2 (Pin_2), J23.2 (Pin_2), J24.2 (Pin_2); no longer R134.1, R135.1, R136.1, R137.1
- net GND: now also Q11.3 (S), Q15.3 (S), Q19.3 (S), Q23.3 (S), Q3.3 (S), Q33.2 (D), Q35.2 (D), Q7.3 (S); no longer A1.4 (GND)
- net at Q20.3 (C), R113.1: now also Q17.1 (G)
- net at A1.20 (A1), R135.2: now also Q27.1 (G), Q31.1 (G)
- net at Q4.3 (C), R97.1: now also Q1.1 (G)
- net at D248.2 (A): now also Q37.1 (C); no longer Q37.3 (E)
- net at A1.13 (D10), R104.1: now also Q7.1 (G)
- net at Q12.3 (C), R105.1: now also Q9.1 (G)
- net at A1.11 (D8), R106.2, R107.1: now also Q10.1 (G)
- net at 6A1.1 (K), C10.1, C9.1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: now also Q37.3 (E); no longer Q37.1 (C)
- net at A1.5 (D2), R122.2, R125.1: now also Q22.1 (G)
- net at J12.3 (Pin_3): now also Q22.2 (D)
- net at A1.6 (D3), R126.1: now also Q23.1 (G)
- net at J11.1 (Pin_1): now also Q17.2 (D)
- net at Q24.3 (C), R121.1: now also Q21.1 (G)
- net at J12.1 (Pin_1): now also Q21.2 (D)
- net at Q34.3 (C), R130.2: now also Q35.1 (G)
- net at A1.14 (D11), R100.1: now also Q3.1 (G)
- net at J4.1 (Pin_1): now also Q1.2 (D)
- net at J4.3 (Pin_3): now also Q2.2 (D)
- net at A1.12 (D9), R108.1: now also Q11.1 (G)
- net at J5.1 (Pin_1): now also Q5.2 (D)
- net at J5.3 (Pin_3): now also Q6.2 (D)
- net at A1.23 (A4), R132.1, R133.2: now also Q33.1 (G)
- net at A1.15 (D12), R102.2, R103.1: now also Q6.1 (G)
- net at A1.10 (D7), R110.2, R111.1: now also Q14.1 (G)
- net at J7.3 (Pin_3): now also Q14.2 (D)
- net at A1.21 (A2), R136.2: now also Q26.1 (G), Q30.1 (G)
- net at A1.8 (D5), R118.1: now also Q19.1 (G)
- net at A1.19 (A0), Q32.1 (G), R134.2: now also Q28.1 (G)
- net at Q32.2 (D): now also Q29.2 (D), Q30.2 (D), Q31.2 (D), Q35.3 (S)
- net at A1.7 (D4), R114.2, R117.1: now also Q18.1 (G)
- net at J11.3 (Pin_3): now also Q18.2 (D)
- net at Q32.3 (S): now also J15.1 (Pin_1)
- net at A1.16 (D13), R98.2, R99.1: now also Q2.1 (G)
- net at A1.9 (D6), R112.1: now also Q15.1 (G)
- net at A1.22 (A3), R137.2: now also Q25.1 (G), Q29.1 (G)
- net at Q16.3 (C), R109.1: now also Q13.1 (G)
- net at Q8.3 (C), R101.1: now also Q5.1 (G)
- net at J7.1 (Pin_1): now also Q13.2 (D)
- net at J6.1 (Pin_1): now also Q9.2 (D)
- net at J6.3 (Pin_3): now also Q10.2 (D)
- new net: Q17.3 (S), Q18.3 (S), Q19.2 (D)
- new net: Q25.2 (D), Q26.2 (D), Q27.2 (D), Q28.2 (D), Q33.3 (S)
- new net: J23.3 (Pin_3), Q26.3 (S)
- new net: J24.1 (Pin_1), Q29.3 (S)
- new net: J24.3 (Pin_3), Q25.3 (S)
- new net: Q1.3 (S), Q2.3 (S), Q3.2 (D)
- new net: Q21.3 (S), Q22.3 (S), Q23.2 (D)
- new net: Q10.3 (S), Q11.2 (D), Q9.3 (S)
- new net: Q13.3 (S), Q14.3 (S), Q15.2 (D)
- new net: J23.1 (Pin_1), Q30.3 (S)
- new net: Q5.3 (S), Q6.3 (S), Q7.2 (D)
- new net: J22.1 (Pin_1), Q31.3 (S)
- new net: J22.3 (Pin_3), Q27.3 (S)
- new net: J15.3 (Pin_3), Q28.3 (S)
Other:
- note added: "18V over"
- note added: "9.1V under"
- note added: "A"
- note added: "O"
- note added: "RAPTOR"
- note added: "Y"
- moved on the sheet: Q32, Q34, Q37, R130, R132, R133, R134, R135, R136, R137

Commit message: v1.13
Yet more schematic changes
Parts:
- removed 6A1: D, symbol Device:D
- removed C12: 0.1u, symbol Device:C
- removed C3, C4, C7, C8: 200uF, symbol Device:C_Polarized
- removed C5, C6: 100uF, symbol Device:C_Polarized
- removed C9: 4.7u, symbol Device:C_Polarized
- removed D241, D242, D243, D244: 1N5822, symbol Diode:1N5822
- removed L1, L2, L3, L4: 47uH, symbol Device:L
- removed R116, R123, R124: 4.7K, symbol Device:R
- removed R119, R120, R127, R128: 1K, symbol Device:R
- removed U1, U2, U3, U4: LM2596S-ADJ, symbol Regulator_Switching:LM2596S-ADJ
- added A1, A2, A3, A4: LM2596 DC-DC Buck, afootprints:LM2596 Buck Converter, symbol asymbols:LM2596_DC-DC_Step_Down_Module
- added C3: 0.22u, symbol Device:C
- added D241: 1N4739A, Diode_THT:D_DO-41_SOD81_P10.16mm_Horizontal, symbol Diode:1N47xxA
- added Q39: IRF4905, Package_TO_SOT_THT:TO-220-3_Vertical, symbol Transistor_FET:IRF4905
- A5: renamed from A1; footprint (none) -> afootprints:ArduinoNano
- C1, C2: value 100uF -> 330uF
- C11: value 10u -> 10uF
- D245, D246, D248, D249, D250, D251, D252: footprint (none) -> Diode_THT:D_DO-41_SOD81_P10.16mm_Horizontal
- D247: footprint (none) -> Diode_THT:D_P600_R-6_P20.00mm_Horizontal
- J1, J10, J17, J19, J2, J20, J21, J3, J8, J9: now left out of the parts list
- J11, J12, J15, J16, J22, J23, J24, J4, J5, J6, J7: footprint (none) -> afootprints:PoiLee 3-Pin
- J14: footprint (none) -> Connector_PinHeader_2.54mm:PinHeader_2x04_P2.54mm_Vertical
- K1: footprint (none) -> Relay_THT:Relay_SPDT_Finder_40.51
- Q1, Q10, Q11, Q13, Q14, Q15, Q17, Q18, Q19, Q2, Q21, Q22, Q23, Q25, Q26, Q27, Q28, Q29, Q3, Q30, Q31, Q33, Q35, Q5, Q6, Q7, Q9: footprint (none) -> afootprints:IRLR7843
- Q12, Q16, Q20, Q24, Q34, Q4, Q8: footprint (none) -> afootprints:2N3904SMD
- Q32, Q36: footprint (none) -> Package_TO_SOT_THT:TO-220-3_Vertical
- Q37, Q38: footprint (none) -> Package_TO_SOT_THT:TO-92_Inline
- R100, R101, R102, R103, R104, R105, R106, R107, R108, R109, R110, R111, R112, R113, R114, R117, R118, R121, R122, R125, R126, R130, R131, R132, R133, R134, R135, R136, R137, R138, R139, R85, R86, R87, R88, R89, R90, R91, R92, R93, R94, R95, R96, R97, R98, R99: footprint (none) -> afootprints:1206 R
- R115: value 4.7K -> 10K; footprint (none) -> afootprints:THTresistor
- R140, R141, R142, R143, R145: footprint (none) -> afootprints:THTresistor
- U5: footprint (none) -> afootprints:L7805
Connections:
- net +12V: no longer C1.1, C2.1, Q36.2 (D), U5.1 (IN)
- net BUCK_A: now also A1.2 (Vout); no longer R115.2
- net BUCK_B: now also A2.2 (Vout)
- net BUCK_C: now also A3.2 (Vout)
- net BUCK_D: now also A4.2 (Vout)
- net GND: now also R115.1, A1.3 (GND), A1.4 (GND), A2.3 (GND), A2.4 (GND), A3.3 (GND), A3.4 (GND), A4.3 (GND), A4.4 (GND), C3.2
- net at C10.1, Q36.3 (S), Q37.3 (E)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: now also C3.1, D241.1 (K), Q39.3 (S); no longer D247.1 (A1)
- net at F1.1: now also D247.1 (A1), Q39.2 (D)
- new net: A1.1 (Vin), A2.1 (Vin), A3.1 (Vin), A4.1 (Vin), C1.1, C2.1, Q36.2 (D), U5.1 (IN)
- new net: D241.2 (A), Q39.1 (G), R115.2
Other:
- note added: "Reverse Polarity"
- note added: "TVS"
- moved on the sheet: C10, C11, D181, D182, D183, D184, D185, D186, D187, D188, D189, D190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
