File: Toyota Satoshi Emblem/Toyota Satoshi Emblem.kicad_sch (KiCad schematic)
At the start: 462 parts, among them J1 Conn_01x03_Male, J10 Conn_01x03_Male, J11 Letter Terminal, J12 Letter Terminal, J13 Turn Signal Wires, J14 Power Port Term., J15 Raptor Term, J16 Serial Terminal, J17 S-Pads, J18 Turn Signal Term., J19 S-Pads, J2 Conn_01x03_Male, J20 S-Pads, J21 S-Pads, J22 Raptor Term, J23 Raptor Term, J24 Raptor Term, J25 Turn Signal Term., J3 Conn_01x03_Male, J4 Letter Terminal, J5 Letter Terminal, J6 Letter Terminal, J7 Letter Terminal, J8 Conn_01x03_Male, J9 Conn_01x03_Male, K1 FINDER-40.51, Q1 IRLR7843, Q10 IRLR7843, Q11 IRLR7843, Q12 2N3904, Q13 IRLR7843, Q14 IRLR7843, Q15 IRLR7843, Q16 2N3904, Q17 IRLR7843, Q18 IRLR7843, Q19 IRLR7843, Q2 IRLR7843, Q20 2N3904, Q21 IRLR7843, Q22 IRLR7843, Q23 IRLR7843, Q24 2N3904, Q25 IRLR7843, Q26 IRLR7843, Q27 IRLR7843, Q28 IRLR7843, Q29 IRLR7843, Q3 IRLR7843, Q30 IRLR7843, Q31 IRLR7843, Q32 IRLR7843, Q33 IRLR7843, Q34 2N3904, Q35 IRLR7843, Q36 IRF4905, Q37 BC327, Q38 BC337, Q39 IRF4905, Q4 2N3904, Q5 IRLR7843, Q6 IRLR7843, Q7 IRLR7843, Q8 2N3904, Q9 IRLR7843, U5 L7805

Commit message: v1.17
Last push before making some major changes in regards to the processor
Connections:
- net GND: now also A1.3 (GND), A2.3 (GND), A3.3 (GND), A4.3 (GND), A5.29 (GND); no longer A1.4 (GND), A2.4 (GND), A3.4 (GND), A4.4 (GND)
Changed lines of the file:
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@@
     (title "Toyota Satoshi Emblem LED Board")
     (date "2022-02-16")
-    (rev "1.16")
+    (rev "1.17")
   )
   (junction (at 80.01 161.29) (diameter 0) (color 0 0 0 0)
@@
   (junction (at 252.73 26.67) (diameter 0) (color 0 0 0 0)
   )
+  (junction (at 273.685 161.29) (diameter 0) (color 0 0 0 0)
+  )
   (junction (at 300.99 52.07) (diameter 0) (color 0 0 0 0)
   )
@@
   (junction (at 264.16 219.71) (diameter 0) (color 0 0 0 0)
   )
-  (junction (at 276.225 161.29) (diameter 0) (color 0 0 0 0)
-  )
   (junction (at 232.41 219.71) (diameter 0) (color 0 0 0 0)
   )
@@
   (junction (at 151.13 45.72) (diameter 0) (color 0 0 0 0)
   )
+  (junction (at 249.555 161.29) (diameter 0) (color 0 0 0 0)
+  )
   (junction (at 355.6 34.29) (diameter 0) (color 0 0 0 0)
   )
@@
   (junction (at 113.0299 91.4399) (diameter 0) (color 0 0 0 0)
   )
-  (junction (at 227.965 161.29) (diameter 0) (color 0 0 0 0)
-  )
   (junction (at 16.51 26.67) (diameter 0) (color 0 0 0 0)
   )
@@
   (junction (at 54.61 91.44) (diameter 0) (color 0 0 0 0)
   )
+  (junction (at 225.425 161.29) (diameter 0) (color 0 0 0 0)
+  )
   (junction (at 182.88 196.85) (diameter 0) (color 0 0 0 0)
   )
@@
   (junction (at 54.61 26.67) (diameter 0) (color 0 0 0 0)
   )
-  (junction (at 252.095 161.29) (diameter 0) (color 0 0 0 0)
-  )
   (junction (at 59.69 85.09) (diameter 0) (color 0 0 0 0)
   )
@@
     (stroke (width 0) (type default) (color 0 0 0 0))
   )
+  (wire (pts (xy 249.555 155.575) (xy 249.555 161.29))
+    (stroke (width 0) (type default) (color 0 0 0 0))
+  )
   (wire (pts (xy 59.69 233.68) (xy 58.42 233.68))
     (stroke (width 0) (type default) (color 0 0 0 0))
@@
     (stroke (width 0) (type default) (color 0 0 0 0))
   )
-  (wire (pts (xy 207.645 161.29) (xy 227.965 161.29))
+  (wire (pts (xy 207.645 161.29) (xy 225.425 161.29))
     (stroke (width 0) (type default) (color 0 0 0 0))
   )
@@
     (stroke (width 0) (type default) (color 0 0 0 0))
   )
-  (wire (pts (xy 252.095 155.575) (xy 252.095 161.29))
-    (stroke (width 0) (type default) (color 0 0 0 0))
-  )
   (wire (pts (xy 204.47 33.02) (xy 204.47 39.37))
     (stroke (width 0) (type default) (color 0 0 0 0))
@@
     (stroke (width 0) (type default) (color 0 0 0 0))
   )
-  (wire (pts (xy 252.095 161.29) (xy 276.225 161.29))
-    (stroke (width 0) (type default) (color 0 0 0 0))
-  )
   (wire (pts (xy 165.1 39.37) (xy 167.64 39.37))
     (stroke (width 0) (type default) (color 0 0 0 0))
@@
     (stroke (width 0) (type default) (color 0 0 0 0))
   )
-  (wire (pts (xy 227.965 161.29) (xy 252.095 161.29))
+  (wire (pts (xy 225.425 161.29) (xy 249.555 161.29))
     (stroke (width 0) (type default) (color 0 0 0 0))
   )
@@
     (stroke (width 0) (type default) (color 0 0 0 0))
   )
-  (wire (pts (xy 300.355 155.575) (xy 300.355 161.29))
-    (stroke (width 0) (type default) (color 0 0 0 0))
-  )
   (wire (pts (xy 54.61 104.14) (xy 57.15 104.14))
     (stroke (width 0) (type default) (color 0 0 0 0))
@@
     (stroke (width 0) (type default) (color 0 0 0 0))
   )
+  (wire (pts (xy 297.815 155.575) (xy 297.815 161.29))
+    (stroke (width 0) (type default) (color 0 0 0 0))
+  )
   (wire (pts (xy 238.76 104.14) (xy 234.95 104.14))
     (stroke (width 0) (type default) (color 0 0 0 0))
@@
     (stroke (width 0) (type default) (color 0 0 0 0))
   )
-  (wire (pts (xy 276.225 161.29) (xy 300.355 161.29))
+  (wire (pts (xy 249.555 161.29) (xy 273.685 161.29))
     (stroke (width 0) (type default) (color 0 0 0 0))
   )
@@
     (stroke (width 0) (type default) (color 0 0 0 0))
   )
+  (wire (pts (xy 225.425 155.575) (xy 225.425 161.29))
+    (stroke (width 0) (type default) (color 0 0 0 0))
+  )
   (wire (pts (xy 364.49 17.78) (xy 410.21 17.78))
     (stroke (width 0) (type default) (color 0 0 0 0))
@@
     (stroke (width 0) (type default) (color 0 0 0 0))
   )
-  (wire (pts (xy 227.965 155.575) (xy 227.965 161.29))
-    (stroke (width 0) (type default) (color 0 0 0 0))
-  )
   (wire (pts (xy 113.03 233.68) (xy 106.68 233.68))
     (stroke (width 0) (type default) (color 0 0 0 0))
@@
     (stroke (width 0) (type default) (color 0 0 0 0))
   )
+  (wire (pts (xy 273.685 155.575) (xy 273.685 161.29))
+    (stroke (width 0) (type default) (color 0 0 0 0))
+  )
   (wire (pts (xy 209.55 97.79) (xy 209.55 104.14))
     (stroke (width 0) (type default) (color 0 0 0 0))
@@
     (stroke (width 0) (type default) (color 0 0 0 0))
   )
+  (wire (pts (xy 280.67 242.57) (xy 280.67 246.38))
+    (stroke (width 0) (type default) (color 0 0 0 0))
+  )
   (wire (pts (xy 143.51 179.07) (xy 143.51 179.705))
     (stroke (width 0) (type default) (color 0 0 0 0))
@@
     (stroke (width 0) (type default) (color 0 0 0 0))
   )
+  (wire (pts (xy 273.685 161.29) (xy 297.815 161.29))
+    (stroke (width 0) (type default) (color 0 0 0 0))
+  )
   (wire (pts (xy 180.34 209.55) (xy 180.34 210.82))
     (stroke (width 0) (type default) (color 0 0 0 0))
@@
     (stroke (width 0) (type default) (color 0 0 0 0))
   )
-  (wire (pts (xy 276.225 155.575) (xy 276.225 161.29))
-    (stroke (width 0) (type default) (color 0 0 0 0))
-  )
   (wire (pts (xy 330.2 176.53) (xy 345.44 176.53))
     (stroke (width 0) (type default) (color 0 0 0 0))
@@
     (pin "2")
   )
+  (symbol (lib_id "power:GND") (at 280.67 246.38 0) (unit 1)
+    (in_bom yes) (on_board yes) (fields_autoplaced)
+    (property "Reference" "#PWR0103" (id 0) (at 280.67 252.73 0)
+      (effects (font (size 1.27 1.27)) hide)
+    )
+    (property "Value" "GND" (id 1) (at 280.67 251.46 0))
+    (property "Footprint" "" (id 2) (at 280.67 246.38 0)
+      (effects (font (size 1.27 1.27)) hide)
+    )
+    (property "Datasheet" "" (id 3) (at 280.67 246.38 0)
+      (effects (font (size 1.27 1.27)) hide)
+    )
+    (pin "1")
+  )
   (symbol (lib_id "Device:R") (at 69.85 220.98 90) (unit 1)
     (in_bom yes) (on_board yes)
@@
       (reference "#PWR0102") (unit 1) (value "GND") (footprint "")
     )
+    (path "/31f74275-ee4e-4d6a-8436-5519f98f27f0"
+      (reference "#PWR0103") (unit 1) (value "GND") (footprint "")
+    )
     (path "/995cde89-43da-42dc-b2f2-1d0c9b26802d"

Commit message: v2.0
Improved ATmega2560 micro. Future-proofing, but unfortunately have to rebuild the board and led plates yet again.
Parts:
- removed A5: Arduino_Nano_v3.x, Module:Arduino_Nano, symbol MCU_Module:Arduino_Nano_v3.x
- removed J13: Turn Signal Wires, TerminalBlock_Phoenix:TerminalBlock_Phoenix_MKDS-3-2-5.08_1x02_P5.08mm_Horizontal, symbol Connector:Conn_01x02_Male
- removed J14: Power Port Term., Connector_PinHeader_2.54mm:PinHeader_2x04_P2.54mm_Vertical, symbol Connector_Generic:Conn_02x04_Odd_Even
- removed J15, J22, J23, J24: Raptor Term, TerminalBlock_Phoenix:TerminalBlock_Phoenix_PT-1,5-3-5.0-H_1x03_P5.00mm_Horizontal, symbol Connector:Conn_01x03_Female
- removed Q25, Q26, Q27, Q28, Q29, Q30, Q31, Q32, Q33, Q35: IRLR7843, afootprints:IRLR7843, symbol asymbols:IRLR7843
- removed Q34: 2N3904, Package_TO_SOT_THT:TO-92_Inline, symbol Transistor_BJT:2N3904
- removed R130, R133, R134, R135, R136, R137: 10K, afootprints:1206 R, symbol Device:R
- removed R132, R138: 1K, afootprints:1206 R, symbol Device:R
- added D? (x2): 1N47xxA, Diode_THT:D_DO-41_SOD81_P10.16mm_Horizontal, symbol Diode:1N47xxA
- added D? (x2): 1N4733A, Diode_THT:D_DO-41_SOD81_P10.16mm_Horizontal, symbol Diode:1N47xxA
- added J?: Serial 1, TerminalBlock_Phoenix:TerminalBlock_Phoenix_PT-1,5-2-5.0-H_1x02_P5.00mm_Horizontal, symbol Connector:Conn_01x02_Male
- added J? (x4): Letter Terminal, TerminalBlock_Phoenix:TerminalBlock_Phoenix_PT-1,5-3-5.0-H_1x03_P5.00mm_Horizontal, symbol Connector:Conn_01x03_Female
- added J?: Misc. Input Term., TerminalBlock_Phoenix:TerminalBlock_Phoenix_PT-1,5-2-5.0-H_1x02_P5.00mm_Horizontal, symbol Connector:Conn_01x02_Female
- added J?: Relay Power, TerminalBlock_Phoenix:TerminalBlock_Phoenix_PT-1,5-2-5.0-H_1x02_P5.00mm_Horizontal, symbol Connector:Conn_01x02_Male
- added J?: Serial 2, TerminalBlock_Phoenix:TerminalBlock_Phoenix_PT-1,5-2-5.0-H_1x02_P5.00mm_Horizontal, symbol Connector:Conn_01x02_Male
- added J?: P Out2, TerminalBlock_Phoenix:TerminalBlock_Phoenix_PT-1,5-2-5.0-H_1x02_P5.00mm_Horizontal, symbol Connector:Conn_01x02_Male
- added J?: P Out1, TerminalBlock_Phoenix:TerminalBlock_Phoenix_PT-1,5-2-5.0-H_1x02_P5.00mm_Horizontal, symbol Connector:Conn_01x02_Male
- added Q? (x4): 2N3904, Package_TO_SOT_THT:TO-92_Inline, symbol Transistor_BJT:2N3904
- added Q? (x12): IRLR7843, afootprints:IRLR7843, symbol asymbols:IRLR7843
- added R? (x9): 1K, afootprints:1206 R, symbol Device:R
- added R? (x12): 10K, afootprints:1206 R, symbol Device:R
- added U?: MEGA_PRO_EMBED_CH340G_/_ATMEGA2560, MODULE_MEGA_PRO_EMBED_CH340G_/_ATMEGA2560, symbol asymbols:MEGA_PRO_EMBED_CH340G_/_ATMEGA2560
- A1: value LM2596 DC-DC Buck -> LM2596 Buck A
- A2: value LM2596 DC-DC Buck -> LM2596 Buck B
- A3: value LM2596 DC-DC Buck -> LM2596 Buck C
- A4: value LM2596 DC-DC Buck -> LM2596 Buck D
- J16: value Serial Terminal -> Serial 3
- J25: value Turn Signal Term. -> Power In
Connections:
- net +12V: now also J?.1 (Pin_1), J?.1 (Pin_1); no longer A1.1 (Vin), A2.1 (Vin), A3.1 (Vin), A4.1 (Vin)
- net +5V: now also U?.5V_1 (5V), U?.5V_2 (5V), U?.5V_3 (5V)
- net BUCK_D: now also J?.2 (Pin_2), J?.2 (Pin_2), J?.2 (Pin_2), J?.2 (Pin_2), R?.2, R?.2, R?.2, R?.2, R?.2, R?.2, R?.2, R?.2
- net GND: now also D?.2 (A), D?.2 (A), D?.2 (A), D?.2 (A), J?.2 (Pin_2), J?.2 (Pin_2); no longer K1.A1
- net POWER: no longer K1.14
- net at J18.1 (Pin_1): now also R?.2
- net at J18.2 (Pin_2): now also R?.2; no longer R139.1
- net at Q10.1 (G), R106.2, R107.1: now also U?.D23
- net at D249.1 (K): now also R?.1, U?.D3; no longer R139.2
- net at Q18.1 (G), R114.2, R117.1: now also U?.D21
- net at D245.1 (K), R131.1: now also U?.D15
- net at Q3.1 (G), R100.1: now also U?.D8
- net at Q11.1 (G), R108.1: now also U?.D6
- net at Q23.1 (G), R126.1: now also U?.D2
- net at Q19.1 (G), R118.1: now also U?.D3
- net at Q14.1 (G), R110.2, R111.1: now also U?.D22
- net at Q22.1 (G), R122.2, R125.1: now also U?.D20
- net at J16.2 (Pin_2): now also U?.D14
- net at D250.1 (K): now also R?.1, U?.D5
- net at Q6.1 (G), R102.2, R103.1: now also U?.D24
- net at Q15.1 (G), R112.1: now also U?.D5
- net at Q2.1 (G), R98.2, R99.1: now also U?.D25
- net at Q7.1 (G), R104.1: now also U?.D7
- net BUCK_A: no longer names the net of A1.2 (Vout), J11.2 (Pin_2), J12.2 (Pin_2), R113.2, R118.2, R121.2, R126.2
- net BUCK_B: no longer names the net of A2.2 (Vout), J6.2 (Pin_2), J7.2 (Pin_2), R105.2, R108.2, R109.2, R112.2
- net BUCK_C: no longer names the net of A3.2 (Vout), J4.2 (Pin_2), J5.2 (Pin_2), R100.2, R101.2, R104.2, R97.2
- new net: Q?.2 (B), R?.1 (x4)
- new net: Q?.1 (G), R?.1, R?.2, U?.A2
- new net: J?.1 (Pin_1), R?.2 (x2)
- new net: J?.2 (Pin_2), U?.D18
- new net: J?.1 (Pin_1), Q?.2 (D) (x4)
- new net: J?.3 (Pin_3), Q?.2 (D) (x4)
- new net: Q?.1 (G), R?.1, U?.D10
- new net: Q?.1 (G), R?.1, U?.D9
- new net: Q?.1 (E), Q?.1 (E), Q?.1 (E), Q?.1 (E), Q?.3 (S), Q?.3 (S), Q?.3 (S), Q?.3 (S), R?.2, R?.2, R?.2, R?.2
- new net: Q?.1 (G), Q?.3 (C), R?.1 (x4)
- new net: J?.1 (Pin_1), R139.2
- new net: J?.2 (Pin_2), R?.2
- new net: J?.1 (Pin_1), K1.14
- new net: D?.1 (K), R?.1, U?.D17
- new net: A1.1 (Vin), A2.1 (Vin), A3.1 (Vin), A4.1 (Vin)
- new net: Q?.1 (G), R?.1, U?.D12
- new net: Q?.2 (D), Q?.3 (S), Q?.3 (S) (x4)
- new net: D?.1 (K), R?.1, U?.D7
- new net: Q?.1 (G), R?.1, R?.2, U?.A0
- new net: Q?.1 (G), R?.1, R?.2, U?.D28' (D28)
- new net: D?.1 (K), R139.1, U?.D9
- new net: D?.1 (K), R?.1, U?.D19
- new net: Q?.1 (G), R?.1, R?.2, U?.D26
- new net: Q?.1 (G), R?.1, U?.D11
- new net: U?.3V3_1 (3V3), U?.3V3_2 (3V3)
- new net: J?.2 (Pin_2), U?.D16
- new net: U?.GND_1 (GND), U?.GND_2 (GND), U?.GND_3 (GND)
- new net: U?.VIN_1 (VIN), U?.VIN_2 (VIN)
- new net CHASSIS GND: J?.2 (Pin_2), K1.A1
Other:
- note removed: "A"
- note removed: "O"
- note removed: "RAPTOR"
- note removed: "T"
- note removed: "Y"
- moved on the sheet: A1, A2, A3, A4, C1, C11, C2, C3, C4, D1, D10, D100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

Commit message: v2.1
probably made some improvements
Parts:
- removed D145, D146, D147, D148, D149, D15, D150, D163, D164, D165, D166, D167, D168, D169, D170, D171, D172, D173, D174, D175, D176, D177, D178, D179, D18, D180, D189, D192, D195, D204, D21, D219, D222, D225, D234, D237, D24, D240: ALED, afootprints:5730 LED A, symbol Device:LED
- removed D151, D152, D153, D154, D155, D156, D157, D158, D159, D160, D161, D162: WLED, afootprints:5730 LED W, symbol Device:LED
- removed J10, J8, J9: Conn_01x03_Male, symbol Connector:Conn_01x03_Male
- removed J11, J12, J4, J5, J6, J7, J? (x4): Letter Terminal, TerminalBlock_Phoenix:TerminalBlock_Phoenix_PT-1,5-3-5.0-H_1x03_P5.00mm_Horizontal, symbol Connector:Conn_01x03_Female
- removed J16: Serial 3, TerminalBlock_Phoenix:TerminalBlock_Phoenix_PT-1,5-2-5.0-H_1x02_P5.00mm_Horizontal, symbol Connector:Conn_01x02_Male
- removed J18: Turn Signal Term., TerminalBlock_Phoenix:TerminalBlock_Phoenix_PT-1,5-2-5.0-H_1x02_P5.00mm_Horizontal, symbol Connector:Conn_01x02_Female
- removed J25: Power In, TerminalBlock_Phoenix:TerminalBlock_Phoenix_PT-1,5-2-5.0-H_1x02_P5.00mm_Horizontal, symbol Connector:Conn_01x02_Female
- removed J?: Serial 1, TerminalBlock_Phoenix:TerminalBlock_Phoenix_PT-1,5-2-5.0-H_1x02_P5.00mm_Horizontal, symbol Connector:Conn_01x02_Male
- removed J?: Misc. Input Term., TerminalBlock_Phoenix:TerminalBlock_Phoenix_PT-1,5-2-5.0-H_1x02_P5.00mm_Horizontal, symbol Connector:Conn_01x02_Female
- removed J?: Serial 2, TerminalBlock_Phoenix:TerminalBlock_Phoenix_PT-1,5-2-5.0-H_1x02_P5.00mm_Horizontal, symbol Connector:Conn_01x02_Male
- removed J?: P Out2, TerminalBlock_Phoenix:TerminalBlock_Phoenix_PT-1,5-2-5.0-H_1x02_P5.00mm_Horizontal, symbol Connector:Conn_01x02_Male
- removed J?: P Out1, TerminalBlock_Phoenix:TerminalBlock_Phoenix_PT-1,5-2-5.0-H_1x02_P5.00mm_Horizontal, symbol Connector:Conn_01x02_Male
- removed R117, R125, R? (x4): 10K, afootprints:1206 R, symbol Device:R
- added D206, D208, D209, D211: LED, LED_SMD:LED_1206_3216Metric_Pad1.42x1.75mm_HandSolder, symbol Device:LED
- added D212, D213, D214: RED 1206, LED_SMD:LED_1206_3216Metric_Pad1.42x1.75mm_HandSolder, symbol Device:LED
- added D25, D26, D28, D29: WLED, afootprints:5730 LED W, symbol Device:LED
- added J11, J12, J13, J14, J15, J16: Letter Terminal, TerminalBlock_Phoenix:TerminalBlock_Phoenix_MKDS-1,5-3_1x03_P5.00mm_Horizontal, symbol Connector:Screw_Terminal_01x03
- added J17: Power 1, TerminalBlock_Phoenix:TerminalBlock_Phoenix_MKDS-1,5-2_1x02_P5.00mm_Horizontal, symbol Connector:Screw_Terminal_01x02
- added J18: Power 2, TerminalBlock_Phoenix:TerminalBlock_Phoenix_MKDS-1,5-2_1x02_P5.00mm_Horizontal, symbol Connector:Screw_Terminal_01x02
- added J19, J20, J23, J25: Raptor Terminal, TerminalBlock_Phoenix:TerminalBlock_Phoenix_MKDS-1,5-3-5.08_1x03_P5.08mm_Horizontal, symbol Connector:Screw_Terminal_01x03
- added J21: Serial 3, TerminalBlock_Phoenix:TerminalBlock_Phoenix_MKDS-1,5-2_1x02_P5.00mm_Horizontal, symbol Connector:Screw_Terminal_01x02
- added J22: Serial 2, TerminalBlock_Phoenix:TerminalBlock_Phoenix_MKDS-1,5-2_1x02_P5.00mm_Horizontal, symbol Connector:Screw_Terminal_01x02
- added J24: Serial 1, TerminalBlock_Phoenix:TerminalBlock_Phoenix_MKDS-1,5-2_1x02_P5.00mm_Horizontal, symbol Connector:Screw_Terminal_01x02
- added J26: Turn Sig., TerminalBlock_Phoenix:TerminalBlock_Phoenix_MKDS-1,5-2_1x02_P5.00mm_Horizontal, symbol Connector:Screw_Terminal_01x02
- added J27: Misc. Sig., TerminalBlock_Phoenix:TerminalBlock_Phoenix_MKDS-1,5-2_1x02_P5.00mm_Horizontal, symbol Connector:Screw_Terminal_01x02
- added J29: Power In, TerminalBlock_Phoenix:TerminalBlock_Phoenix_MKDS-1,5-2_1x02_P5.00mm_Horizontal, symbol Connector:Screw_Terminal_01x02
- added J4, J5, J6: Letter Pads, symbol Connector:Conn_01x03_Male
- added R116, R118, R151, R153, R155, R157, R159, R161, R163, R165, R167, R169: 1K, afootprints:1206 R, symbol Device:R
- added R124: 50, afootprints:1206 R, symbol Device:R
- added R150, R152, R154, R156, R158, R160, R162, R164, R166, R168: 10K, afootprints:1206 R, symbol Device:R
- added SW1: SW_DIP_x10, Button_Switch_THT:SW_DIP_SPSTx10_Slide_9.78x27.58mm_W7.62mm_P2.54mm, symbol Switch:SW_DIP_x10
- A1: value LM2596 Buck A -> LM2596 Buck
- A2: value LM2596 Buck B -> LM2596 Buck
- A3: value LM2596 Buck C -> LM2596 Buck
- A4: value LM2596 Buck D -> LM2596 Buck
- D103, D104, D105, D106, D107, D108, D27, D30, D49, D50, D51, D52, D53, D54, D55, D56, D57, D58, D59, D60, D73, D74, D75, D76, D77, D78, D79, D80, D81, D82, D83, D84: value ALED -> WLED; footprint afootprints:5730 LED A -> afootprints:5730 LED W
- D194: renamed from D249; value 1N4733A -> 1N4732A
- D195: renamed from D250; value 1N4733A -> 1N4732A
- D196, D197: renamed from D?; value 1N4733A -> 1N4732A
- D207, D210: value ALED -> LED; footprint afootprints:5730 LED A -> LED_SMD:LED_1206_3216Metric_Pad1.42x1.75mm_HandSolder
- D37, D38, D39, D40, D41, D42, D61, D62, D63, D64, D65, D66, D67, D68, D69, D70, D71, D72, D91, D92, D93, D94, D95, D96: value WLED -> ALED; footprint afootprints:5730 LED W -> afootprints:5730 LED A
- J1, J2, J3: value Conn_01x03_Male -> Letter Pads
- J10: renamed from J21; value S-Pads -> Raptor Pads
- J7: renamed from J17; value S-Pads -> Raptor Pads
- J8: renamed from J19; value S-Pads -> Raptor Pads
- J9: renamed from J20; value S-Pads -> Raptor Pads
- R103, R107, R111, R99: value 10K -> 1K
- U1: renamed from U?; footprint MODULE_MEGA_PRO_EMBED_CH340G_/_ATMEGA2560 -> afootprints:MODULE_MEGA_PRO_EMBED_CH340G___ATMEGA2560
- gave numbers to parts that had none: 36
- renumbered C3 to C1, C4 to C2, C11 to C3, C1 to C4, C2 to C5, D181 to D145, D182 to D146, D183 to D147, D184 to D148, D185 to D149, D16 to D15, D186 to D150, D187 to D151, D188 to D152, D190 to D153, D191 to D154, D193 to D155, D194 to D156, D196 to D157, D197 to D158, D198 to D159, D17 to D16, D199 to D160, D200 to D161, D201 to D162, D202 to D163, D203 to D164, D205 to D165, D206 to D166, D208 to D167, D209 to D168, D211 to D169, D19 to D17, D212 to D170, D213 to D171, D214 to D172, D215 to D173, D216 to D174, D217 to D175, D218 to D176, D220 to D177, D221 to D178, D223 to D179, D20 to D18, D224 to D180, D226 to D181, D227 to D182, D228 to D183, D229 to D184, D230 to D185, D231 to D186, D232 to D187, D233 to D188, D235 to D189, D22 to D19, D236 to D190, D238 to D191, D239 to D192, D245 to D193, D23 to D20, D246 to D200, D247 to D201, D241 to D202, D248 to D203, D251 to D204, D252 to D205, D25 to D21, D26 to D22, D28 to D23, D29 to D24, Q20 to Q22, Q21 to Q25, Q22 to Q26, Q23 to Q27, Q24 to Q30, Q39 to Q41, Q36 to Q42, Q37 to Q43, Q38 to Q44, R118 to R119, R126 to R127, R139 to R135, R131 to R139, R140 to R144, R141 to R145, R142 to R146, R143 to R147, R115 to R148, R145 to R149, U5 to U2
Connections:
- net +12V: now also A1.1 (Vin), A2.1 (Vin), A3.1 (Vin), A4.1 (Vin), J17.1 (Pin_1), J18.1 (Pin_1)
- net +5V: now also R150.1, R152.1, R154.1, R156.1, R158.1, R160.1, R162.1, R164.1, R166.1, R168.1
- net BUCK_D: now also J19.2 (Pin_2), J20.2 (Pin_2), J23.2 (Pin_2), J25.2 (Pin_2), R124.2
- net CHASSIS GND: no longer K1.A1
- net GND: now also D207.1 (K), D210.1 (K), Q23.3 (S), Q24.1 (E), Q31.3 (S), Q32.1 (E), Q35.3 (S), Q36.1 (E), Q39.3 (S), Q40.1 (E), U1.GND_1 (GND), U1.GND_2 (GND), U1.GND_3 (GND), D206.1 (K), D208.1 (K), D209.1 (K), D211.1 (K), D214.1 (K), J17.2 (Pin_2), J18.2 (Pin_2), J29.2 (Pin_2), R151.1, R153.1, R155.1, R157.1, R159.1, R161.1, R163.1, R165.1, R167.1, R169.1; no longer R103.2, R107.2, R111.2, R99.2
- net at D138.1 (K), D144.1 (K): now also D134.1 (K), D136.1 (K), D140.1 (K), D142.1 (K), J6.3 (Pin_3); no longer D135.1 (K), D141.1 (K)
- net BUCK_C: now reaches R113.2, R119.2, R121.2, R127.2
- net BUCK_C: now also A3.2 (Vout), J15.2 (Pin_2), J16.2 (Pin_2); no longer A1.2 (Vout)
- net at D18.1 (K): now also D14.1 (K), D16.1 (K), D20.1 (K), D22.1 (K), D24.1 (K), J1.3 (Pin_3)
- net at D107.1 (K): now also D101.1 (K), D103.1 (K), D105.1 (K), D97.1 (K), D99.1 (K), J5.1 (Pin_1); no longer D108.2 (A)
- net at D78.2 (A): now also R39.2; no longer D77.1 (K)
- net at Q38.1 (G), R138.2: now also U1.D29, R168.2, SW1.10; no longer U1.A2
- net at R133.2: now also J27.1 (Pin_1)
- net at R132.2: now also J27.2 (Pin_2)
- net at D124.2 (A): now also R62.2; no longer R50.2
- net at D50.1 (K): now also D49.2 (A); no longer D51.2 (A)
- net BUCK_A: now reaches R100.2, R101.2, R104.2, R97.2
- net BUCK_A: now also A1.2 (Vout), J11.2 (Pin_2), J12.2 (Pin_2); no longer A3.2 (Vout)
- net at R143.2: now also J24.1 (Pin_1)
- net TX1: now reaches U1.D18
- net TX1: now also D199.1 (K), R143.1, R99.2
- net at Q20.2 (D): now also J19.1 (Pin_1)
- net at Q21.2 (D): now also J19.3 (Pin_3)
- net at J10.3 (Pin_3): now also D188.1 (K), D190.1 (K), D192.1 (K)
- net at R13.2: now also D26.2 (A); no longer D32.2 (A)
- net at R61.1, R62.1, R63.1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: now also J6.2 (Pin_2)
- net at D92.1 (K): now also D86.1 (K), D88.1 (K), D90.1 (K), D94.1 (K), D96.1 (K), J4.3 (Pin_3); no longer D91.2 (A)
- net at R37.2: now also D74.2 (A); no longer D92.2 (A)
- net at Q10.1 (G), R106.2, U1.D23: now also R156.2, SW1.4; no longer R107.1
- net at R59.2: now also D117.2 (A)
- net at D115.2 (A): now also R58.2; no longer R47.2
- net at D178.1 (K): now also D176.1 (K), D180.1 (K), J9.3 (Pin_3)
- net at D57.2 (A): now also D58.1 (K); no longer D56.1 (K)
- net at D194.1 (K), R132.1: now also U1.A0; no longer U1.D3
- net at Q18.1 (G), R114.2, U1.D21: now also R152.2, SW1.2
- net at Q18.2 (D): now also J15.3 (Pin_3)
- net at D168.1 (K): now also D164.1 (K), D166.1 (K), J8.3 (Pin_3); no longer D210.2 (A)
- net at D121.1 (K), D123.1 (K), D125.1 (K)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: now also J6.1 (Pin_1)
- net at R14.2: now also D28.2 (A); no longer D34.2 (A)
- net at R37.1, R38.1, R39.1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: now also J4.2 (Pin_2)
- net at R46.2: now also D91.2 (A); no longer D112.2 (A)
- net at R63.2: now also D126.2 (A)
- net at R19.2: now also D37.2 (A); no longer D43.2 (A)
- net at D93.2 (A): now also R47.2; no longer D94.1 (K)
- net at D94.2 (A): now also D93.1 (K); no longer R38.2
- net at J7.3 (Pin_3): now also D152.1 (K), D154.1 (K), D156.1 (K)
- net at D27.2 (A): now also D28.1 (K); no longer D22.1 (K)
- net at D62.1 (K): now also D64.1 (K), D66.1 (K), D68.1 (K), D70.1 (K), D72.1 (K), J3.3 (Pin_3); no longer D61.2 (A)
- net at D62.2 (A): now also D61.1 (K); no longer R25.2
- net at R69.2: now also D137.2 (A)
- net at R28.2: now also D56.2 (A); no longer D68.2 (A)
- net at D31.1 (K), D33.1 (K), D35.1 (K)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: now also D27.1 (K), D25.1 (K), D29.1 (K); no longer D37.1 (K), D39.1 (K), D41.1 (K)
- net at D38.1 (K): now also D40.1 (K), D42.1 (K), D44.1 (K), D46.1 (K), D48.1 (K), J2.3 (Pin_3); no longer D37.2 (A)
- net at R49.1, R50.1, R51.1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: now also J5.2 (Pin_2)
- net at R54.2: now also D108.2 (A); no longer D132.2 (A)
- net RX3: now reaches D193.1 (K), R139.1, U1.D15
- net RX3: now also R118.2
- net at R135.2: now also J26.1 (Pin_1)
- net at R134.2: now also J26.2 (Pin_2)
- net at Q1.2 (D): now also J11.1 (Pin_1)
- net at Q2.2 (D): now also J11.3 (Pin_3)
- net BUCK_B: now reaches A2.2 (Vout), R105.2, R108.2, R109.2, R112.2
- net BUCK_B: now also J13.2 (Pin_2), J14.2 (Pin_2)
- net at R22.2: now also D43.2 (A); no longer D52.2 (A)
- net at D49.1 (K): now also D51.1 (K), D53.1 (K), D55.1 (K), D57.1 (K), D59.1 (K), J3.1 (Pin_1); no longer D50.2 (A)
- net at R21.2: now also D41.2 (A); no longer D49.2 (A)
- net at R57.2: now also D113.2 (A); no longer D139.2 (A)
- net at J28.1 (Pin_1), K1.14: now also K1.A1
- net at Q5.2 (D): now also J12.1 (Pin_1)
- net at Q6.2 (D): now also J12.3 (Pin_3)
- net at R18.2: now also D36.2 (A); no longer D42.2 (A)
- net at D135.2 (A): now also R68.2; no longer D134.1 (K)
- net at Q37.2 (D): now also J25.1 (Pin_1)
- net at Q38.2 (D): now also J25.3 (Pin_3)
- net TX2: now reaches D198.1 (K), R142.1
- net TX2: now also R107.2, U1.D16; no longer U1.D17
- net at R51.2: now also D102.2 (A); no longer D126.2 (A)
- net at R36.2: now also D71.2 (A); no longer D88.2 (A)
- net at D74.1 (K): now also D73.2 (A); no longer D75.2 (A)
- net at D73.1 (K): now also D75.1 (K), D77.1 (K), D79.1 (K), D81.1 (K), D83.1 (K), J4.1 (Pin_1); no longer D74.2 (A)
- net at Q28.2 (D): now also J20.1 (Pin_1)
- net at Q29.2 (D): now also J20.3 (Pin_3)
- net at R23.2: now also D45.2 (A); no longer D55.2 (A)
- net at R61.2: now also D122.2 (A)
- net at D128.2 (A): now also R64.2; no longer R52.2
- net at R49.2: now also D98.2 (A); no longer D122.2 (A)
- net at D196.1 (K), R134.1: now also U1.A2; no longer U1.D7
- net at Q14.1 (G), R110.2, U1.D22: now also R154.2, SW1.3; no longer R111.1
- net at D63.2 (A): now also R32.2; no longer D64.1 (K)
- net at D64.2 (A): now also D63.1 (K); no longer R26.2
- net at D80.1 (K): now also D79.2 (A); no longer D81.2 (A)
- net at Q34.1 (G), R130.2: now also U1.D28, R166.2, SW1.9; no longer U1.A0
- net at D110.1 (K): now also D112.1 (K), D114.1 (K), D116.1 (K), D118.1 (K), D120.1 (K), J5.3 (Pin_3); no longer D111.2 (A)
- net at D87.2 (A): now also R44.2; no longer D86.1 (K)
- net at D47.2 (A): now also R24.2; no longer D46.1 (K)
- net at R20.2: now also D39.2 (A); no longer D46.2 (A)
- net at D70.2 (A): now also D69.1 (K); no longer R29.2
- net at Q34.2 (D): now also J23.3 (Pin_3)
- net at D82.2 (A): now also R41.2; no longer R34.2
- net at Q26.1 (G), R122.2, U1.D20: now also R150.2, SW1.1
- net at Q26.2 (D): now also J16.3 (Pin_3)
- net at R67.2: now also D133.2 (A)
- net at D80.2 (A): now also R40.2; no longer D79.1 (K)
- net at R33.2: now also D65.2 (A); no longer D79.2 (A)
- net at R139.2: now also J21.1 (Pin_1)
- net TX3: now reaches U1.D14
- net TX3: now also J21.2 (Pin_2), R116.2
- net at Q6.1 (G), R102.2, U1.D24: now also R158.2, SW1.5; no longer R103.1
- net at D95.2 (A): now also R48.2; no longer D96.1 (K)
- net at D96.2 (A): now also D95.1 (K); no longer R39.2
- net at D69.2 (A): now also R35.2; no longer D70.1 (K)
- net at R31.2: now also D61.2 (A); no longer D73.2 (A)
- net at R65.2: now also D130.2 (A)
- net at Q29.1 (G), R125.2: now also U1.D27, R164.2, SW1.8; no longer U1.D28' (D28)
- net at D197.1 (K), R135.1: now also U1.A3; no longer U1.D9
- net at Q14.2 (D): now also J14.3 (Pin_3)
- net at D60.2 (A): now also R30.2; no longer D59.1 (K)
- net at R142.2: now also J22.1 (Pin_1)
- net at D84.2 (A): now also R42.2; no longer D83.1 (K)
- net at D83.2 (A): now also D84.1 (K); no longer D82.1 (K)
- net at D59.2 (A): now also D60.1 (K); no longer D58.1 (K)
- net at R66.2: now also D132.2 (A)
- net at D105.2 (A): now also D106.1 (K); no longer D104.1 (K)
- net at D104.2 (A): now also R52.2; no longer D103.1 (K)
- net at D143.2 (A): now also R72.2; no longer D142.1 (K)
- net at Q2.1 (G), R98.2, U1.D25: now also R160.2, SW1.6; no longer R99.1
- net at D207.2 (A): now also R103.1; no longer D166.1 (K)
- net at R43.2: now also D85.2 (A); no longer D103.2 (A)
- net at D136.2 (A): now also D135.1 (K); no longer R56.2
- net at D106.2 (A): now also R53.2; no longer R44.2
- net at D72.2 (A): now also D71.1 (K); no longer R30.2
- net at Q21.1 (G), R117.2, U1.D26: now also R162.2, SW1.7
- net at D89.2 (A): now also R45.2; no longer D88.1 (K)
- net at D107.2 (A): now also D108.1 (K); no longer D106.1 (K)
- net at D77.2 (A): now also D78.1 (K); no longer D76.1 (K)
- net at R55.2: now also D109.2 (A); no longer D133.2 (A)
- net at D76.2 (A): now also R38.2; no longer R32.2
- net at D67.2 (A): now also R34.2; no longer D68.1 (K)
- net at Q33.2 (D): now also J23.1 (Pin_1)
- net at Q13.2 (D): now also J14.1 (Pin_1)
- net at D38.2 (A): now also D37.1 (K); no longer R16.2
- net at D119.2 (A): now also R60.2; no longer D118.1 (K)
- net at D118.2 (A): now also D117.1 (K); no longer R48.2
- net at Q25.2 (D): now also J16.1 (Pin_1)
- net at R17.2: now also D34.2 (A); no longer D40.2 (A)
- net at D58.2 (A): now also R29.2; no longer R24.2
- net at D142.2 (A): now also D141.1 (K); no longer R58.2
- net at D100.2 (A): now also R50.2; no longer R41.2
- net at D195.1 (K), R133.1: now also U1.A1; no longer U1.D5
- net at Q17.2 (D): now also J15.1 (Pin_1)
- net at D30.2 (A): now also R15.2; no longer D24.1 (K)
- net at R71.2: now also D141.2 (A)
- net at D54.2 (A): now also R27.2; no longer D53.1 (K)
- net at D53.2 (A): now also D54.1 (K); no longer D52.1 (K)
- net at D66.2 (A): now also D65.1 (K); no longer R27.2
- net at Q9.2 (D): now also J13.1 (Pin_1)
- net at Q10.2 (D): now also J13.3 (Pin_3)
- net RX2: now reaches U1.D17
- net RX2: now also R111.2, J22.2 (Pin_2)
- net RX1: now reaches U1.D19
- net RX1: now also R103.2, J24.2 (Pin_2)
- net at R70.2: now also D139.2 (A)
- net POWER: no longer names the net of F1.2
- net POWER: now also J29.1 (Pin_1)
- new net: R169.2, SW1.11
- new net: R167.2, SW1.12
- new net: R165.2, SW1.13
- new net: R163.2, SW1.14
- new net: R161.2, SW1.15
- new net: R159.2, SW1.16
- new net: R157.2, SW1.17
- new net: R155.2, SW1.18
- new net: R153.2, SW1.19
- new net: R151.2, SW1.20
- new net: D208.2 (A), R107.1
- new net: D55.2 (A), D56.1 (K)
- new net: D29.2 (A), D30.1 (K)
- new net: D91.1 (K), D92.2 (A)
- new net: D213.1 (K), D214.2 (A)
- new net: D212.1 (K), D213.2 (A)
- new net: D111.2 (A), R56.2
- new net: D81.2 (A), D82.1 (K)
- new net: D212.2 (A), R124.1
- new net: D32.2 (A), R16.2
- new net: D206.2 (A), R99.1
- new net: D25.2 (A), D26.1 (K)
- new net: D210.2 (A), R116.1
- new net: D209.2 (A), R111.1
- new net: D211.2 (A), R118.1
- new net: D87.1 (K), D88.2 (A)
- new net: D39.1 (K), D40.2 (A)
- new net: D51.2 (A), D52.1 (K)
- new net: D52.2 (A), R26.2
- new net: D45.1 (K), D46.2 (A)
- new net: D41.1 (K), D42.2 (A)
- new net: D67.1 (K), D68.2 (A)
- new net: D103.2 (A), D104.1 (K)
- new net: D50.2 (A), R25.2
- new net: D111.1 (K), D112.2 (A)
- new net: D75.2 (A), D76.1 (K)
Other:
- moved on the sheet: C1, C2, C3, C4, C5, D193, D194, D195, D196, D197, D198, D199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

Commit message: v2.5
Power/control board progress
Parts:
- Q41, Q42: footprint Package_TO_SOT_THT:TO-220-3_Vertical -> afootprints:IRF4905
Changed lines of the file:
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@@
     (title "Toyota Satoshi Emblem LED Board")
     (date "2022-04-23")
-    (rev "2.4")
+    (rev "2.5")
     (comment 1 "Daniel Hoefer")
     (comment 2 "Daniel Hoefer")
@@
     (property "Reference" "Q42" (id 0) (at 161.925 222.885 90))
     (property "Value" "IRF4905" (id 1) (at 161.925 225.425 90))
-    (property "Footprint" "Package_TO_SOT_THT:TO-220-3_Vertical" (id 2) (at 160.02 226.695 0)
+    (property "Footprint" "afootprints:IRF4905" (id 2) (at 160.02 226.695 0)
       (effects (font (size 1.27 1.27) italic) (justify left) hide)
     )
@@
     (property "Reference" "Q41" (id 0) (at 78.74 231.14 90))
     (property "Value" "IRF4905" (id 1) (at 85.725 237.49 0))
-    (property "Footprint" "Package_TO_SOT_THT:TO-220-3_Vertical" (id 2) (at 85.725 226.695 0)
+    (property "Footprint" "afootprints:IRF4905" (id 2) (at 85.725 226.695 0)
       (effects (font (size 1.27 1.27) italic) (justify left) hide)
     )
@@
     )
     (path "/fd375310-3381-4311-b1cc-0be7b09f83d4"
-      (reference "Q41") (unit 1) (value "IRF4905") (footprint "Package_TO_SOT_THT:TO-220-3_Vertical")
+      (reference "Q41") (unit 1) (value "IRF4905") (footprint "afootprints:IRF4905")
     )
     (path "/14742c2c-9edd-4391-a874-64e776e4f81e"
-      (reference "Q42") (unit 1) (value "IRF4905") (footprint "Package_TO_SOT_THT:TO-220-3_Vertical")
+      (reference "Q42") (unit 1) (value "IRF4905") (footprint "afootprints:IRF4905")
     )
     (path "/888085dd-f9d1-4c25-bb33-becfd12e628d"
