File: Toyota Satoshi Emblem/Toyota Satoshi Emblem.kicad_sch (KiCad schematic)
At the start: 467 parts, among them J1 Letter Pads, J10 Raptor Pads, J11 Letter Terminal, J12 Letter Terminal, J13 Letter Terminal, J14 Letter Terminal, J15 Letter Terminal, J16 Letter Terminal, J17 Power 1, J18 Power 2, J19 Raptor Terminal, J2 Letter Pads, J20 Raptor Terminal, J21 Serial 3, J22 Serial 2, J23 Raptor Terminal, J24 Serial 1, J25 Raptor Terminal, J26 Turn Sig., J27 Misc. Sig., J28 Relay Power, J29 Power In, J3 Letter Pads, J4 Letter Pads, J5 Letter Pads, J6 Letter Pads, J7 Raptor Pads, J8 Raptor Pads, J9 Raptor Pads, K1 FINDER-40.51, Q1 IRLR7843, Q10 IRLR7843, Q11 IRLR7843, Q12 2N3904, Q13 IRLR7843, Q14 IRLR7843, Q15 IRLR7843, Q16 2N3904, Q17 IRLR7843, Q18 IRLR7843, Q19 IRLR7843, Q2 IRLR7843, Q20 IRLR7843, Q21 IRLR7843, Q22 2N3904, Q23 IRLR7843, Q24 2N3904, Q25 IRLR7843, Q26 IRLR7843, Q27 IRLR7843, Q28 IRLR7843, Q29 IRLR7843, Q3 IRLR7843, Q30 2N3904, Q31 IRLR7843, Q32 2N3904, Q33 IRLR7843, Q34 IRLR7843, Q35 IRLR7843, Q36 2N3904, Q37 IRLR7843, Q38 IRLR7843, Q39 IRLR7843, Q4 2N3904, Q40 2N3904, Q41 IRF4905, Q42 IRF4905, Q43 BC327, Q44 BC337, Q5 IRLR7843, Q6 IRLR7843, Q7 IRLR7843, Q8 2N3904, Q9 IRLR7843, SW1 SW_DIP_x10, U1 MEGA_PRO_EMBED_CH340G_{slash}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, U2 L7805

Commit message: v2.6
More power/control board progress
Parts:
- Q12, Q16, Q22, Q24, Q30, Q32, Q36, Q4, Q40, Q8: footprint Package_TO_SOT_THT:TO-92_Inline -> Package_TO_SOT_SMD:SOT-23
Changed lines of the file:
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@@
     (title "Toyota Satoshi Emblem LED Board")
     (date "2022-04-23")
-    (rev "2.5")
+    (rev "2.6")
     (comment 1 "Daniel Hoefer")
     (comment 2 "Daniel Hoefer")
@@
       (effects (font (size 1.27 1.27)) (justify left))
     )
-    (property "Footprint" "Package_TO_SOT_THT:TO-92_Inline" (id 2) (at 340.995 127.635 0)
+    (property "Footprint" "Package_TO_SOT_SMD:SOT-23" (id 2) (at 340.995 127.635 0)
       (effects (font (size 1.27 1.27) italic) (justify left) hide)
     )
@@
       (effects (font (size 1.27 1.27)) (justify left))
     )
-    (property "Footprint" "Package_TO_SOT_THT:TO-92_Inline" (id 2) (at 340.995 79.375 0)
+    (property "Footprint" "Package_TO_SOT_SMD:SOT-23" (id 2) (at 340.995 79.375 0)
       (effects (font (size 1.27 1.27) italic) (justify left) hide)
     )
@@
       (effects (font (size 1.27 1.27)) (justify left))
     )
-    (property "Footprint" "Package_TO_SOT_THT:TO-92_Inline" (id 2) (at 131.445 205.105 0)
+    (property "Footprint" "Package_TO_SOT_SMD:SOT-23" (id 2) (at 131.445 205.105 0)
       (effects (font (size 1.27 1.27) italic) (justify left) hide)
     )
@@
       (effects (font (size 1.27 1.27)) (justify left))
     )
-    (property "Footprint" "Package_TO_SOT_THT:TO-92_Inline" (id 2) (at 131.445 132.715 0)
+    (property "Footprint" "Package_TO_SOT_SMD:SOT-23" (id 2) (at 131.445 132.715 0)
       (effects (font (size 1.27 1.27) italic) (justify left) hide)
     )
@@
       (effects (font (size 1.27 1.27)) (justify left))
     )
-    (property "Footprint" "Package_TO_SOT_THT:TO-92_Inline" (id 2) (at 340.995 151.765 0)
+    (property "Footprint" "Package_TO_SOT_SMD:SOT-23" (id 2) (at 340.995 151.765 0)
       (effects (font (size 1.27 1.27) italic) (justify left) hide)
     )
@@
       (effects (font (size 1.27 1.27)) (justify left))
     )
-    (property "Footprint" "Package_TO_SOT_THT:TO-92_Inline" (id 2) (at 340.995 103.505 0)
+    (property "Footprint" "Package_TO_SOT_SMD:SOT-23" (id 2) (at 340.995 103.505 0)
       (effects (font (size 1.27 1.27) italic) (justify left) hide)
     )
@@
       (effects (font (size 1.27 1.27)) (justify left))
     )
-    (property "Footprint" "Package_TO_SOT_THT:TO-92_Inline" (id 2) (at 340.995 55.245 0)
+    (property "Footprint" "Package_TO_SOT_SMD:SOT-23" (id 2) (at 340.995 55.245 0)
       (effects (font (size 1.27 1.27) italic) (justify left) hide)
     )
@@
       (effects (font (size 1.27 1.27)) (justify left))
     )
-    (property "Footprint" "Package_TO_SOT_THT:TO-92_Inline" (id 2) (at 131.445 180.975 0)
+    (property "Footprint" "Package_TO_SOT_SMD:SOT-23" (id 2) (at 131.445 180.975 0)
       (effects (font (size 1.27 1.27) italic) (justify left) hide)
     )
@@
       (effects (font (size 1.27 1.27)) (justify left))
     )
-    (property "Footprint" "Package_TO_SOT_THT:TO-92_Inline" (id 2) (at 340.995 31.115 0)
+    (property "Footprint" "Package_TO_SOT_SMD:SOT-23" (id 2) (at 340.995 31.115 0)
       (effects (font (size 1.27 1.27) italic) (justify left) hide)
     )
@@
       (effects (font (size 1.27 1.27)) (justify left))
     )
-    (property "Footprint" "Package_TO_SOT_THT:TO-92_Inline" (id 2) (at 131.445 156.845 0)
+    (property "Footprint" "Package_TO_SOT_SMD:SOT-23" (id 2) (at 131.445 156.845 0)
       (effects (font (size 1.27 1.27) italic) (justify left) hide)
     )
@@
     )
     (path "/d080b80b-8e24-4835-bdca-98a351852494"
-      (reference "Q4") (unit 1) (value "2N3904") (footprint "Package_TO_SOT_THT:TO-92_Inline")
+      (reference "Q4") (unit 1) (value "2N3904") (footprint "Package_TO_SOT_SMD:SOT-23")
     )
     (path "/e33e9b8b-2d1f-4515-8e7c-42e86d6442e6"
@@
     )
     (path "/bf33fdb4-7fad-4a2a-b684-563160065159"
-      (reference "Q8") (unit 1) (value "2N3904") (footprint "Package_TO_SOT_THT:TO-92_Inline")
+      (reference "Q8") (unit 1) (value "2N3904") (footprint "Package_TO_SOT_SMD:SOT-23")
     )
     (path "/f4997be3-57ad-4e13-872c-6c7cd3cb036e"
@@
     )
     (path "/1008f2dd-7392-40de-8ea9-c990f44c3bb7"
-      (reference "Q12") (unit 1) (value "2N3904") (footprint "Package_TO_SOT_THT:TO-92_Inline")
+      (reference "Q12") (unit 1) (value "2N3904") (footprint "Package_TO_SOT_SMD:SOT-23")
     )
     (path "/8f0ca3ca-e251-49e5-9d73-d95fe312aa21"
@@
     )
     (path "/948239e2-e3fd-457b-a447-72feb742c550"
-      (reference "Q16") (unit 1) (value "2N3904") (footprint "Package_TO_SOT_THT:TO-92_Inline")
+      (reference "Q16") (unit 1) (value "2N3904") (footprint "Package_TO_SOT_SMD:SOT-23")
     )
     (path "/bf9cbfcf-0f17-452d-be52-d5cf8da24a72"
@@
     )
     (path "/0853ff58-e64d-4143-b5e8-4b7ceedfdc16"
-      (reference "Q22") (unit 1) (value "2N3904") (footprint "Package_TO_SOT_THT:TO-92_Inline")
+      (reference "Q22") (unit 1) (value "2N3904") (footprint "Package_TO_SOT_SMD:SOT-23")
     )
     (path "/434c72af-bce5-447e-9037-ac349280aab6"
@@
     )
     (path "/646e38e8-7543-4c2f-bf38-1cf7d7c4dcb9"
-      (reference "Q24") (unit 1) (value "2N3904") (footprint "Package_TO_SOT_THT:TO-92_Inline")
+      (reference "Q24") (unit 1) (value "2N3904") (footprint "Package_TO_SOT_SMD:SOT-23")
     )
     (path "/f91454f5-4790-49be-a036-00b27cd7cac8"
@@
     )
     (path "/924d96e9-0a37-4069-a61e-b4b485eba1e4"
-      (reference "Q30") (unit 1) (value "2N3904") (footprint "Package_TO_SOT_THT:TO-92_Inline")
+      (reference "Q30") (unit 1) (value "2N3904") (footprint "Package_TO_SOT_SMD:SOT-23")
     )
     (path "/84eeb39f-304d-4d63-b496-b0c71700a3f6"
@@
     )
     (path "/fcd76f20-a1a1-417c-8d3f-c8e0cc6e2d95"
-      (reference "Q32") (unit 1) (value "2N3904") (footprint "Package_TO_SOT_THT:TO-92_Inline")
+      (reference "Q32") (unit 1) (value "2N3904") (footprint "Package_TO_SOT_SMD:SOT-23")
     )
     (path "/8e2ac359-dc33-4ce2-b79d-b453ff026e82"
@@
     )
     (path "/cde1c00f-d68c-4397-94f7-c14814d89c43"
-      (reference "Q36") (unit 1) (value "2N3904") (footprint "Package_TO_SOT_THT:TO-92_Inline")
+      (reference "Q36") (unit 1) (value "2N3904") (footprint "Package_TO_SOT_SMD:SOT-23")
     )
     (path "/58214775-e58a-4ae2-8a3a-a2018ea1ffc8"
@@
     )
     (path "/19eca234-e270-47b6-ab60-118a1b67c529"
-      (reference "Q40") (unit 1) (value "2N3904") (footprint "Package_TO_SOT_THT:TO-92_Inline")
+      (reference "Q40") (unit 1) (value "2N3904") (footprint "Package_TO_SOT_SMD:SOT-23")
     )
     (path "/fd375310-3381-4311-b1cc-0be7b09f83d4"
