File: Toyota Satoshi Emblem/Toyota Satoshi Emblem.kicad_pcb (KiCad board)
At the start: 2 copper layers, 175 x 100 mm, 366 parts

Commit message: v1.12
many changes
Parts:
- moved D196 132.0 mm to (73.3, 182.1)
- moved D197 132.0 mm to (83.0, 182.1)
- moved D198 132.0 mm to (92.8, 182.1)
- moved D199 132.0 mm to (99.3, 182.1)
- moved D200 132.0 mm to (109.0, 182.1)
- moved D201 132.0 mm to (118.8, 182.1)
- moved D202 132.0 mm to (76.5, 182.1)
- moved D203 132.0 mm to (79.8, 182.1)
- moved D204 132.0 mm to (86.3, 182.1)
- moved D205 132.0 mm to (89.5, 182.1)
- moved D206 132.0 mm to (96.0, 182.1)
- moved D207 132.0 mm to (102.5, 182.1)
- moved D208 132.0 mm to (105.8, 182.1)
- moved D209 132.0 mm to (112.3, 182.1)
- moved D210 132.0 mm to (115.5, 182.1)
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Connections:
- R61 pad 1: Net-(R61-Pad1) -> Net-(J10-Pad2)
- R62 pad 1: Net-(R61-Pad1) -> Net-(J10-Pad2)
- R63 pad 1: Net-(R61-Pad1) -> Net-(J10-Pad2)
- R64 pad 1: Net-(R61-Pad1) -> Net-(J10-Pad2)
- R65 pad 1: Net-(R61-Pad1) -> Net-(J10-Pad2)
- R66 pad 1: Net-(R61-Pad1) -> Net-(J10-Pad2)
- R67 pad 1: Net-(R61-Pad1) -> Net-(J10-Pad2)
- R68 pad 1: Net-(R61-Pad1) -> Net-(J10-Pad2)
- R69 pad 1: Net-(R61-Pad1) -> Net-(J10-Pad2)
- R70 pad 1: Net-(R61-Pad1) -> Net-(J10-Pad2)
- R71 pad 1: Net-(R61-Pad1) -> Net-(J10-Pad2)
- R72 pad 1: Net-(R61-Pad1) -> Net-(J10-Pad2)
- R73 pad 1: Net-(R76-Pad1) -> Net-(J17-Pad2)
- R74 pad 1: Net-(R76-Pad1) -> Net-(J17-Pad2)
- R75 pad 1: Net-(R76-Pad1) -> Net-(J17-Pad2)
- R76 pad 1: Net-(R76-Pad1) -> Net-(J17-Pad2)
- R77 pad 1: Net-(R76-Pad1) -> Net-(J17-Pad2)
- R78 pad 1: Net-(R76-Pad1) -> Net-(J17-Pad2)
- R79 pad 1: Net-(R82-Pad1) -> Net-(J19-Pad2)
- R80 pad 1: Net-(R82-Pad1) -> Net-(J19-Pad2)
- R81 pad 1: Net-(R82-Pad1) -> Net-(J19-Pad2)
- R82 pad 1: Net-(R82-Pad1) -> Net-(J19-Pad2)
- R83 pad 1: Net-(R82-Pad1) -> Net-(J19-Pad2)
- R84 pad 1: Net-(R82-Pad1) -> Net-(J19-Pad2)
- R85 pad 1: Net-(R85-Pad1) -> Net-(J20-Pad2)
- R86 pad 1: Net-(R85-Pad1) -> Net-(J20-Pad2)
- R87 pad 1: Net-(R85-Pad1) -> Net-(J20-Pad2)
- R88 pad 1: Net-(R85-Pad1) -> Net-(J20-Pad2)
- R89 pad 1: Net-(R85-Pad1) -> Net-(J20-Pad2)
- R90 pad 1: Net-(R85-Pad1) -> Net-(J20-Pad2)
- R91 pad 1: Net-(R91-Pad1) -> Net-(J21-Pad2)
- R92 pad 1: Net-(R91-Pad1) -> Net-(J21-Pad2)
- R93 pad 1: Net-(R91-Pad1) -> Net-(J21-Pad2)
- R94 pad 1: Net-(R91-Pad1) -> Net-(J21-Pad2)
- R95 pad 1: Net-(R91-Pad1) -> Net-(J21-Pad2)
- R96 pad 1: Net-(R91-Pad1) -> Net-(J21-Pad2)
Routing:
- net Net-(R61-Pad1): track 175.8 -> 0.00 mm
- net Net-(J10-Pad2): track 0.00 -> 175.8 mm
- net Net-(J17-Pad2): track 0.00 -> 41.5 mm
- net Net-(J19-Pad2): track 0.00 -> 41.5 mm
- net Net-(R85-Pad1): track 41.5 -> 0.00 mm
- net Net-(J20-Pad2): track 0.00 -> 41.5 mm
- net Net-(R76-Pad1): track 41.5 -> 0.00 mm
- net Net-(R82-Pad1): track 41.5 -> 0.00 mm
- net Net-(J21-Pad2): track 0.00 -> 41.5 mm
- net Net-(R91-Pad1): track 41.5 -> 0.00 mm
Other:
- board size 175 x 100 mm -> 175 x 151 mm

Commit message: v1.13
Yet more schematic changes
Parts:
- moved R72 0.17 mm to (127.7, 203.9)
- moved R66 0.17 mm to (130.0, 202.6)
- moved D162 0.15 mm to (125.1, 210.1)
- moved D177 0.15 mm to (125.1, 202.7)
- moved D176 0.15 mm to (128.2, 210.1)
- moved D179 0.10 mm to (134.8, 202.8)
- moved D5 0.10 mm to (32.6, 182.5)
- moved R65 0.10 mm to (132.2, 204.1)
Connections:
- R79 pad 1: Net-(J19-Pad2) -> Net-(R79-Pad1)
- R80 pad 1: Net-(J19-Pad2) -> Net-(R79-Pad1)
- R81 pad 1: Net-(J19-Pad2) -> Net-(R79-Pad1)
- R82 pad 1: Net-(J19-Pad2) -> Net-(R79-Pad1)
- R83 pad 1: Net-(J19-Pad2) -> Net-(R79-Pad1)
- R84 pad 1: Net-(J19-Pad2) -> Net-(R79-Pad1)
- R85 pad 1: Net-(J20-Pad2) -> Net-(R85-Pad1)
- R86 pad 1: Net-(J20-Pad2) -> Net-(R85-Pad1)
- R87 pad 1: Net-(J20-Pad2) -> Net-(R85-Pad1)
- R88 pad 1: Net-(J20-Pad2) -> Net-(R85-Pad1)
- R89 pad 1: Net-(J20-Pad2) -> Net-(R85-Pad1)
- R90 pad 1: Net-(J20-Pad2) -> Net-(R85-Pad1)
- REF** pad 1: Net-(R91-Pad1) -> Net-(J21-Pad2)
- REF** pad 1: Net-(R61-Pad1) -> Net-(J10-Pad2)
- REF** pad 1: Net-(R76-Pad1) -> Net-(J17-Pad2)
- REF** pad 1: Net-(R82-Pad1) -> Net-(R79-Pad1)
Routing:
- net Net-(R79-Pad1): track 0.00 -> 41.5 mm
- net Net-(J19-Pad2): track 41.5 -> 0.00 mm
- net Net-(R85-Pad1): track 0.00 -> 41.5 mm
- net Net-(J20-Pad2): track 41.5 -> 0.00 mm
- net Net-(D161-Pad2): track 11.8 -> 12.4 mm

Commit message: v1.14
Control board pcb in the works
Parts:
- added A1: LM2596 DC-DC Buck, afootprints:LM2596 Buck Converter, B.Cu at (84.9, 116.1)
- added A2: LM2596 DC-DC Buck, afootprints:LM2596 Buck Converter, B.Cu at (127.9, 116.1)
- added A3: LM2596 DC-DC Buck, afootprints:LM2596 Buck Converter, B.Cu at (63.4, 116.1)
- added A4: LM2596 DC-DC Buck, afootprints:LM2596 Buck Converter, B.Cu at (106.4, 116.1)
- added A5: Arduino_Nano_v3.x, afootprints:ArduinoNano, F.Cu at (139.4, 117.0)
- added C1: 330uF, Capacitor_THT:C_Radial_D8.0mm_H11.5mm_P3.50mm, B.Cu at (181.5, 108.2)
- added C11: 10uF, Capacitor_THT:C_Radial_D4.0mm_H7.0mm_P1.50mm, F.Cu at (270.0, 154.0)
- added C2: 330uF, Capacitor_THT:C_Radial_D8.0mm_H11.5mm_P3.50mm, B.Cu at (187.2, 117.2)
- added C3: 0.1uF 50V, Capacitor_THT:C_Disc_D7.5mm_W5.0mm_P5.00mm, F.Cu at (281.5, 150.5)
- added C4: 47uF 50V, Capacitor_THT:C_Radial_D5.0mm_H11.0mm_P2.00mm, F.Cu at (250.0, 151.0)
- added D241: 1N4739A, Diode_THT:D_DO-41_SOD81_P10.16mm_Horizontal, F.Cu at (281.9, 159.5)
- added D245: 1N47xxA, Diode_THT:D_DO-41_SOD81_P10.16mm_Horizontal, F.Cu at (314.5, 84.8)
- added D246: 1N4007, Diode_THT:D_DO-41_SOD81_P10.16mm_Horizontal, F.Cu at (252.9, 159.5)
- added D247: 5KP16A, Diode_THT:D_P600_R-6_P20.00mm_Horizontal, F.Cu at (184.0, 157.0)
- added D248: 1N4007, Diode_THT:D_DO-41_SOD81_P10.16mm_Horizontal, F.Cu at (243.9, 165.5)
- added D249: 1N4733A, Diode_THT:D_DO-41_SOD81_P10.16mm_Horizontal, F.Cu at (314.5, 80.6)
- added D250: 1N4733A, Diode_THT:D_DO-41_SOD81_P10.16mm_Horizontal, F.Cu at (225.9, 148.5)
- added D251: 1N4746A, Diode_THT:D_DO-41_SOD81_P10.16mm_Horizontal, F.Cu at (314.5, 76.3)
- added D252: 1N4739A, Diode_THT:D_DO-41_SOD81_P10.16mm_Horizontal, F.Cu at (225.9, 152.8)
- added F1: 10A, afootprints:Univ_AUTO_Fuse, F.Cu at (176.8, 159.0)
- added J11: Letter Terminal, TerminalBlock_Phoenix:TerminalBlock_Phoenix_PT-1,5-3-5.0-H_1x03_P5.00mm_Horizontal, B.Cu at (134.0, 157.5)
- added J12: Letter Terminal, TerminalBlock_Phoenix:TerminalBlock_Phoenix_PT-1,5-3-5.0-H_1x03_P5.00mm_Horizontal, F.Cu at (119.0, 117.5)
- added J14: Power Port Terminal, Connector_PinHeader_2.54mm:PinHeader_2x04_P2.54mm_Vertical, F.Cu at (70.5, 157.5)
- added J15: Raptor Term, TerminalBlock_Phoenix:TerminalBlock_Phoenix_PT-1,5-3-5.0-H_1x03_P5.00mm_Horizontal, F.Cu at (94.5, 102.5)
- added J16: Serial Terminal, TerminalBlock_Phoenix:TerminalBlock_Phoenix_PT-1,5-2-5.0-H_1x02_P5.00mm_Horizontal, B.Cu at (161.5, 122.0)
- added J18: Turn Signal Term., TerminalBlock_Phoenix:TerminalBlock_Phoenix_PT-1,5-2-5.0-H_1x02_P5.00mm_Horizontal, B.Cu at (161.5, 132.0)
- added J22: Raptor Term, TerminalBlock_Phoenix:TerminalBlock_Phoenix_PT-1,5-3-5.0-H_1x03_P5.00mm_Horizontal, F.Cu at (119.0, 132.5)
- added J23: Raptor Term, TerminalBlock_Phoenix:TerminalBlock_Phoenix_PT-1,5-3-5.0-H_1x03_P5.00mm_Horizontal, B.Cu at (134.0, 112.5)
- added J24: Raptor Term, TerminalBlock_Phoenix:TerminalBlock_Phoenix_PT-1,5-3-5.0-H_1x03_P5.00mm_Horizontal, B.Cu at (134.0, 142.5)
- added J25: Turn Signal Term., TerminalBlock_Phoenix:TerminalBlock_Phoenix_PT-1,5-2-5.0-H_1x02_P5.00mm_Horizontal, B.Cu at (161.5, 142.0)
- added J4: Letter Terminal, TerminalBlock_Phoenix:TerminalBlock_Phoenix_PT-1,5-3-5.0-H_1x03_P5.00mm_Horizontal, B.Cu at (134.0, 127.5)
- added J5: Letter Terminal, TerminalBlock_Phoenix:TerminalBlock_Phoenix_PT-1,5-3-5.0-H_1x03_P5.00mm_Horizontal, F.Cu at (94.5, 147.5)
- added J6: Letter Terminal, TerminalBlock_Phoenix:TerminalBlock_Phoenix_PT-1,5-3-5.0-H_1x03_P5.00mm_Horizontal, F.Cu at (119.0, 147.5)
- added J7: Letter Terminal, TerminalBlock_Phoenix:TerminalBlock_Phoenix_PT-1,5-3-5.0-H_1x03_P5.00mm_Horizontal, F.Cu at (119.0, 102.5)
- added Q1: IRLR7843, afootprints:IRLR7843, F.Cu at (381.6, 33.9)
- added Q10: IRLR7843, afootprints:IRLR7843, F.Cu at (323.1, 99.8)
- added Q11: IRLR7843, afootprints:IRLR7843, F.Cu at (416.7, 22.9)
- added Q12: 2N3904, afootprints:2N3904SMD, F.Cu at (292.5, 80.9)
- added Q13: IRLR7843, afootprints:IRLR7843, F.Cu at (334.7, 83.7)
- added Q14: IRLR7843, afootprints:IRLR7843, F.Cu at (350.6, 63.7)
- added Q15: IRLR7843, afootprints:IRLR7843, F.Cu at (367.7, 42.4)
- added Q16: 2N3904, afootprints:2N3904SMD, F.Cu at (376.6, 75.8)
- added Q17: IRLR7843, afootprints:IRLR7843, F.Cu at (362.8, 58.5)
- added Q18: IRLR7843, afootprints:IRLR7843, F.Cu at (367.7, 50.5)
- added Q19: IRLR7843, afootprints:IRLR7843, F.Cu at (393.8, 30.9)
- added Q2: IRLR7843, afootprints:IRLR7843, F.Cu at (310.9, 112.6)
- added Q20: 2N3904, afootprints:2N3904SMD, F.Cu at (410.0, 43.2)
- added Q21: IRLR7843, afootprints:IRLR7843, F.Cu at (392.4, 22.9)
- added Q22: IRLR7843, afootprints:IRLR7843, F.Cu at (302.1, 60.0)
- added Q23: IRLR7843, afootprints:IRLR7843, F.Cu at (332.9, 91.8)
- added Q24: 2N3904, afootprints:2N3904SMD, F.Cu at (415.6, 39.2)
- added Q25: IRLR7843, afootprints:IRLR7843, F.Cu at (392.0, 42.0)
- added Q26: IRLR7843, afootprints:IRLR7843, F.Cu at (350.6, 55.6)
- added Q27: IRLR7843, afootprints:IRLR7843, F.Cu at (379.8, 42.4)
- added Q28: IRLR7843, afootprints:IRLR7843, F.Cu at (320.8, 91.0)
- added Q29: IRLR7843, afootprints:IRLR7843, F.Cu at (294.0, 60.0)
- added Q3: IRLR7843, afootprints:IRLR7843, F.Cu at (379.8, 50.5)
- added Q30: IRLR7843, afootprints:IRLR7843, F.Cu at (334.7, 75.7)
- added Q31: IRLR7843, afootprints:IRLR7843, F.Cu at (374.9, 58.5)
- added Q32: IRLR7843, Package_TO_SOT_THT:TO-220-3_Vertical, B.Cu at (170.4, 109.0)
- added Q33: IRLR7843, afootprints:IRLR7843, F.Cu at (404.6, 22.9)
- added Q34: 2N3904, afootprints:2N3904SMD, F.Cu at (432.7, 21.1)
- added Q35: IRLR7843, afootprints:IRLR7843, F.Cu at (285.9, 60.0)
- added Q36: IRF4905, Package_TO_SOT_THT:TO-220-3_Vertical, B.Cu at (164.9, 104.0)
- added Q37: BC327, Package_TO_SOT_THT:TO-92_Inline, F.Cu at (269.7, 164.9)
- added Q38: BC337, Package_TO_SOT_THT:TO-92_Inline, F.Cu at (268.7, 146.4)
- added Q39: IRF4905, Package_TO_SOT_THT:TO-220-3_Vertical, F.Cu at (246.5, 141.9)
- added Q4: 2N3904, afootprints:2N3904SMD, F.Cu at (292.5, 76.4)
- added Q5: IRLR7843, afootprints:IRLR7843, F.Cu at (323.1, 107.9)
- added Q6: IRLR7843, afootprints:IRLR7843, F.Cu at (310.9, 104.6)
- added Q7: IRLR7843, afootprints:IRLR7843, F.Cu at (362.8, 66.6)
- added Q8: 2N3904, afootprints:2N3904SMD, F.Cu at (403.4, 49.2)
- added Q9: IRLR7843, afootprints:IRLR7843, F.Cu at (335.2, 99.8)
- added R100: 10K, afootprints:1206 R, F.Cu at (365.7, 84.3)
- added R101: 10K, afootprints:1206 R, F.Cu at (397.9, 53.5)
- added R102: 1K, afootprints:1206 R, F.Cu at (339.4, 112.3)
- added R103: 10K, afootprints:1206 R, F.Cu at (352.6, 99.5)
- added R104: 10K, afootprints:1206 R, F.Cu at (398.1, 48.5)
- added R105: 10K, afootprints:1206 R, F.Cu at (381.6, 71.1)
- added R106: 1K, afootprints:1206 R, F.Cu at (350.3, 93.4)
- added R107: 10K, afootprints:1206 R, F.Cu at (381.6, 68.0)
- added R108: 10K, afootprints:1206 R, F.Cu at (304.9, 118.2)
- added R109: 10K, afootprints:1206 R, F.Cu at (365.7, 81.2)
- added R110: 1K, afootprints:1206 R, F.Cu at (365.7, 75.1)
- added R111: 10K, afootprints:1206 R, F.Cu at (388.2, 59.2)
- added R112: 10K, afootprints:1206 R, F.Cu at (387.2, 65.0)
- added R113: 10K, afootprints:1206 R, F.Cu at (392.3, 53.5)
- added R114: 1K, afootprints:1206 R, F.Cu at (352.6, 96.4)
- added R115: 10K, afootprints:THTresistor, F.Cu at (298.2, 170.7)
- added R117: 10K, afootprints:1206 R, F.Cu at (360.1, 86.3)
- added R118: 10K, afootprints:1206 R, F.Cu at (365.7, 78.2)
- added R121: 10K, afootprints:1206 R, F.Cu at (418.2, 29.9)
- added R122: 1K, afootprints:1206 R, F.Cu at (340.4, 106.2)
- added R125: 10K, afootprints:1206 R, F.Cu at (381.6, 65.0)
- added R126: 10K, afootprints:1206 R, F.Cu at (310.5, 118.2)
- added R130: 10K, afootprints:1206 R, F.Cu at (393.8, 59.6)
- added R131: 1K, afootprints:1206 R, F.Cu at (371.3, 75.1)
- added R132: 1K, afootprints:1206 R, F.Cu at (410.3, 39.5)
- added R133: 10K, afootprints:1206 R, F.Cu at (412.6, 28.4)
- added R134: 10K, afootprints:1206 R, F.Cu at (371.3, 78.2)
- added R135: 10K, afootprints:1206 R, F.Cu at (393.8, 56.5)
- added R136: 10K, afootprints:1206 R, F.Cu at (412.6, 31.5)
- added R137: 10K, afootprints:1206 R, F.Cu at (412.6, 34.5)
- added R138: 1K, afootprints:1206 R, F.Cu at (340.4, 109.3)
- added R139: 1K, afootprints:1206 R, F.Cu at (365.7, 87.3)
- added R140: 3.3K, afootprints:THTresistor, F.Cu at (293.7, 153.5)
- added R141: 3.3K, afootprints:THTresistor, F.Cu at (308.0, 155.5)
- added R142: 1.5K, afootprints:THTresistor, F.Cu at (310.3, 158.6)
- added R143: 1.5K, afootprints:THTresistor, F.Cu at (298.2, 167.5)
- added R145: 10K, afootprints:THTresistor, F.Cu at (273.2, 142.0)
- added R97: 10K, afootprints:1206 R, F.Cu at (346.0, 106.2)
- added R98: 1K, afootprints:1206 R, F.Cu at (355.9, 92.1)
- added R99: 10K, afootprints:1206 R, F.Cu at (398.8, 45.4)
- added U5: L7805, afootprints:L7805, F.Cu at (159.2, 109.0)
Routing:
- net (no net): track 0.00 -> 36.9 mm
Other:
- board size 175 x 151 mm -> 175 x 164 mm
