File: Toyota Satoshi Emblem/Toyota Satoshi Emblem.kicad_pcb (KiCad board)
At the start: 2 copper layers, 175 x 164 mm, 480 parts, among them J11 Letter Terminal, J12 Letter Terminal, J14 Power Port Terminal, J15 Raptor Term, J16 Serial Terminal, J18 Turn Signal Term., J22 Raptor Term, J23 Raptor Term, J24 Raptor Term, J25 Turn Signal Term., J4 Letter Terminal, J5 Letter Terminal, J6 Letter Terminal, J7 Letter Terminal, Q1 IRLR7843, Q10 IRLR7843, Q11 IRLR7843, Q12 2N3904, Q13 IRLR7843, Q14 IRLR7843, Q15 IRLR7843, Q16 2N3904, Q17 IRLR7843, Q18 IRLR7843, Q19 IRLR7843, Q2 IRLR7843, Q20 2N3904, Q21 IRLR7843, Q22 IRLR7843, Q23 IRLR7843, Q24 2N3904, Q25 IRLR7843, Q26 IRLR7843, Q27 IRLR7843, Q28 IRLR7843, Q29 IRLR7843, Q3 IRLR7843, Q30 IRLR7843, Q31 IRLR7843, Q32 IRLR7843, Q33 IRLR7843, Q34 2N3904, Q35 IRLR7843, Q36 IRF4905, Q37 BC327, Q38 BC337, Q39 IRF4905, Q4 2N3904, Q5 IRLR7843, Q6 IRLR7843, Q7 IRLR7843, Q8 2N3904, Q9 IRLR7843, U5 L7805

Commit message: v1.15
Power sector of PCB mostly completed
Parts:
- added REF**: MountingHole_2.5mm_Pad_TopBottom, MountingHole:MountingHole_2.5mm_Pad_TopBottom, F.Cu at (187.8, 103.2)
- added REF**: MountingHole_3.5mm, MountingHole:MountingHole_3.5mm, F.Cu at (172.5, 128.0)
- added REF**: MountingHole_2.5mm_Pad_TopBottom, MountingHole:MountingHole_2.5mm_Pad_TopBottom, F.Cu at (187.8, 156.8)
- D247: footprint Diode_THT:D_P600_R-6_P20.00mm_Horizontal -> afootprints:5KP16A; moved to B.Cu
- D252: value 1N4739A -> 1N4738A
- Q32: footprint Package_TO_SOT_THT:TO-220-3_Vertical -> afootprints:IRLR7843; moved to F.Cu
- Q36: footprint Package_TO_SOT_THT:TO-220-3_Vertical -> afootprints:IRF4905; moved to F.Cu
- Q39: footprint Package_TO_SOT_THT:TO-220-3_Vertical -> afootprints:IRF4905
- R115: footprint afootprints:THTresistor -> afootprints:1206 R
- R140, R141: value 3.3K -> 1K; footprint afootprints:THTresistor -> afootprints:1206 R; moved to B.Cu
- R142, R143: value 1.5K -> 1K; footprint afootprints:THTresistor -> afootprints:1206 R; moved to B.Cu
- R145: footprint afootprints:THTresistor -> afootprints:1206 R; moved to B.Cu
- moved Q1 340.5 mm to (42.7, 1.00)
- moved Q17 340.5 mm to (23.9, 25.6)
- moved Q28 340.5 mm to (-18.1, 58.1)
- moved Q7 340.5 mm to (23.9, 33.6)
- moved R100 340.5 mm to (26.8, 51.4)
- moved R105 340.5 mm to (42.7, 38.1)
- moved R107 340.5 mm to (42.7, 35.1)
- moved R109 340.5 mm to (26.8, 48.3)
- moved R110 340.5 mm to (26.8, 42.2)
- moved R118 340.5 mm to (26.8, 45.2)
- moved R122 340.5 mm to (1.53, 73.3)
- moved R125 340.5 mm to (42.7, 32.0)
- moved Q10 340.5 mm to (-15.8, 66.9)
- moved Q11 340.5 mm to (77.8, -10.1)
- moved Q12 340.5 mm to (-46.4, 48.0)
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Routing:
- net GND: track 0.00 -> 177.6 mm
- net Net-(C3-Pad1): track 0.00 -> 120.5 mm
- net +5V: track 0.00 -> 74.0 mm
- net Net-(D247-Pad1): track 0.00 -> 72.8 mm
- net Net-(D246-Pad1): track 0.00 -> 44.9 mm
- net +12V: track 0.00 -> 39.1 mm
- net (no net): track 36.9 -> 0.00 mm
- net Net-(A5-Pad2): track 0.00 -> 36.2 mm
- net Net-(A5-Pad24): track 0.00 -> 31.7 mm
- net Net-(D241-Pad2): track 0.00 -> 23.9 mm
- net Net-(A5-Pad1): track 0.00 -> 23.2 mm
- net Net-(A5-Pad25): track 0.00 -> 22.9 mm
- net Net-(D248-Pad2): track 0.00 -> 21.4 mm
- net /POWER: track 0.00 -> 19.5 mm
- net Net-(Q38-Pad2): track 0.00 -> 11.5 mm
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Other:
- board text added: "low"

Commit message: v1.16
Realized critical errors were made when choosing trace widths. Control PCB will need to be redesigned
Parts:
- added REF**: MountingHole_3.5mm, MountingHole:MountingHole_3.5mm, F.Cu at (53.0, 156.0)
- added REF**: MountingHole_3.5mm, MountingHole:MountingHole_3.5mm, F.Cu at (53.0, 104.0)
- added REF**: MountingHole_3.5mm, MountingHole:MountingHole_3.5mm, F.Cu at (53.0, 130.0)
- C1, C2: value 330uF -> 470uF
- J14: value Power Port Terminal -> Power Port Term.
- J15, J22, Q25, Q26, Q27, Q28, Q29, Q30, Q31, Q32, Q33, Q34, Q35, R130, R132, R133: moved to B.Cu
- J4: moved to F.Cu
- moved Q1 261.2 mm to (302.2, 31.3)
- moved Q11 261.2 mm to (337.3, 20.2)
- moved Q17 261.2 mm to (283.4, 55.9)
- moved Q20 261.2 mm to (330.5, 40.6)
- moved Q22 261.2 mm to (222.6, 57.4)
- moved Q7 261.2 mm to (283.4, 63.9)
- moved R100 261.2 mm to (286.3, 81.6)
- moved R105 261.2 mm to (302.2, 68.4)
- moved R107 261.2 mm to (302.2, 65.4)
- moved R109 261.2 mm to (286.2, 78.6)
- moved R110 261.2 mm to (286.2, 72.5)
- moved R118 261.2 mm to (286.2, 75.5)
- moved R121 261.2 mm to (338.7, 27.3)
- moved R122 261.2 mm to (261.0, 103.6)
- moved R125 261.2 mm to (302.2, 62.3)
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Connections:
- A1 pad 3: GND -> unconnected-(A1-Pad3)
- A2 pad 3: GND -> unconnected-(A2-Pad3)
- A3 pad 3: GND -> unconnected-(A3-Pad3)
- A4 pad 3: GND -> unconnected-(A4-Pad3)
- J14 pad 2: /BUCK_B -> /BUCK_C
- J14 pad 3: +12V -> /BUCK_B
- J14 pad 4: GND -> /BUCK_D
- J14 pad 5: GND -> +12V
- J14 pad 7: /BUCK_D -> GND
- J14 pad 8: /BUCK_C -> GND
Routing:
- net Net-(A5-Pad23): track 0.00 -> 147.8 mm, vias 0 -> 4
- net GND: track 177.6 -> 279.3 mm
- net Net-(A5-Pad19): track 0.00 -> 95.9 mm, vias 0 -> 2
- net /BUCK_D: track 0.00 -> 93.9 mm, vias 0 -> 3
- net Net-(A5-Pad22): track 0.00 -> 87.7 mm, vias 0 -> 2
- net Net-(Q29-Pad2): track 0.00 -> 81.7 mm
- net Net-(J15-Pad1): track 0.00 -> 73.9 mm, vias 0 -> 2
- net Net-(A5-Pad21): track 0.00 -> 69.7 mm
- net Net-(J15-Pad3): track 0.00 -> 62.7 mm, vias 0 -> 2
- net Net-(A5-Pad20): track 0.00 -> 56.0 mm
- net Net-(Q25-Pad2): track 0.00 -> 49.3 mm
- net Net-(J23-Pad3): track 0.00 -> 42.3 mm
- net Net-(J24-Pad3): track 0.00 -> 39.2 mm
- net Net-(J24-Pad1): track 0.00 -> 30.2 mm
- net Net-(J22-Pad3): track 0.00 -> 29.6 mm, vias 0 -> 2
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
Commit message: v1.17
Last push before making some major changes in regards to the processor
Parts:
- removed the REF** at (172.5, 128.0)
- removed the REF** at (53.0, 130.0)
- added REF**: MountingHole_2.5mm_Pad_TopBottom, MountingHole:MountingHole_2.5mm_Pad_TopBottom, F.Cu at (19.2, 156.8)
- added REF**: MountingHole_2.5mm_Pad_TopBottom, MountingHole:MountingHole_2.5mm_Pad_TopBottom, F.Cu at (19.2, 103.2)
- A1, A2, A3, A4, C1, C2, J11, J15, J22, J23, J24: moved to F.Cu
- moved Q2 298.0 mm to (-52.1, 18.7)
- moved R102 298.0 mm to (-23.7, 18.4)
- moved R108 298.0 mm to (-58.2, 24.2)
- moved R126 298.0 mm to (-52.6, 24.2)
- moved J22 97.6 mm to (45.0, 117.5), turned to -90 degrees
- moved J24 91.2 mm to (45.0, 132.5), turned to -90 degrees
- moved C1 90.8 mm to (105.2, 154.5), turned to 0 degrees
- moved J14 85.1 mm to (42.2, 77.3)
- moved Q26 84.3 mm to (19.7, 134.4)
- moved Q27 83.7 mm to (19.7, 141.6)
- moved A4 79.5 mm to (56.0, 150.0)
- moved Q31 78.2 mm to (25.8, 156.4)
- moved C2 76.2 mm to (114.2, 154.5), turned to 0 degrees
- moved Q28 75.1 mm to (91.5, 65.2)
- moved Q32 75.1 mm to (84.0, 65.2)
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Connections:
- A1 pad 3: unconnected-(A1-Pad3) -> GND
- A1 pad 4: GND -> unconnected-(A1-Pad4)
- A2 pad 3: unconnected-(A2-Pad3) -> GND
- A2 pad 4: GND -> unconnected-(A2-Pad4)
- A3 pad 3: unconnected-(A3-Pad3) -> GND
- A3 pad 4: GND -> unconnected-(A3-Pad4)
- A4 pad 3: unconnected-(A4-Pad3) -> GND
- A4 pad 4: GND -> unconnected-(A4-Pad4)
- A5 pad 29: unconnected-(A5-Pad29) -> GND
Routing:
- net +12V: track 65.4 -> 242.6 mm, vias 1 -> 8
- net Net-(A5-Pad23): track 147.8 -> 0.00 mm, vias 4 -> 0
- net Net-(A5-Pad19): track 95.9 -> 0.00 mm, vias 2 -> 0
- net /BUCK_D: track 93.9 -> 0.00 mm, vias 3 -> 0
- net Net-(A5-Pad22): track 87.7 -> 0.00 mm, vias 2 -> 0
- net Net-(Q29-Pad2): track 81.7 -> 0.00 mm
- net Net-(J15-Pad1): track 73.9 -> 0.00 mm, vias 2 -> 0
- net Net-(A5-Pad21): track 69.7 -> 0.00 mm
- net Net-(J15-Pad3): track 62.7 -> 0.00 mm, vias 2 -> 0
- net Net-(D241-Pad2): track 23.9 -> 76.4 mm
- net Net-(Q25-Pad2): track 49.3 -> 0.00 mm
- net Net-(J23-Pad3): track 42.3 -> 0.00 mm
- net GND: track 279.3 -> 319.6 mm
- net Net-(J24-Pad3): track 39.2 -> 0.00 mm
- net Net-(A5-Pad20): track 56.0 -> 17.3 mm
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Other:
- board size 175 x 164 mm -> 175 x 178 mm
- board text removed: "low"

Commit message: v2.1
probably made some improvements
Parts:
- removed A1, A2, A3, A4: LM2596 DC-DC Buck, afootprints:LM2596 Buck Converter
- removed A5: Arduino_Nano_v3.x, afootprints:ArduinoNano
- removed C1, C2: 470uF, Capacitor_THT:C_Radial_D8.0mm_H11.5mm_P3.50mm
- removed C11: 10uF, Capacitor_THT:C_Radial_D4.0mm_H7.0mm_P1.50mm
- removed C3: 0.1uF 50V, Capacitor_THT:C_Disc_D7.5mm_W5.0mm_P5.00mm
- removed C4: 47uF 50V, Capacitor_THT:C_Radial_D5.0mm_H11.0mm_P2.00mm
- removed D241: 1N4739A, Diode_THT:D_DO-41_SOD81_P10.16mm_Horizontal
- removed D245: 1N47xxA, Diode_THT:D_DO-41_SOD81_P10.16mm_Horizontal
- removed D246, D248: 1N4007, Diode_THT:D_DO-41_SOD81_P10.16mm_Horizontal
- removed D247: 5KP16A, afootprints:5KP16A
- removed D249, D250: 1N4733A, Diode_THT:D_DO-41_SOD81_P10.16mm_Horizontal
- removed D251: 1N4746A, Diode_THT:D_DO-41_SOD81_P10.16mm_Horizontal
- removed D252: 1N4738A, Diode_THT:D_DO-41_SOD81_P10.16mm_Horizontal
- removed F1: 10A, afootprints:Univ_AUTO_Fuse
- removed J11, J12, J4, J5, J6, J7: Letter Terminal, TerminalBlock_Phoenix:TerminalBlock_Phoenix_PT-1,5-3-5.0-H_1x03_P5.00mm_Horizontal
- removed J14: Power Port Term., Connector_PinHeader_2.54mm:PinHeader_2x04_P2.54mm_Vertical
- removed J15, J22, J23, J24: Raptor Term, TerminalBlock_Phoenix:TerminalBlock_Phoenix_PT-1,5-3-5.0-H_1x03_P5.00mm_Horizontal
- removed J16: Serial Terminal, TerminalBlock_Phoenix:TerminalBlock_Phoenix_PT-1,5-2-5.0-H_1x02_P5.00mm_Horizontal
- removed J18, J25: Turn Signal Term., TerminalBlock_Phoenix:TerminalBlock_Phoenix_PT-1,5-2-5.0-H_1x02_P5.00mm_Horizontal
- removed Q1, Q10, Q11, Q13, Q14, Q15, Q17, Q18, Q19, Q2, Q21, Q22, Q23, Q25, Q26, Q27, Q28, Q29, Q3, Q30, Q31, Q32, Q33, Q35, Q5, Q6, Q7, Q9: IRLR7843, afootprints:IRLR7843
- removed Q12, Q16, Q20, Q24, Q34, Q4, Q8: 2N3904, afootprints:2N3904SMD
- removed Q36, Q39: IRF4905, afootprints:IRF4905
- removed Q37: BC327, Package_TO_SOT_THT:TO-92_Inline
- removed Q38: BC337, Package_TO_SOT_THT:TO-92_Inline
- removed R100, R101, R103, R104, R105, R107, R108, R109, R111, R112, R113, R115, R117, R118, R121, R125, R126, R130, R133, R134, R135, R136, R137, R145, R97, R99: 10K, afootprints:1206 R
- removed R102, R106, R110, R114, R122, R131, R132, R138, R139, R140, R141, R142, R143, R98: 1K, afootprints:1206 R
- removed the REF** at (187.8, 103.2)
- removed the REF** at (19.2, 156.8)
- removed the REF** at (24.8, 149.0)
- removed the REF** at (19.2, 103.2)
- removed the REF** at (187.8, 156.8)
- removed the REF** at (24.8, 111.0)
- removed U5: L7805, afootprints:L7805
- added R79: 4.7, afootprints:1206 R, F.Cu at (-62.6, 294.1)
- moved D181 186.8 mm to (-86.8, 298.6)
- moved D182 186.8 mm to (-77.0, 298.6)
- moved D183 186.8 mm to (-67.3, 298.6)
- moved D184 186.8 mm to (-60.8, 298.6)
- moved D185 186.8 mm to (-51.0, 298.6)
- moved D187 186.8 mm to (-83.5, 298.6)
- moved D188 186.8 mm to (-80.3, 298.6)
- moved D189 186.8 mm to (-73.8, 298.6)
- moved D190 186.8 mm to (-70.5, 298.6)
- moved D191 186.8 mm to (-64.0, 298.6)
- moved D192 186.8 mm to (-57.5, 298.6)
- moved D193 186.8 mm to (-54.3, 298.6)
- moved D100 122.1 mm to (173.9, 325.8)
- moved D103 122.1 mm to (159.3, 307.7)
- moved D122 122.1 mm to (158.0, 332.9)
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Routing:
- net GND: track 319.6 -> 0.00 mm
- net +12V: track 242.6 -> 0.00 mm, vias 8 -> 0
- net Net-(C3-Pad1): track 137.1 -> 0.00 mm
- net Net-(D246-Pad1): track 77.0 -> 0.00 mm, vias 1 -> 0
- net Net-(D241-Pad2): track 76.4 -> 0.00 mm
- net Net-(A5-Pad2): track 51.7 -> 0.00 mm
- net +5V: track 45.4 -> 0.00 mm
- net Net-(D247-Pad1): track 43.7 -> 0.00 mm
- net Net-(A5-Pad24): track 41.6 -> 0.00 mm
- net Net-(D248-Pad2): track 33.7 -> 0.00 mm
- net Net-(A5-Pad25): track 30.9 -> 0.00 mm
- net Net-(J18-Pad1): track 24.3 -> 0.00 mm
- net Net-(A5-Pad1): track 23.7 -> 0.00 mm
- net Net-(J18-Pad2): track 19.0 -> 0.00 mm
- net Net-(A5-Pad20): track 17.3 -> 0.00 mm
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Other:
- board size 175 x 178 mm -> 283.5 x 299.1 mm
- board text removed: "7.5V"
- board text removed: "a"
- board text removed: "w"

Commit message: v2.2
Letter T and O are complete
Parts:
- removed D100, D101, D102, D121, D122, D123, D124, D125, D126, D127, D128, D129, D130, D131, D132, D151, D152, D153, D154, D155, D156, D157, D158, D159, D160, D161, D162, D181, D182, D183, D184, D185, D186, D196, D197, D198, D199, D200, D201, D211, D212, D213, D214, D215, D216, D226, D227, D228, D229, D230, D231, D61, D62, D63, D64, D65, D66, D67, D68, D69, D70, D71, D72, D91, D92, D93, D94, D95, D96, D97, D98, D99: WLED, afootprints:5730 LED W
- removed D103, D104, D105, D106, D107, D108, D109, D110, D111, D112, D113, D114, D115, D116, D117, D118, D119, D120, D133, D134, D135, D136, D137, D138, D139, D140, D141, D142, D143, D144, D145, D146, D147, D148, D149, D150, D163, D164, D165, D166, D167, D168, D169, D170, D171, D172, D173, D174, D175, D176, D177, D178, D179, D180, D187, D188, D189, D190, D191, D192, D193, D194, D195, D202, D203, D204, D205, D206, D207, D208, D209, D210, D217, D218, D219, D220, D221, D222, D223, D224, D225, D232, D233, D234, D235, D236, D237, D238, D239, D240, D49, D50, D51, D52, D53, D54, D55, D56, D57, D58, D59, D60, D73, D74, D75, D76, D77, D78, D79, D80, D81, D82, D83, D84, D85, D86, D87, D88, D89, D90: ALED, afootprints:5730 LED A
- removed R25, R26, R28, R29, R30, R31, R32, R33, R34, R35, R36, R37, R38, R40, R41, R42, R43, R44, R45, R46, R47, R48, R49, R50, R52, R53, R54, R55, R56, R57, R58, R59, R60, R61, R62, R64, R65, R66, R67, R68, R69, R70, R71, R72, R73, R74, R75, R76, R77, R78, R79 (x2), R80, R81, R82, R83, R84, R85, R86, R87, R88, R89, R90, R91, R92, R93, R94, R95, R96: 4.7, afootprints:1206 R
- removed R27, R39, R51, R63: 4,7, afootprints:1206 R
- removed REF** (x12): Pad 2, afootprints:Pad 2
- removed REF** (x18): Pad 1, afootprints:Pad 1
- added P: Pad 1, afootprints:Pad 1, F.Cu at (75.0, 56.5)
- added P: Pad 1, afootprints:Pad 1, F.Cu at (79.5, 55.3)
- added P: Pad 1, afootprints:Pad 1, F.Cu at (48.6, 51.7)
- added P: Pad 1, afootprints:Pad 1, F.Cu at (84.5, 54.6)
- added P: Pad 1, afootprints:Pad 1, F.Cu at (48.6, 55.5)
- added wht: Pad 1, afootprints:Pad 1, F.Cu at (48.6, 47.9)
- D25, D26, D27, D28, D29, D30: value ALED -> WLED; footprint afootprints:5730 LED A -> afootprints:5730 LED W
- D37, D38, D39, D40, D41, D42: value WLED -> ALED; footprint afootprints:5730 LED W -> afootprints:5730 LED A
- moved R21 343.5 mm to (119.2, 36.0), turned to -145 degrees
- moved D38 343.1 mm to (85.0, 35.8), turned to -44.1 degrees
- moved R14 341.9 mm to (97.0, 27.8), turned to 105 degrees
- moved D40 340.6 mm to (106.0, 29.6), turned to -102.9 degrees
- moved R15 339.0 mm to (115.8, 42.2), turned to -55 degrees
- moved R20 332.6 mm to (91.2, 29.2), turned to -65 degrees
- moved D39 329.2 mm to (94.7, 29.9), turned to -73.5 degrees
- moved D37 329.1 mm to (79.3, 47.5), turned to -9.7 degrees
- moved R16 317.3 mm to (123.9, 60.3), turned to -115 degrees
- moved D48 316.8 mm to (80.4, 59.5), turned to 21.9 degrees
- moved D41 316.8 mm to (116.0, 34.8), turned to -132.3 degrees
- moved D36 315.8 mm to (83.1, 64.5), turned to 36.6 degrees
- moved R22 314.8 mm to (124.5, 52.8)
- moved D35 302.9 mm to (92.0, 71.6), turned to 66 degrees
- moved D42 302.4 mm to (122.1, 44.3), turned to -161.7 degrees
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Connections:
- D15 pad 2: Net-(D14-Pad1) -> Net-(D15-Pad2)
- D16 pad 1: Net-(D16-Pad1) -> Net-(D14-Pad1)
- D16 pad 2: Net-(D16-Pad2) -> Net-(D15-Pad1)
- D17 pad 2: Net-(D16-Pad1) -> Net-(D17-Pad2)
- D18 pad 1: Net-(D15-Pad1) -> Net-(D14-Pad1)
- D20 pad 1: Net-(D20-Pad1) -> Net-(D14-Pad1)
- D21 pad 1: Net-(D15-Pad1) -> Net-(D21-Pad1)
- D21 pad 2: Net-(D20-Pad1) -> Net-(D21-Pad2)
- D22 pad 1: Net-(D22-Pad1) -> Net-(D14-Pad1)
- D22 pad 2: Net-(D22-Pad2) -> Net-(D21-Pad1)
- D23 pad 2: Net-(D22-Pad1) -> Net-(D23-Pad2)
- D24 pad 1: Net-(D15-Pad1) -> Net-(D14-Pad1)
- D26 pad 1: Net-(D26-Pad1) -> Net-(D25-Pad2)
- D26 pad 2: Net-(D25-Pad1) -> Net-(D26-Pad2)
- D27 pad 1: Net-(D15-Pad1) -> Net-(D25-Pad1)
- D27 pad 2: Net-(D26-Pad1) -> Net-(D27-Pad2)
- D28 pad 1: Net-(D28-Pad1) -> Net-(D27-Pad2)
- D29 pad 1: Net-(D29-Pad1) -> Net-(D25-Pad1)
- D29 pad 2: Net-(D28-Pad1) -> Net-(D29-Pad2)
- D30 pad 1: Net-(D15-Pad1) -> Net-(D29-Pad2)
- D30 pad 2: Net-(D29-Pad1) -> Net-(D30-Pad2)
- D31 pad 1: Net-(D31-Pad1) -> Net-(D25-Pad1)
- D33 pad 1: Net-(D31-Pad1) -> Net-(D25-Pad1)
- D35 pad 1: Net-(D31-Pad1) -> Net-(D25-Pad1)
- D37 pad 1: Net-(D31-Pad1) -> Net-(D37-Pad1)
- D38 pad 1: Net-(D37-Pad2) -> Net-(D38-Pad1)
- D38 pad 2: Net-(D38-Pad2) -> Net-(D37-Pad1)
- D39 pad 1: Net-(D31-Pad1) -> Net-(D39-Pad1)
- D40 pad 1: Net-(D39-Pad2) -> Net-(D38-Pad1)
- D40 pad 2: Net-(D40-Pad2) -> Net-(D39-Pad1)
- D41 pad 1: Net-(D31-Pad1) -> Net-(D41-Pad1)
- D42 pad 1: Net-(D41-Pad2) -> Net-(D38-Pad1)
- D42 pad 2: Net-(D42-Pad2) -> Net-(D41-Pad1)
- D44 pad 1: Net-(D44-Pad1) -> Net-(D38-Pad1)
- D45 pad 2: Net-(D44-Pad1) -> Net-(D45-Pad2)
- D46 pad 1: Net-(D46-Pad1) -> Net-(D38-Pad1)
- D46 pad 2: Net-(D46-Pad2) -> Net-(D45-Pad1)
- D47 pad 2: Net-(D46-Pad1) -> Net-(D47-Pad2)
- D48 pad 1: Net-(D45-Pad1) -> Net-(D38-Pad1)
- R10 pad 2: Net-(D22-Pad2) -> Net-(D19-Pad2)
- R11 pad 2: Net-(D25-Pad2) -> Net-(D21-Pad2)
- R12 pad 2: Net-(D28-Pad2) -> Net-(D23-Pad2)
- R13 pad 2: Net-(D32-Pad2) -> Net-(D26-Pad2)
- R14 pad 2: Net-(D34-Pad2) -> Net-(D28-Pad2)
- R15 pad 2: Net-(D36-Pad2) -> Net-(D30-Pad2)
- R16 pad 2: Net-(D38-Pad2) -> Net-(D32-Pad2)
- R17 pad 2: Net-(D40-Pad2) -> Net-(D34-Pad2)
- R18 pad 2: Net-(D42-Pad2) -> Net-(D36-Pad2)
- R19 pad 2: Net-(D43-Pad2) -> Net-(D37-Pad2)
- R20 pad 2: Net-(D46-Pad2) -> Net-(D39-Pad2)
- R21 pad 2: Net-(D49-Pad2) -> Net-(D41-Pad2)
- R22 pad 2: Net-(D52-Pad2) -> Net-(D43-Pad2)
- R23 pad 2: Net-(D55-Pad2) -> Net-(D45-Pad2)
- R24 pad 2: Net-(D58-Pad2) -> Net-(D47-Pad2)
- R8 pad 2: Net-(D16-Pad2) -> Net-(D15-Pad2)
- R9 pad 2: Net-(D19-Pad2) -> Net-(D17-Pad2)
Routing:
- net Net-(D38-Pad1): track 0.00 -> 200.9 mm
- net Net-(D25-Pad1): track 3.20 -> 195.9 mm
- net Net-(J3-Pad2): track 184.7 -> 0.00 mm
- net Net-(J10-Pad2): track 175.8 -> 0.00 mm
- net Net-(D135-Pad1): track 162.1 -> 0.00 mm
- net Net-(D61-Pad1): track 161.9 -> 0.00 mm
- net Net-(D45-Pad1): track 162.1 -> 20.8 mm
- net Net-(J9-Pad2): track 136.3 -> 0.00 mm
- net Net-(D121-Pad1): track 127.1 -> 0.00 mm
- net Net-(D31-Pad1): track 127.1 -> 0.00 mm
- net Net-(D75-Pad1): track 124.4 -> 0.00 mm
- net Net-(J8-Pad2): track 122.5 -> 0.00 mm
- net Net-(D105-Pad1): track 109.7 -> 0.00 mm
- net Net-(J1-Pad2): track 175.7 -> 74.4 mm
- net Net-(D14-Pad1): track 12.6 -> 111.5 mm
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Other:
- board size 283.5 x 299.1 mm -> 372.3 x 63 mm
- board text removed: "Daniel Hoefer"

Commit message: v2.3
Letter-board completed w/ silkscreen edits
Parts:
- added D100: WLED, afootprints:5730 LED W, F.Cu at (269.0, 30.9)
- added D101: WLED, afootprints:5730 LED W, F.Cu at (253.6, 27.2)
- added D102: WLED, afootprints:5730 LED W, F.Cu at (253.1, 34.6)
- added D103: WLED, afootprints:5730 LED W, F.Cu at (253.9, 76.0)
- added D104: WLED, afootprints:5730 LED W, F.Cu at (253.6, 70.6)
- added D105: WLED, afootprints:5730 LED W, F.Cu at (249.1, 63.1)
- added D106: WLED, afootprints:5730 LED W, F.Cu at (249.1, 48.1)
- added D107: WLED, afootprints:5730 LED W, F.Cu at (258.0, 63.1)
- added D108: WLED, afootprints:5730 LED W, F.Cu at (258.0, 48.1)
- added D109: ALED, afootprints:5730 LED A, F.Cu at (237.9, 34.6)
- added D110: ALED, afootprints:5730 LED A, F.Cu at (237.9, 27.1)
- added D111: ALED, afootprints:5730 LED A, F.Cu at (268.9, 34.6)
- added D112: ALED, afootprints:5730 LED A, F.Cu at (268.9, 27.1)
- added D113: ALED, afootprints:5730 LED A, F.Cu at (247.8, 30.8)
- added D114: ALED, afootprints:5730 LED A, F.Cu at (259.1, 30.8)
- added D115: ALED, afootprints:5730 LED A, F.Cu at (258.0, 70.6)
- added D116: ALED, afootprints:5730 LED A, F.Cu at (249.1, 70.6)
- added D117: ALED, afootprints:5730 LED A, F.Cu at (249.1, 40.6)
- added D118: ALED, afootprints:5730 LED A, F.Cu at (249.1, 55.6)
- added D119: ALED, afootprints:5730 LED A, F.Cu at (258.0, 40.6)
- added D120: ALED, afootprints:5730 LED A, F.Cu at (258.0, 55.6)
- added D121: WLED, afootprints:5730 LED W, F.Cu at (280.0, 51.4)
- added D122: WLED, afootprints:5730 LED W, F.Cu at (286.0, 36.6)
- added D123: WLED, afootprints:5730 LED W, F.Cu at (274.0, 66.3)
- added D124: WLED, afootprints:5730 LED W, F.Cu at (277.0, 76.0)
- added D125: WLED, afootprints:5730 LED W, F.Cu at (312.1, 51.4)
- added D126: WLED, afootprints:5730 LED W, F.Cu at (306.1, 36.6)
- added D127: WLED, afootprints:5730 LED W, F.Cu at (318.1, 66.2)
- added D128: WLED, afootprints:5730 LED W, F.Cu at (315.0, 76.0)
- added D129: WLED, afootprints:5730 LED W, F.Cu at (289.6, 61.8)
- added D130: WLED, afootprints:5730 LED W, F.Cu at (302.4, 61.8)
- added D131: WLED, afootprints:5730 LED W, F.Cu at (296.0, 34.5)
- added D132: WLED, afootprints:5730 LED W, F.Cu at (296.1, 29.2)
- added D133: ALED, afootprints:5730 LED A, F.Cu at (290.5, 30.5)
- added D134: ALED, afootprints:5730 LED A, F.Cu at (286.7, 47.9)
- added D135: ALED, afootprints:5730 LED A, F.Cu at (271.0, 73.8)
- added D136: ALED, afootprints:5730 LED A, F.Cu at (277.0, 58.8)
- added D137: ALED, afootprints:5730 LED A, F.Cu at (301.5, 30.5)
- added D138: ALED, afootprints:5730 LED A, F.Cu at (305.4, 47.9)
- added D139: ALED, afootprints:5730 LED A, F.Cu at (321.0, 73.6)
- added D140: ALED, afootprints:5730 LED A, F.Cu at (315.1, 58.8)
- added D141: ALED, afootprints:5730 LED A, F.Cu at (281.9, 67.6)
- added D142: ALED, afootprints:5730 LED A, F.Cu at (295.9, 58.5)
- added D143: ALED, afootprints:5730 LED A, F.Cu at (310.1, 67.6)
- added D144: ALED, afootprints:5730 LED A, F.Cu at (295.9, 65.0)
- added D49: WLED, afootprints:5730 LED W, F.Cu at (137.0, 42.6)
- added D50: WLED, afootprints:5730 LED W, F.Cu at (128.4, 29.1)
- added D51: WLED, afootprints:5730 LED W, F.Cu at (148.1, 45.0)
- added D52: WLED, afootprints:5730 LED W, F.Cu at (139.9, 31.3)
- added D53: WLED, afootprints:5730 LED W, F.Cu at (165.9, 42.6)
- added D54: WLED, afootprints:5730 LED W, F.Cu at (174.5, 29.2)
- added D55: WLED, afootprints:5730 LED W, F.Cu at (154.7, 45.0)
- added D56: WLED, afootprints:5730 LED W, F.Cu at (162.8, 31.3)
- added D57: WLED, afootprints:5730 LED W, F.Cu at (146.0, 59.1)
- added D58: WLED, afootprints:5730 LED W, F.Cu at (146.0, 74.2)
- added D59: WLED, afootprints:5730 LED W, F.Cu at (156.5, 59.1)
- added D60: WLED, afootprints:5730 LED W, F.Cu at (156.8, 74.2)
- added D61: ALED, afootprints:5730 LED A, F.Cu at (132.7, 35.8)
- added D62: ALED, afootprints:5730 LED A, F.Cu at (141.3, 49.3)
- added D63: ALED, afootprints:5730 LED A, F.Cu at (133.5, 27.0)
- added D64: ALED, afootprints:5730 LED A, F.Cu at (144.0, 38.2)
- added D65: ALED, afootprints:5730 LED A, F.Cu at (170.2, 35.9)
- added D66: ALED, afootprints:5730 LED A, F.Cu at (161.6, 49.4)
- added D67: ALED, afootprints:5730 LED A, F.Cu at (169.2, 27.0)
- added D68: ALED, afootprints:5730 LED A, F.Cu at (158.8, 38.2)
- added D69: ALED, afootprints:5730 LED A, F.Cu at (151.4, 76.2)
- added D70: ALED, afootprints:5730 LED A, F.Cu at (146.2, 66.7)
- added D71: ALED, afootprints:5730 LED A, F.Cu at (156.5, 66.7)
- added D72: ALED, afootprints:5730 LED A, F.Cu at (151.4, 57.2)
- added D73: WLED, afootprints:5730 LED W, F.Cu at (179.8, 51.3)
- added D74: WLED, afootprints:5730 LED W, F.Cu at (182.7, 40.4)
- added D75: WLED, afootprints:5730 LED W, F.Cu at (190.6, 32.3)
- added D76: WLED, afootprints:5730 LED W, F.Cu at (201.4, 29.1)
- added D77: WLED, afootprints:5730 LED W, F.Cu at (212.4, 31.6)
- added D78: WLED, afootprints:5730 LED W, F.Cu at (220.8, 39.2)
- added D79: WLED, afootprints:5730 LED W, F.Cu at (224.3, 49.9)
- added D80: WLED, afootprints:5730 LED W, F.Cu at (221.0, 62.9)
- added D81: WLED, afootprints:5730 LED W, F.Cu at (214.8, 69.6)
- added D82: WLED, afootprints:5730 LED W, F.Cu at (204.2, 73.5)
- added D83: WLED, afootprints:5730 LED W, F.Cu at (193.0, 71.6)
- added D84: WLED, afootprints:5730 LED W, F.Cu at (184.2, 64.6)
- added D85: ALED, afootprints:5730 LED A, F.Cu at (180.4, 47.6)
- added D86: ALED, afootprints:5730 LED A, F.Cu at (186.1, 35.8)
- added D87: ALED, afootprints:5730 LED A, F.Cu at (195.8, 30.0)
- added D88: ALED, afootprints:5730 LED A, F.Cu at (207.1, 29.6)
- added D89: ALED, afootprints:5730 LED A, F.Cu at (217.1, 34.9)
- added D90: ALED, afootprints:5730 LED A, F.Cu at (223.2, 44.3)
- added D91: ALED, afootprints:5730 LED A, F.Cu at (223.9, 55.6)
- added D92: ALED, afootprints:5730 LED A, F.Cu at (219.0, 65.8)
- added D93: ALED, afootprints:5730 LED A, F.Cu at (209.7, 72.2)
- added D94: ALED, afootprints:5730 LED A, F.Cu at (198.5, 73.3)
- added D95: ALED, afootprints:5730 LED A, F.Cu at (188.2, 68.7)
- added D96: ALED, afootprints:5730 LED A, F.Cu at (181.4, 59.6)
- added D97: WLED, afootprints:5730 LED W, F.Cu at (232.5, 30.9)
- added D98: WLED, afootprints:5730 LED W, F.Cu at (237.9, 30.9)
- added D99: WLED, afootprints:5730 LED W, F.Cu at (274.4, 30.9)
- added P: Pad 1, afootprints:Pad 1, F.Cu at (284.5, 54.3)
- added P: Pad 1, afootprints:Pad 1, F.Cu at (253.5, 51.6)
- added P: Pad 1, afootprints:Pad 1, F.Cu at (281.0, 58.4)
- added P: Pad 1, afootprints:Pad 1, F.Cu at (284.4, 60.0)
- added P: Pad 1, afootprints:Pad 1, F.Cu at (151.4, 51.5)
- added P: Pad 1, afootprints:Pad 1, F.Cu at (155.2, 52.0)
- added P: Pad 1, afootprints:Pad 1, F.Cu at (180.6, 55.4)
- added P: Pad 1, afootprints:Pad 1, F.Cu at (253.5, 55.3)
- added P: Pad 1, afootprints:Pad 1, F.Cu at (147.5, 52.0)
- added P: Pad 1, afootprints:Pad 1, F.Cu at (185.6, 54.7)
- added P: Pad 1, afootprints:Pad 1, F.Cu at (176.1, 56.6)
- added R25: 4.7, afootprints:1206 R, F.Cu at (136.7, 32.2)
- added R26: 4.7, afootprints:1206 R, F.Cu at (139.4, 36.4)
- added R27: 4,7, afootprints:1206 R, F.Cu at (168.2, 32.8)
- added R28: 4.7, afootprints:1206 R, F.Cu at (166.2, 31.5)
- added R29: 4.7, afootprints:1206 R, F.Cu at (149.8, 70.2)
- added R30: 4.7, afootprints:1206 R, F.Cu at (153.0, 65.3)
- added R31: 4.7, afootprints:1206 R, F.Cu at (137.1, 37.6)
- added R32: 4.7, afootprints:1206 R, F.Cu at (134.7, 33.4)
- added R33: 4.7, afootprints:1206 R, F.Cu at (165.9, 37.0)
- added R34: 4.7, afootprints:1206 R, F.Cu at (163.6, 35.6)
- added R35: 4.7, afootprints:1206 R, F.Cu at (153.0, 70.3)
- added R36: 4.7, afootprints:1206 R, F.Cu at (149.8, 65.3)
- added R37: 4.7, afootprints:1206 R, F.Cu at (183.3, 37.5)
- added R38: 4.7, afootprints:1206 R, F.Cu at (198.1, 27.8)
- added R39: 4,7, afootprints:1206 R, F.Cu at (216.8, 42.3)
- added R40: 4.7, afootprints:1206 R, F.Cu at (225.0, 60.4)
- added R41: 4.7, afootprints:1206 R, F.Cu at (207.6, 74.8)
- added R42: 4.7, afootprints:1206 R, F.Cu at (184.6, 68.1)
- added R43: 4.7, afootprints:1206 R, F.Cu at (185.3, 46.3)
- added R44: 4.7, afootprints:1206 R, F.Cu at (192.3, 29.3)
- added R45: 4.7, afootprints:1206 R, F.Cu at (220.3, 36.1)
- added R46: 4.7, afootprints:1206 R, F.Cu at (225.6, 52.8)
- added R47: 4.7, afootprints:1206 R, F.Cu at (213.6, 73.3)
- added R48: 4.7, afootprints:1206 R, F.Cu at (189.3, 71.8)
- added R49: 4.7, afootprints:1206 R, F.Cu at (247.0, 28.1)
- added R50: 4.7, afootprints:1206 R, F.Cu at (264.0, 28.6)
- added R51: 4,7, afootprints:1206 R, F.Cu at (260.4, 27.5)
- added R52: 4.7, afootprints:1206 R, F.Cu at (252.2, 64.3)
- added R53: 4.7, afootprints:1206 R, F.Cu at (251.9, 39.4)
- added R54: 4.7, afootprints:1206 R, F.Cu at (260.6, 34.9)
- added R55: 4.7, afootprints:1206 R, F.Cu at (242.9, 33.3)
- added R56: 4.7, afootprints:1206 R, F.Cu at (264.0, 33.5)
- added R57: 4.7, afootprints:1206 R, F.Cu at (242.9, 28.4)
- added R58: 4.7, afootprints:1206 R, F.Cu at (254.9, 64.3)
- added R59: 4.7, afootprints:1206 R, F.Cu at (247.0, 34.4)
- added R60: 4.7, afootprints:1206 R, F.Cu at (255.3, 39.4)
- added R61: 4.7, afootprints:1206 R, F.Cu at (290.5, 41.0)
- added R62: 4.7, afootprints:1206 R, F.Cu at (276.4, 69.3)
- added R63: 4,7, afootprints:1206 R, F.Cu at (301.9, 44.0)
- added R64: 4.7, afootprints:1206 R, F.Cu at (315.5, 69.3)
- added R65: 4.7, afootprints:1206 R, F.Cu at (303.8, 65.0)
- added R66: 4.7, afootprints:1206 R, F.Cu at (299.9, 38.0)
- added R67: 4.7, afootprints:1206 R, F.Cu at (291.5, 38.0)
- added R68: 4.7, afootprints:1206 R, F.Cu at (278.6, 64.0)
- added R69: 4.7, afootprints:1206 R, F.Cu at (301.0, 41.0)
- added R70: 4.7, afootprints:1206 R, F.Cu at (313.5, 63.7)
- added R71: 4.7, afootprints:1206 R, F.Cu at (280.0, 73.0)
- added R72: 4.7, afootprints:1206 R, F.Cu at (312.5, 73.0)
- added wht-: Pad 1, afootprints:Pad 1, F.Cu at (253.4, 47.9)
- moved R12 0.22 mm to (50.4, 39.4)
- moved P 0.20 mm to (48.6, 55.3)
- moved D1 0.10 mm to (27.6, 30.9)
- moved D10 0.10 mm to (44.2, 48.1)
- moved D11 0.10 mm to (53.1, 63.1)
- moved D12 0.10 mm to (53.1, 48.1)
- moved D13 0.10 mm to (33.0, 34.6)
- moved D14 0.10 mm to (33.0, 27.1)
- moved D15 0.10 mm to (64.0, 34.6)
- moved D16 0.10 mm to (64.0, 27.1)
- moved D17 0.10 mm to (42.9, 30.8)
- moved D18 0.10 mm to (54.2, 30.8)
- moved D2 0.10 mm to (33.0, 30.9)
- moved D21 0.10 mm to (44.2, 40.6)
- moved D22 0.10 mm to (44.2, 55.6)
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Routing:
- net Net-(J4-Pad2): track 0.00 -> 219.1 mm
- net Net-(J3-Pad2): track 0.00 -> 217.6 mm
- net Net-(D86-Pad1): track 0.00 -> 200.9 mm
- net Net-(D73-Pad1): track 0.00 -> 193.8 mm
- net Net-(D134-Pad1): track 0.00 -> 177.1 mm
- net Net-(D101-Pad1): track 0.00 -> 147.4 mm
- net Net-(J6-Pad2): track 0.00 -> 120.2 mm
- net Net-(D110-Pad1): track 0.00 -> 111.5 mm
- net Net-(D121-Pad1): track 0.00 -> 105.8 mm
- net Net-(D62-Pad1): track 0.00 -> 83.6 mm
- net Net-(J5-Pad2): track 0.00 -> 74.5 mm
- net Net-(D49-Pad1): track 0.00 -> 50.8 mm
- net Net-(D75-Pad2): track 0.00 -> 29.0 mm
- net Net-(D89-Pad1): track 0.00 -> 22.1 mm
- net Net-(D135-Pad2): track 0.00 -> 22.1 mm
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Other:
- board text added: "7V+"
- board text added: "Daniel Hoefer"
- board text added: "Daniel Hoefer Toyota Emblem May 2022 Rev: 2.3"
- board text added: "Romans 8:31"
- board text added: "amb-"
- board text added: "wht-"
- board text removed: "- - - - T O Y O T A"
- board text removed: "Daniel Hoefer Toyota Emblem March 2022 Rev: 1.12"
