File: Toyota Satoshi Emblem/Toyota Satoshi Emblem.kicad_pcb (KiCad board)
At the start: 2 copper layers, 372.3 x 63 mm, 234 parts

Commit message: v2.4
Letter-Board and Raptor Lights completed. Onto the Control Board
Parts:
- added 7V+: Pad 2, afootprints:Pad 2, F.Cu at (54.5, 97.7)
- added 7V+: Pad 2, afootprints:Pad 2, F.Cu at (131.0, 97.7)
- added 7V+: Pad 2, afootprints:Pad 2, F.Cu at (282.5, 97.7)
- added 7V+: Pad 2, afootprints:Pad 2, F.Cu at (206.5, 97.7)
- added D145: WLED, afootprints:5730 LED W, F.Cu at (32.1, 92.3)
- added D146: WLED, afootprints:5730 LED W, F.Cu at (39.1, 92.3)
- added D147: WLED, afootprints:5730 LED W, F.Cu at (53.1, 92.3)
- added D148: WLED, afootprints:5730 LED W, F.Cu at (46.1, 92.3)
- added D149: WLED, afootprints:5730 LED W, F.Cu at (60.1, 92.3)
- added D150: WLED, afootprints:5730 LED W, F.Cu at (67.1, 92.3)
- added D151: ALED, afootprints:5730 LED A, F.Cu at (42.6, 92.3)
- added D152: ALED, afootprints:5730 LED A, F.Cu at (35.6, 92.3)
- added D153: ALED, afootprints:5730 LED A, F.Cu at (56.6, 92.3)
- added D154: ALED, afootprints:5730 LED A, F.Cu at (49.6, 92.3)
- added D155: ALED, afootprints:5730 LED A, F.Cu at (70.6, 92.5)
- added D156: ALED, afootprints:5730 LED A, F.Cu at (63.6, 92.3)
- added D157: WLED, afootprints:5730 LED W, F.Cu at (108.6, 92.3)
- added D158: WLED, afootprints:5730 LED W, F.Cu at (115.6, 92.3)
- added D159: WLED, afootprints:5730 LED W, F.Cu at (129.6, 92.3)
- added D160: WLED, afootprints:5730 LED W, F.Cu at (122.6, 92.3)
- added D161: WLED, afootprints:5730 LED W, F.Cu at (136.6, 92.3)
- added D162: WLED, afootprints:5730 LED W, F.Cu at (143.6, 92.3)
- added D163: ALED, afootprints:5730 LED A, F.Cu at (119.1, 92.3)
- added D164: ALED, afootprints:5730 LED A, F.Cu at (112.1, 92.3)
- added D165: ALED, afootprints:5730 LED A, F.Cu at (133.1, 92.3)
- added D166: ALED, afootprints:5730 LED A, F.Cu at (126.1, 92.3)
- added D167: ALED, afootprints:5730 LED A, F.Cu at (147.1, 92.5)
- added D168: ALED, afootprints:5730 LED A, F.Cu at (140.1, 92.3)
- added D169: WLED, afootprints:5730 LED W, F.Cu at (184.1, 92.3)
- added D170: WLED, afootprints:5730 LED W, F.Cu at (191.1, 92.3)
- added D171: WLED, afootprints:5730 LED W, F.Cu at (205.1, 92.3)
- added D172: WLED, afootprints:5730 LED W, F.Cu at (198.1, 92.3)
- added D173: WLED, afootprints:5730 LED W, F.Cu at (212.1, 92.3)
- added D174: WLED, afootprints:5730 LED W, F.Cu at (219.1, 92.3)
- added D175: ALED, afootprints:5730 LED A, F.Cu at (194.6, 92.3)
- added D176: ALED, afootprints:5730 LED A, F.Cu at (187.6, 92.3)
- added D177: ALED, afootprints:5730 LED A, F.Cu at (208.6, 92.3)
- added D178: ALED, afootprints:5730 LED A, F.Cu at (201.6, 92.3)
- added D179: ALED, afootprints:5730 LED A, F.Cu at (222.6, 92.5)
- added D180: ALED, afootprints:5730 LED A, F.Cu at (215.6, 92.3)
- added D181: WLED, afootprints:5730 LED W, F.Cu at (260.1, 92.3)
- added D182: WLED, afootprints:5730 LED W, F.Cu at (267.1, 92.3)
- added D183: WLED, afootprints:5730 LED W, F.Cu at (281.1, 92.3)
- added D184: WLED, afootprints:5730 LED W, F.Cu at (274.1, 92.3)
- added D185: WLED, afootprints:5730 LED W, F.Cu at (288.1, 92.3)
- added D186: WLED, afootprints:5730 LED W, F.Cu at (295.1, 92.3)
- added D187: ALED, afootprints:5730 LED A, F.Cu at (270.6, 92.3)
- added D188: ALED, afootprints:5730 LED A, F.Cu at (263.6, 92.3)
- added D189: ALED, afootprints:5730 LED A, F.Cu at (284.6, 92.3)
- added D190: ALED, afootprints:5730 LED A, F.Cu at (277.6, 92.3)
- added D191: ALED, afootprints:5730 LED A, F.Cu at (298.6, 92.5)
- added D192: ALED, afootprints:5730 LED A, F.Cu at (291.6, 92.3)
- added R73: 4.7, afootprints:1206 R, F.Cu at (31.6, 97.8)
- added R74: 4.7, afootprints:1206 R, F.Cu at (41.3, 97.8)
- added R75: 4.7, afootprints:1206 R, F.Cu at (70.3, 97.8)
- added R76: 4.7, afootprints:1206 R, F.Cu at (36.5, 97.7)
- added R77: 4.7, afootprints:1206 R, F.Cu at (65.6, 97.1)
- added R78: 4.7, afootprints:1206 R, F.Cu at (73.8, 97.0)
- added R79: 4.7, afootprints:1206 R, F.Cu at (108.1, 97.8)
- added R80: 4.7, afootprints:1206 R, F.Cu at (117.8, 97.8)
- added R81: 4.7, afootprints:1206 R, F.Cu at (146.8, 97.8)
- added R82: 4.7, afootprints:1206 R, F.Cu at (113.0, 97.7)
- added R83: 4.7, afootprints:1206 R, F.Cu at (142.1, 97.1)
- added R84: 4.7, afootprints:1206 R, F.Cu at (150.3, 97.0)
- added R85: 4.7, afootprints:1206 R, F.Cu at (183.6, 97.8)
- added R86: 4.7, afootprints:1206 R, F.Cu at (193.3, 97.8)
- added R87: 4.7, afootprints:1206 R, F.Cu at (222.3, 97.8)
- added R88: 4.7, afootprints:1206 R, F.Cu at (188.5, 97.7)
- added R89: 4.7, afootprints:1206 R, F.Cu at (217.6, 97.1)
- added R90: 4.7, afootprints:1206 R, F.Cu at (225.8, 97.0)
- added R91: 4.7, afootprints:1206 R, F.Cu at (259.6, 97.8)
- added R92: 4.7, afootprints:1206 R, F.Cu at (269.3, 97.8)
- added R93: 4.7, afootprints:1206 R, F.Cu at (298.3, 97.8)
- added R94: 4.7, afootprints:1206 R, F.Cu at (264.5, 97.7)
- added R95: 4.7, afootprints:1206 R, F.Cu at (293.6, 97.1)
- added R96: 4.7, afootprints:1206 R, F.Cu at (301.8, 97.0)
- added amb-: Pad 2, afootprints:Pad 2, F.Cu at (200.2, 97.7)
- added amb-: Pad 2, afootprints:Pad 2, F.Cu at (124.7, 97.7)
- added amb-: Pad 2, afootprints:Pad 2, F.Cu at (276.2, 97.7)
- added amb-: Pad 2, afootprints:Pad 2, F.Cu at (48.2, 97.7)
- added wht-: Pad 2, afootprints:Pad 2, F.Cu at (60.9, 97.8)
- added wht-: Pad 2, afootprints:Pad 2, F.Cu at (212.9, 97.8)
- added wht-: Pad 2, afootprints:Pad 2, F.Cu at (137.4, 97.8)
- added wht-: Pad 2, afootprints:Pad 2, F.Cu at (288.9, 97.8)
Routing:
- net Net-(D157-Pad1): track 0.00 -> 55.0 mm
- net Net-(D145-Pad1): track 0.00 -> 54.2 mm
- net Net-(D169-Pad1): track 0.00 -> 54.2 mm
- net Net-(D181-Pad1): track 0.00 -> 54.2 mm
- net Net-(J8-Pad2): track 0.00 -> 51.9 mm
- net Net-(J9-Pad2): track 0.00 -> 51.9 mm
- net Net-(J7-Pad2): track 0.00 -> 51.9 mm
- net Net-(J10-Pad2): track 0.00 -> 51.9 mm
- net Net-(D188-Pad1): track 0.00 -> 36.4 mm
- net Net-(D176-Pad1): track 0.00 -> 36.4 mm
- net Net-(D152-Pad1): track 0.00 -> 36.4 mm
- net Net-(D164-Pad1): track 0.00 -> 36.4 mm
- net Net-(D182-Pad2): track 0.00 -> 11.0 mm
- net Net-(D170-Pad2): track 0.00 -> 11.0 mm
- net Net-(D158-Pad2): track 0.00 -> 11.0 mm
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Other:
- board size 372.3 x 63 mm -> 299.5 x 76.1 mm
- board text added: "Daniel"
- board text added: "Daniel Hoefer Toyota Emblem May 2022 Rev: 2.4"
- board text added: "Hoefer"
- board text removed: "Daniel Hoefer Toyota Emblem May 2022 Rev: 2.3"
- board text removed: "Isaiah 60:1"

Commit message: v2.5
Power/control board progress
Parts:
- added A1: LM2596 Buck, afootprints:LM2596 Buck Converter, F.Cu at (37.2, 162.0)
- added A2: LM2596 Buck, afootprints:LM2596 Buck Converter, F.Cu at (59.2, 162.0)
- added A3: LM2596 Buck, afootprints:LM2596 Buck Converter, F.Cu at (81.2, 162.0)
- added A4: LM2596 Buck, afootprints:LM2596 Buck Converter, F.Cu at (103.2, 162.0)
- added C1: 0.1uF 50V, Capacitor_THT:C_Disc_D7.5mm_W5.0mm_P5.00mm, F.Cu at (324.2, 162.8)
- added C2: 47uF 50V, Capacitor_THT:C_Radial_D5.0mm_H11.0mm_P2.00mm, F.Cu at (292.8, 159.0)
- added C3: 10uF, Capacitor_THT:C_Radial_D4.0mm_H7.0mm_P1.50mm, F.Cu at (355.0, 160.0)
- added C4: 470uF, Capacitor_THT:C_Radial_D8.0mm_H11.5mm_P3.50mm, F.Cu at (170.8, 163.0)
- added C5: 470uF, Capacitor_THT:C_Radial_D8.0mm_H11.5mm_P3.50mm, F.Cu at (161.8, 163.0)
- added D193: 1N47xxA, Diode_THT:D_DO-41_SOD81_P10.16mm_Horizontal, F.Cu at (146.5, 130.0)
- added D194: 1N4732A, Diode_THT:D_DO-41_SOD81_P10.16mm_Horizontal, F.Cu at (146.5, 153.5)
- added D195: 1N4732A, Diode_THT:D_DO-41_SOD81_P10.16mm_Horizontal, F.Cu at (150.0, 153.5)
- added D196: 1N4732A, Diode_THT:D_DO-41_SOD81_P10.16mm_Horizontal, F.Cu at (165.0, 133.7)
- added D197: 1N4732A, Diode_THT:D_DO-41_SOD81_P10.16mm_Horizontal, F.Cu at (165.0, 147.2)
- added D198: 1N47xxA, Diode_THT:D_DO-41_SOD81_P10.16mm_Horizontal, F.Cu at (150.0, 130.0)
- added D199: 1N47xxA, Diode_THT:D_DO-41_SOD81_P10.16mm_Horizontal, F.Cu at (165.0, 110.0)
- added D200: 1N4007, Diode_THT:D_DO-41_SOD81_P10.16mm_Horizontal, F.Cu at (232.5, 212.8)
- added D201: 5KP16A, Diode_THT:D_P600_R-6_P20.00mm_Horizontal, F.Cu at (185.0, 110.5)
- added D202: 1N4739A, Diode_THT:D_DO-41_SOD81_P10.16mm_Horizontal, F.Cu at (254.2, 192.4)
- added D203: 1N4007, Diode_THT:D_DO-41_SOD81_P10.16mm_Horizontal, F.Cu at (217.6, 229.0)
- added D204: 1N4746A, Diode_THT:D_DO-41_SOD81_P10.16mm_Horizontal, F.Cu at (232.5, 208.6)
- added D205: 1N4738A, Diode_THT:D_DO-41_SOD81_P10.16mm_Horizontal, F.Cu at (292.4, 145.1)
- added D206: LED, LED_SMD:LED_1206_3216Metric_Pad1.42x1.75mm_HandSolder, F.Cu at (148.0, 111.5)
- added D207: LED, LED_SMD:LED_1206_3216Metric_Pad1.42x1.75mm_HandSolder, F.Cu at (148.0, 114.5)
- added D208: LED, LED_SMD:LED_1206_3216Metric_Pad1.42x1.75mm_HandSolder, F.Cu at (148.0, 117.5)
- added D209: LED, LED_SMD:LED_1206_3216Metric_Pad1.42x1.75mm_HandSolder, F.Cu at (148.0, 120.5)
- added D210: LED, LED_SMD:LED_1206_3216Metric_Pad1.42x1.75mm_HandSolder, F.Cu at (148.0, 123.5)
- added D211: LED, LED_SMD:LED_1206_3216Metric_Pad1.42x1.75mm_HandSolder, F.Cu at (148.0, 126.5)
- added D212: RED 1206, LED_SMD:LED_1206_3216Metric_Pad1.42x1.75mm_HandSolder, F.Cu at (222.8, 232.8)
- added D213: RED 1206, LED_SMD:LED_1206_3216Metric_Pad1.42x1.75mm_HandSolder, F.Cu at (210.8, 232.8)
- added D214: RED 1206, LED_SMD:LED_1206_3216Metric_Pad1.42x1.75mm_HandSolder, F.Cu at (234.8, 232.8)
- added F1: 10A, afootprints:Univ_AUTO_Fuse, F.Cu at (199.8, 108.7)
- added J11: Letter Terminal, TerminalBlock_Phoenix:TerminalBlock_Phoenix_MKDS-1,5-3_1x03_P5.00mm_Horizontal, F.Cu at (294.1, 125.5)
- added J12: Letter Terminal, TerminalBlock_Phoenix:TerminalBlock_Phoenix_MKDS-1,5-3_1x03_P5.00mm_Horizontal, F.Cu at (284.4, 169.8)
- added J13: Letter Terminal, TerminalBlock_Phoenix:TerminalBlock_Phoenix_MKDS-1,5-3_1x03_P5.00mm_Horizontal, F.Cu at (311.1, 137.3)
- added J14: Letter Terminal, TerminalBlock_Phoenix:TerminalBlock_Phoenix_MKDS-1,5-3_1x03_P5.00mm_Horizontal, F.Cu at (311.1, 125.5)
- added J15: Letter Terminal, TerminalBlock_Phoenix:TerminalBlock_Phoenix_MKDS-1,5-3_1x03_P5.00mm_Horizontal, F.Cu at (294.1, 137.3)
- added J16: Letter Terminal, TerminalBlock_Phoenix:TerminalBlock_Phoenix_MKDS-1,5-3_1x03_P5.00mm_Horizontal, F.Cu at (216.9, 221.2)
- added J17: Power 1, TerminalBlock_Phoenix:TerminalBlock_Phoenix_MKDS-1,5-2_1x02_P5.00mm_Horizontal, F.Cu at (193.1, 159.5)
- added J18: Power 2, TerminalBlock_Phoenix:TerminalBlock_Phoenix_MKDS-1,5-2_1x02_P5.00mm_Horizontal, F.Cu at (193.1, 148.5)
- added J19: Raptor Terminal, TerminalBlock_Phoenix:TerminalBlock_Phoenix_MKDS-1,5-3-5.08_1x03_P5.08mm_Horizontal, F.Cu at (255.9, 180.4)
- added J20: Raptor Terminal, TerminalBlock_Phoenix:TerminalBlock_Phoenix_MKDS-1,5-3-5.08_1x03_P5.08mm_Horizontal, F.Cu at (238.6, 192.3)
- added J21: Serial 3, TerminalBlock_Phoenix:TerminalBlock_Phoenix_MKDS-1,5-2_1x02_P5.00mm_Horizontal, B.Cu at (158.0, 133.5)
- added J22: Serial 2, TerminalBlock_Phoenix:TerminalBlock_Phoenix_MKDS-1,5-2_1x02_P5.00mm_Horizontal, B.Cu at (158.0, 122.5)
- added J23: Raptor Terminal, TerminalBlock_Phoenix:TerminalBlock_Phoenix_MKDS-1,5-3-5.08_1x03_P5.08mm_Horizontal, F.Cu at (216.9, 209.3)
- added J24: Serial 1, TerminalBlock_Phoenix:TerminalBlock_Phoenix_MKDS-1,5-2_1x02_P5.00mm_Horizontal, B.Cu at (158.0, 111.5)
- added J25: Raptor Terminal, TerminalBlock_Phoenix:TerminalBlock_Phoenix_MKDS-1,5-3-5.08_1x03_P5.08mm_Horizontal, F.Cu at (238.6, 180.4)
- added J26: Turn Sig., TerminalBlock_Phoenix:TerminalBlock_Phoenix_MKDS-1,5-2_1x02_P5.00mm_Horizontal, B.Cu at (158.0, 144.5)
- added J27: Misc. Sig., TerminalBlock_Phoenix:TerminalBlock_Phoenix_MKDS-1,5-2_1x02_P5.00mm_Horizontal, B.Cu at (158.0, 155.5)
- added J28: Relay Power, TerminalBlock_Phoenix:TerminalBlock_Phoenix_PT-1,5-2-5.0-H_1x02_P5.00mm_Horizontal, F.Cu at (284.5, 204.6)
- added J29: Power In, TerminalBlock_Phoenix:TerminalBlock_Phoenix_MKDS-1,5-2_1x02_P5.00mm_Horizontal, F.Cu at (193.1, 137.5)
- added Q1: IRLR7843, afootprints:IRLR7843, F.Cu at (318.2, 163.1)
- added Q10: IRLR7843, afootprints:IRLR7843, F.Cu at (336.9, 143.6)
- added Q11: IRLR7843, afootprints:IRLR7843, F.Cu at (238.6, 227.0)
- added Q12: 2N3904, Package_TO_SOT_THT:TO-92_Inline, F.Cu at (369.5, 134.4)
- added Q13: IRLR7843, afootprints:IRLR7843, F.Cu at (345.0, 135.6)
- added Q14: IRLR7843, afootprints:IRLR7843, F.Cu at (289.9, 179.4)
- added Q15: IRLR7843, afootprints:IRLR7843, F.Cu at (312.6, 147.0)
- added Q16: 2N3904, Package_TO_SOT_THT:TO-92_Inline, F.Cu at (342.8, 154.7)
- added Q17: IRLR7843, afootprints:IRLR7843, F.Cu at (357.1, 123.3)
- added Q18: IRLR7843, afootprints:IRLR7843, F.Cu at (345.0, 127.5)
- added Q19: IRLR7843, afootprints:IRLR7843, F.Cu at (252.7, 218.5)
- added Q2: IRLR7843, afootprints:IRLR7843, F.Cu at (302.1, 179.4)
- added Q20: IRLR7843, afootprints:IRLR7843, F.Cu at (284.8, 195.5)
- added Q21: IRLR7843, afootprints:IRLR7843, F.Cu at (277.8, 187.5)
- added Q22: 2N3904, Package_TO_SOT_THT:TO-92_Inline, F.Cu at (375.1, 128.3)
- added Q23: IRLR7843, afootprints:IRLR7843, F.Cu at (324.8, 147.0)
- added Q24: 2N3904, Package_TO_SOT_THT:TO-92_Inline, F.Cu at (355.0, 142.4)
- added Q25: IRLR7843, afootprints:IRLR7843, F.Cu at (312.6, 155.0)
- added Q26: IRLR7843, afootprints:IRLR7843, F.Cu at (264.9, 206.6)
- added Q27: IRLR7843, afootprints:IRLR7843, F.Cu at (277.0, 206.6)
- added Q28: IRLR7843, afootprints:IRLR7843, F.Cu at (332.8, 127.5)
- added Q29: IRLR7843, afootprints:IRLR7843, F.Cu at (332.8, 135.6)
- added Q3: IRLR7843, afootprints:IRLR7843, F.Cu at (272.6, 198.6)
- added Q30: 2N3904, Package_TO_SOT_THT:TO-92_Inline, F.Cu at (349.3, 154.7)
- added Q31: IRLR7843, afootprints:IRLR7843, F.Cu at (250.7, 226.6)
- added Q32: 2N3904, Package_TO_SOT_THT:TO-92_Inline, F.Cu at (342.8, 160.5)
- added Q33: IRLR7843, afootprints:IRLR7843, F.Cu at (264.9, 214.7)
- added Q34: IRLR7843, afootprints:IRLR7843, F.Cu at (306.1, 171.1)
- added Q35: IRLR7843, afootprints:IRLR7843, F.Cu at (252.7, 210.5)
- added Q36: 2N3904, Package_TO_SOT_THT:TO-92_Inline, F.Cu at (363.0, 134.4)
- added Q37: IRLR7843, afootprints:IRLR7843, F.Cu at (238.6, 219.0)
- added Q38: IRLR7843, afootprints:IRLR7843, F.Cu at (277.8, 179.4)
- added Q39: IRLR7843, afootprints:IRLR7843, F.Cu at (306.1, 163.1)
- added Q4: 2N3904, Package_TO_SOT_THT:TO-92_Inline, F.Cu at (375.1, 122.5)
- added Q40: 2N3904, Package_TO_SOT_THT:TO-92_Inline, F.Cu at (381.7, 122.5)
- added Q41: IRF4905, afootprints:IRF4905, F.Cu at (171.5, 128.0)
- added Q42: IRF4905, afootprints:IRF4905, F.Cu at (184.6, 142.0)
- added Q43: BC327, Package_TO_SOT_THT:TO-92_Inline, F.Cu at (355.0, 148.2)
- added Q44: BC337, Package_TO_SOT_THT:TO-92_Inline, F.Cu at (333.3, 162.8)
- added Q5: IRLR7843, afootprints:IRLR7843, F.Cu at (289.9, 187.5)
- added Q6: IRLR7843, afootprints:IRLR7843, F.Cu at (324.8, 155.0)
- added Q7: IRLR7843, afootprints:IRLR7843, F.Cu at (262.9, 226.6)
- added Q8: 2N3904, Package_TO_SOT_THT:TO-92_Inline, F.Cu at (361.5, 142.4)
- added Q9: IRLR7843, afootprints:IRLR7843, F.Cu at (260.5, 198.6)
- added R100: 10K, afootprints:1206 R, F.Cu at (265.1, 220.2)
- added R101: 10K, afootprints:1206 R, F.Cu at (246.5, 232.1)
- added R102: 1K, afootprints:1206 R, F.Cu at (301.5, 208.9)
- added R103: 1K, afootprints:1206 R, B.Cu at (148.0, 114.5)
- added R104: 10K, afootprints:1206 R, F.Cu at (308.7, 190.1)
- added R105: 10K, afootprints:1206 R, F.Cu at (318.4, 180.5)
- added R106: 1K, afootprints:1206 R, F.Cu at (318.4, 183.6)
- added R107: 1K, afootprints:1206 R, B.Cu at (148.0, 117.5)
- added R108: 10K, afootprints:1206 R, F.Cu at (257.7, 232.1)
- added R109: 10K, afootprints:1206 R, F.Cu at (330.5, 174.6)
- added R110: 1K, afootprints:1206 R, F.Cu at (336.5, 166.8)
- added R111: 1K, afootprints:1206 R, B.Cu at (148.0, 120.5)
- added R112: 10K, afootprints:1206 R, F.Cu at (289.3, 221.7)
- added R113: 10K, afootprints:1206 R, F.Cu at (388.1, 126.6)
- added R114: 1K, afootprints:1206 R, F.Cu at (368.8, 138.4)
- added R115: 10K, afootprints:1206 R, F.Cu at (263.3, 232.1)
- added R116: 1K, afootprints:1206 R, B.Cu at (148.0, 123.5)
- added R117: 1K, afootprints:1206 R, F.Cu at (324.0, 180.5)
- added R118: 1K, afootprints:1206 R, B.Cu at (148.0, 126.5)
- added R119: 10K, afootprints:1206 R, F.Cu at (382.5, 126.6)
- added R120: 10K, afootprints:1206 R, F.Cu at (298.9, 212.0)
- added R121: 10K, afootprints:1206 R, F.Cu at (356.6, 155.3)
- added R122: 1K, afootprints:1206 R, F.Cu at (336.5, 169.9)
- added R123: 10K, afootprints:1206 R, F.Cu at (301.5, 205.9)
- added R124: 50, afootprints:1206 R, F.Cu at (295.8, 205.9)
- added R125: 1K, afootprints:1206 R, F.Cu at (314.4, 190.1)
- added R127: 10K, afootprints:1206 R, F.Cu at (293.2, 212.1)
- added R128: 10K, afootprints:1206 R, F.Cu at (259.5, 220.2)
- added R129: 10K, afootprints:1206 R, F.Cu at (313.0, 199.2)
- added R130: 1K, afootprints:1206 R, F.Cu at (389.0, 120.8)
- added R132: 1K, afootprints:1206 R, B.Cu at (148.0, 149.0)
- added R133: 1K, afootprints:1206 R, B.Cu at (148.0, 146.5)
- added R134: 1K, afootprints:1206 R, B.Cu at (148.5, 158.5)
- added R135: 1K, afootprints:1206 R, B.Cu at (148.5, 156.0)
- added R136: 10K, afootprints:1206 R, F.Cu at (307.1, 205.3)
- added R137: 10K, afootprints:1206 R, F.Cu at (307.4, 202.3)
- added R138: 1K, afootprints:1206 R, F.Cu at (342.1, 170.7)
- added R139: 1K, afootprints:1206 R, F.Cu at (154.5, 130.5)
- added R141: 10K, afootprints:1206 R, F.Cu at (299.9, 157.2)
- added R142: 1K, afootprints:1206 R, F.Cu at (153.5, 124.5)
- added R143: 1K, afootprints:1206 R, F.Cu at (162.0, 115.0)
- added R144: 1K, afootprints:1206 R, F.Cu at (376.8, 132.4)
- added R145: 1K, afootprints:1206 R, F.Cu at (318.4, 186.6)
- added R146: 1K, afootprints:1206 R, F.Cu at (368.8, 141.5)
- added R147: 1K, afootprints:1206 R, F.Cu at (281.7, 224.8)
- added R148: 10K, afootprints:1206 R, F.Cu at (283.7, 221.7)
- added R149: 10K, afootprints:1206 R, F.Cu at (308.7, 193.1)
- added R150: 10K, afootprints:1206 R, B.Cu at (122.7, 140.0)
- added R151: 1K, afootprints:1206 R, B.Cu at (115.2, 140.0)
- added R152: 10K, afootprints:1206 R, B.Cu at (122.7, 137.5)
- added R153: 1K, afootprints:1206 R, B.Cu at (115.2, 137.5)
- added R154: 10K, afootprints:1206 R, B.Cu at (122.7, 135.0)
- added R155: 1K, afootprints:1206 R, B.Cu at (115.2, 135.0)
- added R156: 10K, afootprints:1206 R, B.Cu at (122.7, 132.5)
- added R157: 1K, afootprints:1206 R, B.Cu at (115.2, 132.5)
- added R158: 10K, afootprints:1206 R, B.Cu at (122.7, 130.0)
- added R159: 1K, afootprints:1206 R, B.Cu at (115.2, 130.0)
- added R160: 10K, afootprints:1206 R, B.Cu at (122.7, 127.5)
- added R161: 1K, afootprints:1206 R, B.Cu at (115.2, 127.5)
- added R162: 10K, afootprints:1206 R, B.Cu at (122.7, 125.0)
- added R163: 1K, afootprints:1206 R, B.Cu at (115.2, 125.0)
- added R164: 10K, afootprints:1206 R, B.Cu at (122.7, 122.5)
- added R165: 1K, afootprints:1206 R, B.Cu at (115.2, 122.5)
- added R166: 10K, afootprints:1206 R, B.Cu at (122.7, 120.0)
- added R167: 1K, afootprints:1206 R, B.Cu at (115.2, 120.0)
- added R168: 10K, afootprints:1206 R, B.Cu at (122.7, 117.5)
- added R169: 1K, afootprints:1206 R, B.Cu at (115.2, 117.5)
- added R97: 10K, afootprints:1206 R, F.Cu at (336.1, 176.0)
- added R98: 1K, afootprints:1206 R, F.Cu at (314.4, 196.2)
- added R99: 1K, afootprints:1206 R, B.Cu at (148.0, 111.5)
- added SW1: SW_DIP_x10, Button_Switch_THT:SW_DIP_SPSTx10_Slide_9.78x27.58mm_W7.62mm_P2.54mm, F.Cu at (126.5, 139.9)
- added U1: MEGA_PRO_EMBED_CH340G_/_ATMEGA2560, afootprints:MODULE_MEGA_PRO_EMBED_CH340G___ATMEGA2560, F.Cu at (125.2, 135.0)
- added U2: L7805, afootprints:L7805, B.Cu at (137.5, 154.0)
Routing:
- net GND: track 0.00 -> 87.0 mm, vias 0 -> 75
- net /TX1: track 0.00 -> 61.6 mm
- net /RX1: track 0.00 -> 42.0 mm
- net Net-(Q18-Pad1): track 0.00 -> 33.1 mm
- net /TX3: track 0.00 -> 32.1 mm
- net Net-(Q26-Pad1): track 0.00 -> 31.1 mm
- net Net-(Q10-Pad1): track 0.00 -> 30.7 mm
- net /TX2: track 0.00 -> 29.8 mm
- net Net-(Q14-Pad1): track 0.00 -> 28.9 mm
- net Net-(Q2-Pad1): track 0.00 -> 27.4 mm
- net /RX2: track 0.00 -> 26.6 mm
- net Net-(Q6-Pad1): track 0.00 -> 26.1 mm
- net Net-(Q29-Pad1): track 0.00 -> 24.2 mm
- net Net-(Q21-Pad1): track 0.00 -> 22.8 mm
- net +5V: track 0.00 -> 22.5 mm
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- added copper zone on B.Cu, net +12V
- added copper zone on F.Cu, net +12V
- added copper zone on B.Cu, net GND
- added copper zone on F.Cu, net GND
- added copper zone on B.Cu, net Net-(C1-Pad1)
- added copper zone on F.Cu, net Net-(C1-Pad1)
- added copper zone on B.Cu, net Net-(D201-Pad1)
- added copper zone on F.Cu, net Net-(D201-Pad1)
- added copper zone on B.Cu, net Net-(F1-Pad2)
- added copper zone on F.Cu, net Net-(F1-Pad2)
Other:
- board size 299.5 x 76.1 mm -> 299.5 x 144.7 mm
- board text added: "Daniel Hoefer Toyota Emblem May 2022 Rev: 2.5"
- board text removed: "Daniel Hoefer Toyota Emblem May 2022 Rev: 2.4"
