File: Toyota Satoshi Emblem/Toyota Satoshi Emblem.kicad_pcb (KiCad board)
At the start: 2 copper layers, 299.5 x 144.7 mm, 486 parts, among them J11 Letter Terminal, J12 Letter Terminal, J13 Letter Terminal, J14 Letter Terminal, J15 Letter Terminal, J16 Letter Terminal, J17 Power 1, J18 Power 2, J19 Raptor Terminal, J20 Raptor Terminal, J21 Serial 3, J22 Serial 2, J23 Raptor Terminal, J24 Serial 1, J25 Raptor Terminal, J26 Turn Sig., J27 Misc. Sig., J28 Relay Power, J29 Power In, Q1 IRLR7843, Q10 IRLR7843, Q11 IRLR7843, Q12 2N3904, Q13 IRLR7843, Q14 IRLR7843, Q15 IRLR7843, Q16 2N3904, Q17 IRLR7843, Q18 IRLR7843, Q19 IRLR7843, Q2 IRLR7843, Q20 IRLR7843, Q21 IRLR7843, Q22 2N3904, Q23 IRLR7843, Q24 2N3904, Q25 IRLR7843, Q26 IRLR7843, Q27 IRLR7843, Q28 IRLR7843, Q29 IRLR7843, Q3 IRLR7843, Q30 2N3904, Q31 IRLR7843, Q32 2N3904, Q33 IRLR7843, Q34 IRLR7843, Q35 IRLR7843, Q36 2N3904, Q37 IRLR7843, Q38 IRLR7843, Q39 IRLR7843, Q4 2N3904, Q40 2N3904, Q41 IRF4905, Q42 IRF4905, Q43 BC327, Q44 BC337, Q5 IRLR7843, Q6 IRLR7843, Q7 IRLR7843, Q8 2N3904, Q9 IRLR7843, SW1 SW_DIP_x10, U1 MEGA_PRO_EMBED_CH340G_{slash}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, U2 L7805

Commit message: v2.6
More power/control board progress
Parts:
- Q12, Q16, Q22, Q24, Q30, Q32, Q36, Q4, Q40, Q8: footprint Package_TO_SOT_THT:TO-92_Inline -> Package_TO_SOT_SMD:SOT-23
- R145, R147, R148, R149: moved to B.Cu
- U2: moved to F.Cu
- moved Q22 446.1 mm to (-69.7, 162.5)
- moved Q12 440.4 mm to (-69.7, 166.9)
- moved Q4 432.0 mm to (-55.0, 162.5)
- moved Q8 427.2 mm to (-64.8, 171.4)
- moved Q24 425.6 mm to (-69.7, 171.4)
- moved Q36 424.1 mm to (-59.9, 166.9)
- moved Q30 414.3 mm to (-64.8, 166.9)
- moved Q32 402.8 mm to (-59.9, 171.4)
- moved Q16 402.8 mm to (-59.9, 162.5)
- moved D213 402.2 mm to (-190.7, 208.9)
- moved D214 402.2 mm to (-166.7, 208.8)
- moved J16 402.2 mm to (-184.6, 197.3)
- moved J28 402.2 mm to (-116.9, 180.7)
- moved Q1 402.2 mm to (-83.2, 139.2)
- moved Q13 402.2 mm to (-56.5, 111.7)
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Routing:
- net GND: track 87.0 -> 201.7 mm, vias 75 -> 72
- net /BUCK_D: track 0.00 -> 86.1 mm
- net Net-(D197-Pad1): track 0.00 -> 70.4 mm
- net Net-(D196-Pad1): track 0.00 -> 64.9 mm
- net Net-(D195-Pad1): track 0.00 -> 53.5 mm
- net +5V: track 22.5 -> 70.7 mm
- net Net-(D194-Pad1): track 0.00 -> 47.2 mm
- net Net-(C1-Pad1): track 0.00 -> 38.3 mm, vias 47 -> 28
- net Net-(D200-Pad1): track 0.00 -> 30.9 mm
- net +12V: track 0.00 -> 24.5 mm
- net Net-(D200-Pad2): track 0.00 -> 21.4 mm
- net Net-(D203-Pad2): track 0.00 -> 20.1 mm
- net Net-(Q43-Pad2): track 0.00 -> 19.5 mm
- net Net-(D205-Pad1): track 0.00 -> 14.6 mm
- net Net-(D202-Pad2): track 0.00 -> 11.6 mm
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Other:
- outline, holes or cut-outs redrawn
- board text added: "Daniel Hoefer Toyota Emblem May 2022 Rev: 2.6"
- board text removed: "Daniel Hoefer Toyota Emblem May 2022 Rev: 2.5"

Commit message: v2.7
More work on the driver circuits
Parts:
- removed J28: Relay Power, TerminalBlock_Phoenix:TerminalBlock_Phoenix_PT-1,5-2-5.0-H_1x02_P5.00mm_Horizontal
- removed R136, R141: 10K, afootprints:1206 R
- added J30: Sensor Term., TerminalBlock_Phoenix:TerminalBlock_Phoenix_MKDS-1,5-3_1x03_P5.00mm_Horizontal, B.Cu at (203.5, 116.5)
- added Q35: IRLR7843, afootprints:IRLR7843, F.Cu at (88.6, 139.0)
- added R126: 10K, afootprints:1206 R, F.Cu at (134.2, 301.4)
- added R131: 10K, afootprints:1206 R, F.Cu at (134.2, 298.3)
- J11, J13, J14, J15, J16: moved to B.Cu
- R148: moved to F.Cu
- moved D212 237.0 mm to (-0.52, 365.2)
- moved D213 237.0 mm to (-12.5, 365.2)
- moved D214 237.0 mm to (11.5, 365.2)
- moved Q1 237.0 mm to (94.9, 295.5)
- moved Q10 237.0 mm to (113.6, 276.1)
- moved Q12 237.0 mm to (108.5, 323.3)
- moved Q13 237.0 mm to (121.7, 268.0)
- moved Q14 237.0 mm to (66.6, 311.9)
- moved Q16 237.0 mm to (118.3, 318.9)
- moved Q18 237.0 mm to (121.7, 260.0)
- moved Q19 237.0 mm to (29.4, 351.0)
- moved Q2 237.0 mm to (78.8, 311.9)
- moved Q20 237.0 mm to (61.5, 328.0)
- moved Q21 237.0 mm to (54.5, 319.9)
- moved Q22 237.0 mm to (108.5, 318.9)
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Connections:
- R100 pad 1: Net-(Q3-Pad1) -> GND
- R100 pad 2: /BUCK_A -> Net-(Q26-Pad1)
- R104 pad 1: Net-(Q7-Pad1) -> GND
- R104 pad 2: /BUCK_A -> Net-(Q21-Pad1)
- R108 pad 1: Net-(Q11-Pad1) -> GND
- R108 pad 2: /BUCK_B -> Net-(Q29-Pad1)
- R112 pad 1: Net-(Q15-Pad1) -> GND
- R112 pad 2: /BUCK_B -> Net-(Q34-Pad1)
- R119 pad 1: Net-(Q19-Pad1) -> GND
- R119 pad 2: /BUCK_C -> Net-(Q38-Pad1)
- R120 pad 1: Net-(Q23-Pad1) -> GND
- R120 pad 2: /BUCK_D -> Net-(Q2-Pad1)
- R127 pad 1: Net-(Q27-Pad1) -> GND
- R127 pad 2: /BUCK_C -> Net-(Q10-Pad1)
- R128 pad 1: Net-(Q31-Pad1) -> GND
- R128 pad 2: /BUCK_D -> Net-(Q14-Pad1)
- R150 pad 2: Net-(Q26-Pad1) -> Net-(Q3-Pad1)
- R152 pad 2: Net-(Q18-Pad1) -> Net-(Q7-Pad1)
- R154 pad 2: Net-(Q14-Pad1) -> Net-(Q11-Pad1)
- R156 pad 2: Net-(Q10-Pad1) -> Net-(Q15-Pad1)
- R158 pad 2: Net-(Q6-Pad1) -> Net-(Q19-Pad1)
- R160 pad 2: Net-(Q2-Pad1) -> Net-(Q27-Pad1)
- R162 pad 2: Net-(Q21-Pad1) -> Net-(Q23-Pad1)
- R164 pad 2: Net-(Q29-Pad1) -> Net-(Q31-Pad1)
- R166 pad 2: Net-(Q34-Pad1) -> Net-(Q35-Pad1)
- R168 pad 2: Net-(Q38-Pad1) -> Net-(Q39-Pad1)
- SW1 pad 1: Net-(Q26-Pad1) -> Net-(Q3-Pad1)
- SW1 pad 10: Net-(Q38-Pad1) -> Net-(Q39-Pad1)
- SW1 pad 2: Net-(Q18-Pad1) -> Net-(Q7-Pad1)
- SW1 pad 3: Net-(Q14-Pad1) -> Net-(Q11-Pad1)
- SW1 pad 4: Net-(Q10-Pad1) -> Net-(Q15-Pad1)
- SW1 pad 5: Net-(Q6-Pad1) -> Net-(Q19-Pad1)
- SW1 pad 6: Net-(Q2-Pad1) -> Net-(Q27-Pad1)
- SW1 pad 7: Net-(Q21-Pad1) -> Net-(Q23-Pad1)
- SW1 pad 8: Net-(Q29-Pad1) -> Net-(Q31-Pad1)
- SW1 pad 9: Net-(Q34-Pad1) -> Net-(Q35-Pad1)
Routing:
- net GND: track 201.7 -> 292.6 mm, vias 72 -> 74
- net Net-(Q35-Pad1): track 0.00 -> 53.7 mm, vias 0 -> 1
- net Net-(Q7-Pad1): track 0.00 -> 33.1 mm
- net Net-(Q18-Pad1): track 33.1 -> 0.00 mm
- net Net-(Q3-Pad1): track 0.00 -> 31.1 mm
- net Net-(Q26-Pad1): track 31.1 -> 0.00 mm
- net Net-(Q39-Pad1): track 0.00 -> 30.9 mm
- net Net-(Q15-Pad1): track 0.00 -> 30.7 mm
- net Net-(Q10-Pad1): track 30.7 -> 0.00 mm
- net Net-(Q14-Pad1): track 28.9 -> 0.00 mm
- net Net-(Q11-Pad1): track 0.00 -> 28.9 mm
- net Net-(Q27-Pad1): track 0.00 -> 27.4 mm
- net Net-(Q2-Pad1): track 27.4 -> 0.00 mm
- net Net-(Q6-Pad1): track 26.1 -> 0.00 mm
- net Net-(Q19-Pad1): track 0.00 -> 26.1 mm
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Other:
- board text added: "Daniel Hoefer Toyota Emblem May 2022 Rev: 2.7"
- board text added: "Letter Terminal"
- board text removed: "Daniel Hoefer Toyota Emblem May 2022 Rev: 2.6"

Commit message: v2.8
Finished assembling all boards. Next is final design checking and cleaning things up.
Parts:
- removed the Q35 at (29.4, 342.9)
- added REF**: MountingHole_2.2mm_M2, MountingHole:MountingHole_2.2mm_M2, F.Cu at (28.2, 165.2)
- added REF**: MountingHole_2.2mm_M2, MountingHole:MountingHole_2.2mm_M2, F.Cu at (28.2, 110.8)
- added REF**: MountingHole_2.2mm_M2, MountingHole:MountingHole_2.2mm_M2, F.Cu at (211.2, 165.2)
- J11: moved to F.Cu
- J12, Q10, Q11, Q12, Q13, Q14, Q15, Q16, Q17, Q18, Q19, Q22, Q25, Q26, Q27, Q30, Q5, Q6, Q7, Q8, Q9, R101, R102, R105, R106, R109, R110, R113, R114, R121, R122: moved to B.Cu
- moved R108 274.8 mm to (148.5, 114.5)
- moved R128 252.1 mm to (148.5, 127.0)
- moved D213 251.9 mm to (127.8, 156.0), turned to 180 degrees
- moved R100 245.1 mm to (148.5, 132.0)
- moved D214 243.2 mm to (135.5, 156.0), turned to 180 degrees
- moved R115 242.7 mm to (53.2, 122.2)
- moved D212 239.8 mm to (122.2, 159.2), turned to -90 degrees
- moved R120 236.5 mm to (148.5, 119.5)
- moved Q11 235.0 mm to (60.9, 129.0), turned to 180 degrees
- moved R127 233.7 mm to (148.5, 124.5)
- moved Q19 225.9 mm to (100.0, 136.3), turned to -90 degrees
- moved Q27 223.1 mm to (104.2, 121.8), turned to 180 degrees
- moved Q31 222.6 mm to (61.4, 139.0), turned to 180 degrees
- moved Q26 220.4 mm to (69.9, 120.5), turned to 180 degrees
- moved R123 216.4 mm to (72.5, 122.0)
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Connections:
- J30 pad 1: unconnected-(J30-Pad1) -> +5V
- J30 pad 2: unconnected-(J30-Pad2) -> Net-(J30-Pad2)
- J30 pad 3: unconnected-(J30-Pad3) -> GND
- R150 pad 2: Net-(Q3-Pad1) -> Net-(Q27-Pad1)
- R152 pad 2: Net-(Q7-Pad1) -> Net-(Q19-Pad1)
- R154 pad 2: Net-(Q11-Pad1) -> Net-(Q15-Pad1)
- R156 pad 2: Net-(Q15-Pad1) -> Net-(Q11-Pad1)
- R158 pad 2: Net-(Q19-Pad1) -> Net-(Q7-Pad1)
- R160 pad 2: Net-(Q27-Pad1) -> Net-(Q3-Pad1)
- R162 pad 2: Net-(Q23-Pad1) -> Net-(Q39-Pad1)
- R164 pad 2: Net-(Q31-Pad1) -> Net-(Q35-Pad1)
- R166 pad 2: Net-(Q35-Pad1) -> Net-(Q31-Pad1)
- R168 pad 2: Net-(Q39-Pad1) -> Net-(Q23-Pad1)
- SW1 pad 1: Net-(Q3-Pad1) -> Net-(Q27-Pad1)
- SW1 pad 10: Net-(Q39-Pad1) -> Net-(Q23-Pad1)
- SW1 pad 2: Net-(Q7-Pad1) -> Net-(Q19-Pad1)
- SW1 pad 3: Net-(Q11-Pad1) -> Net-(Q15-Pad1)
- SW1 pad 4: Net-(Q15-Pad1) -> Net-(Q11-Pad1)
- SW1 pad 5: Net-(Q19-Pad1) -> Net-(Q7-Pad1)
- SW1 pad 6: Net-(Q27-Pad1) -> Net-(Q3-Pad1)
- SW1 pad 7: Net-(Q23-Pad1) -> Net-(Q39-Pad1)
- SW1 pad 8: Net-(Q31-Pad1) -> Net-(Q35-Pad1)
- SW1 pad 9: Net-(Q35-Pad1) -> Net-(Q31-Pad1)
- U1 pad A4: unconnected-(U1-PadA4) -> Net-(J30-Pad2)
Routing:
- net GND: track 292.6 -> 667.5 mm, vias 74 -> 87
- net Net-(Q14-Pad1): track 0.00 -> 213.5 mm, vias 0 -> 5
- net Net-(Q3-Pad1): track 31.1 -> 207.2 mm, vias 0 -> 2
- net Net-(Q29-Pad1): track 0.00 -> 165.9 mm, vias 0 -> 4
- net Net-(Q2-Pad1): track 0.00 -> 160.7 mm, vias 0 -> 4
- net Net-(Q15-Pad1): track 30.7 -> 183.0 mm, vias 0 -> 3
- net Net-(Q10-Pad1): track 0.00 -> 146.6 mm, vias 0 -> 3
- net Net-(Q21-Pad1): track 0.00 -> 141.5 mm, vias 0 -> 4
- net Net-(Q26-Pad1): track 0.00 -> 137.3 mm, vias 0 -> 1
- net Net-(Q6-Pad1): track 0.00 -> 135.4 mm, vias 0 -> 3
- net Net-(Q31-Pad1): track 24.2 -> 155.8 mm, vias 0 -> 2
- net Net-(Q11-Pad1): track 28.9 -> 160.0 mm, vias 0 -> 1
- net Net-(Q7-Pad1): track 33.1 -> 152.2 mm, vias 0 -> 1
- net Net-(Q23-Pad1): track 22.8 -> 138.9 mm, vias 0 -> 2
- net Net-(Q18-Pad1): track 0.00 -> 106.7 mm, vias 0 -> 3
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Other:
- board text added: "Daniel Hoefer Toyota Emblem May 2022 Rev: 2.8"
- board text removed: "Daniel Hoefer Toyota Emblem May 2022 Rev: 2.7"

Commit message: v2.9
LED pad polarities and mark will be edited to fix error next rev. Otherwise clearances and board DRC parameters have been refined
Parts:
- added MT4: MountingHole_2.2mm_M2, MountingHole:MountingHole_2.2mm_M2, F.Cu at (202.5, 110.8)
- D201: footprint Diode_THT:D_P600_R-6_P20.00mm_Horizontal -> afootprints:5KP16A
- moved D201 0.50 mm to (197.5, 110.5)
- moved D34 0.23 mm to (103.2, 73.6)
- moved J11 0.20 mm to (34.5, 115.0)
- moved R86 0.20 mm to (193.1, 97.8)
- moved R81 0.18 mm to (146.8, 97.6)
- moved R87 0.18 mm to (222.3, 97.6)
- moved R75 0.17 mm to (70.3, 97.6)
- moved D167 0.13 mm to (147.1, 92.7)
- moved D157 0.13 mm to (108.6, 92.5)
- moved D158 0.13 mm to (115.6, 92.5)
- moved D159 0.13 mm to (129.6, 92.5)
- moved D160 0.13 mm to (122.6, 92.5)
- moved D161 0.13 mm to (136.6, 92.5)
- moved D162 0.13 mm to (143.6, 92.5)
- moved D163 0.13 mm to (119.1, 92.5)
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- renumbered REF** to MT1, REF** to MT2, REF** to MT3
Routing:
- net GND: track 667.5 -> 671.5 mm
- net Net-(J3-Pad2): track 217.6 -> 221.6 mm
- net Net-(D134-Pad1): track 177.1 -> 174.1 mm
- net Net-(Q14-Pad1): track 213.5 -> 211.0 mm
- net Net-(D73-Pad1): track 193.8 -> 191.9 mm
- net Net-(D25-Pad1): track 193.8 -> 192.0 mm
- net Net-(Q15-Pad1): track 183.0 -> 181.8 mm
- net Net-(J9-Pad2): track 51.9 -> 52.9 mm
- net Net-(J8-Pad2): track 51.9 -> 52.9 mm
- net Net-(D157-Pad1): track 55.0 -> 54.0 mm
- net Net-(D86-Pad1): track 200.9 -> 199.9 mm
- net Net-(J10-Pad2): track 51.9 -> 52.8 mm
- net Net-(D38-Pad1): track 200.9 -> 200.1 mm
- net Net-(D174-Pad2): track 3.66 -> 3.01 mm
- net Net-(F1-Pad2): vias 27 -> 26
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Other:
- outline, holes or cut-outs redrawn
- rule pad_to_mask_clearance: 0 -> 0.05
- board text added: "DO NOT PLUG USB POWER IN WHEN RED LEDs ARE ON"
- board text added: "Daniel Hoefer Toyota Emblem May 2022 Rev: 2.9"
- board text added: "WARNING:"
- board text added: "What then shall we say to these things? If God is for us, who can be against us?"
- board text added: "letter1"
- board text added: "letter2"
- board text added: "letter3"
- board text added: "letter4"
- board text added: "letter5"
- board text added: "letter6"
- board text added: "raptor1"
- board text added: "raptor2"
- board text added: "raptor3"
- board text added: "raptor4"
