File: Toyota Satoshi Emblem/Raptor GERBER/Raptor Gerber/Raptor Gerber.kicad_pcb (KiCad board)
At the start: 2 copper layers, 50.8 x 11 mm, 23 parts

Commit message: FIC initial
major overhaul, new beginnings
Parts:
- removed the REF** at (17.0, 18.9)
- removed the REF** at (63.8, 18.9)
- added REF**: M2.5_Mechanical, afootprints:M2.5_Mechanical, F.Cu at (16.4, 19.7)
- added REF**: M2.5_Mechanical, afootprints:M2.5_Mechanical, F.Cu at (63.2, 19.7)
- moved R93 1.43 mm to (58.1, 25.1)
- moved R95 1.36 mm to (53.5, 24.4)
- moved D183 1.03 mm to (41.5, 19.6)
- moved D184 1.03 mm to (34.5, 19.6)
- moved D185 1.03 mm to (48.5, 19.6)
- moved D186 1.03 mm to (55.5, 19.6)
- moved D189 1.03 mm to (45.0, 19.6)
- moved D190 1.03 mm to (38.0, 19.6)
- moved D191 1.03 mm to (59.0, 19.6)
- moved D192 1.03 mm to (52.0, 19.6)
- moved R92 1.03 mm to (29.7, 25.1)
- moved wht- 1.03 mm to (49.3, 25.1)
- moved D181 1.03 mm to (20.5, 19.6)
- moved D182 1.03 mm to (27.5, 19.6)
- moved D187 1.03 mm to (31.0, 19.6)
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Routing:
- net (no net): track 229.4 -> 232.3 mm
Other:
- board text removed: "JLCJLCJLCJLC"
