File: Toyota Satoshi Emblem/Stencil/Stencil.kicad_pcb (KiCad board)
At the start: 2 copper layers, 299.5 x 123.4 mm, 445 parts, among them J11 Letter Terminal, J12 Letter Terminal, J13 Letter Terminal, J14 Letter Terminal, J15 Letter Terminal, J16 Letter Terminal, J17 Power 1, J18 Power 2, J19 Raptor Terminal, J20 Raptor Terminal, J21 Serial 3, J22 Serial 2, J23 Raptor Terminal, J24 Serial 1, J25 Raptor Terminal, J26 Turn Sig., J27 Misc. Sig., J29 Power In, J30 Sensor Term., J31 Extra Access, Q1 IRLR7843, Q10 IRLR7843, Q11 IRLR7843, Q12 MMBT3904, Q13 IRLR7843, Q14 IRLR7843, Q15 IRLR7843, Q16 MMBT3904, Q17 IRLR7843, Q18 IRLR7843, Q19 IRLR7843, Q2 IRLR7843, Q20 IRLR7843, Q21 IRLR7843, Q22 MMBT3904, Q23 IRLR7843, Q24 MMBT3904, Q25 IRLR7843, Q26 IRLR7843, Q27 IRLR7843, Q28 IRLR7843, Q29 IRLR7843, Q3 IRLR7843, Q30 MMBT3904, Q31 IRLR7843, Q32 MMBT3904, Q33 IRLR7843, Q34 IRLR7843, Q35 IRLR7843, Q36 MMBT3904, Q37 IRLR7843, Q38 IRLR7843, Q39 IRLR7843, Q4 MMBT3904, Q40 MMBT3904, Q41 IRF4905, Q42 IRF4905, Q43 BC327, Q44 BC337, Q5 IRLR7843, Q6 IRLR7843, Q7 IRLR7843, Q8 MMBT3904, Q9 IRLR7843, SW1 SW_DIP_x10, U1 MEGA_PRO_EMBED_CH340G_{slash}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, U2 L7805

Commit message: FIC initial
major overhaul, new beginnings
Parts:
- added 7V+: Pad 2, afootprints:Pad 2, F.Cu at (261.2, 113.3)
- added D145: WLED, afootprints:5730 LED W, F.Cu at (255.8, 135.7)
- added D146: WLED, afootprints:5730 LED W, F.Cu at (255.8, 128.7)
- added D147: WLED, afootprints:5730 LED W, F.Cu at (255.8, 114.7)
- added D148: WLED, afootprints:5730 LED W, F.Cu at (255.8, 121.7)
- added D149: WLED, afootprints:5730 LED W, F.Cu at (255.8, 107.7)
- added D150: WLED, afootprints:5730 LED W, F.Cu at (255.8, 100.7)
- added D151: ALED, afootprints:5730 LED A, F.Cu at (255.8, 125.2)
- added D152: ALED, afootprints:5730 LED A, F.Cu at (255.8, 132.2)
- added D153: ALED, afootprints:5730 LED A, F.Cu at (255.8, 111.2)
- added D154: ALED, afootprints:5730 LED A, F.Cu at (255.8, 118.2)
- added D155: ALED, afootprints:5730 LED A, F.Cu at (256.0, 97.2)
- added D156: ALED, afootprints:5730 LED A, F.Cu at (255.8, 104.2)
- added R73: 4.7, afootprints:1206 R, F.Cu at (261.3, 136.2)
- added R74: 4.7, afootprints:1206 R, F.Cu at (261.3, 126.5)
- added R75: 4.7, afootprints:1206 R, F.Cu at (261.0, 97.5)
- added R76: 4.7, afootprints:1206 R, F.Cu at (261.2, 131.3)
- added R77: 4.7, afootprints:1206 R, F.Cu at (260.6, 102.2)
- added R78: 4.7, afootprints:1206 R, F.Cu at (260.3, 94.0)
- added REF**: M2.5_Mechanical, afootprints:M2.5_Mechanical, F.Cu at (256.0, 139.8)
- added REF**: M2.5_Mechanical, afootprints:M2.5_Mechanical, F.Cu at (256.0, 93.0)
- added amb-: Pad 2, afootprints:Pad 2, F.Cu at (261.2, 119.6)
- added wht-: Pad 2, afootprints:Pad 2, F.Cu at (261.2, 106.7)
- moved R76 7.27 mm to (240.3, 131.3)
- moved 7V+ 7.27 mm to (240.3, 113.3)
- moved D155 7.27 mm to (235.1, 97.2)
- moved R74 7.27 mm to (240.3, 126.5)
- moved R75 7.27 mm to (240.0, 97.5)
- moved REF** 7.27 mm to (235.1, 93.0)
- moved amb- 7.27 mm to (240.2, 119.6)
- moved R73 7.27 mm to (240.3, 136.2)
- moved REF** 7.27 mm to (235.1, 139.8)
- moved D147 7.27 mm to (234.9, 114.7)
- moved D148 7.27 mm to (234.9, 121.7)
- moved D149 7.27 mm to (234.9, 107.7)
- moved D150 7.27 mm to (234.9, 100.7)
- moved D153 7.27 mm to (234.9, 111.2)
- moved D154 7.27 mm to (234.9, 118.2)
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Routing:
- net (no net): track 10315.6 -> 10543.4 mm
Other:
- board size 299.5 x 123.4 mm -> 299.5 x 119.9 mm
- board text added: "MountingHole_2.2mm_M2"
