File: FIC Board/FIC Board/power_board.kicad_sch (KiCad schematic)
At the start: 110 parts, among them J4 Conn_01x12_Male, J5 Conn_01x08_Male, Q41 IRF4905, Q42 BC327, Q43 BC337, Q44 IRF4905, U2 LM2596S-ADJ, U3 LM2596S-ADJ, U4 LM2596S-ADJ, U5 LM2596S-ADJ, U6 L7805

Commit message: recent updates
Parts:
- removed C10, C11, C12, C6, C7, C8: 100n, Capacitor_SMD:C_0603_1608Metric, symbol Device:C
- removed C14, C15, C16: 220u, Capacitor_SMD:CP_Elec_8x10, symbol Device:C_Polarized
- removed C2, C3, C4: 100u, Capacitor_SMD:CP_Elec_8x10, symbol Device:C_Polarized
- removed D14, D15, D16: SS34, Diode_SMD:D_SMA, symbol Device:D_Schottky
- removed D19, D20, D21: Red LED, LED_SMD:LED_0603_1608Metric, symbol Device:LED
- removed D? (x2): LED, eval-board-1_buck-regulator:CAPACITOR_0603N, symbol Device:LED
- removed J?: Conn_01x02, eval-board-1_buck-regulator:1935776, symbol Connector_Generic:Conn_01x02
- removed L2, L3, L4: 47u, FIC Board-footprints:L_12x12mm_H8mm, symbol Device:L
- removed R58, R59, R60, R66, R67, R68: 10k, Resistor_SMD:R_0603_1608Metric, symbol Device:R
- removed R62, R63: 270, Resistor_SMD:R_0603_1608Metric, symbol Device:R
- removed R? (x2): 10K, eval-board-1_buck-regulator:CAPACITOR_0402N, symbol Device:R_US
- removed R?: 510, eval-board-1_buck-regulator:CAPACITOR_0402N, symbol Device:R_US
- removed R?: 220, eval-board-1_buck-regulator:CAPACITOR_0402N, symbol Device:R_US
- removed R?: 8.87K, eval-board-1_buck-regulator:CAPACITOR_0402N, symbol Device:R_US
- removed RV3, RV4: 10k, Potentiometer_THT:Potentiometer_Bourns_3296X_Horizontal, symbol Device:R_Potentiometer
- removed U3, U4, U5: LM2596S-ADJ, Package_TO_SOT_SMD:TO-263-5_TabPin3, symbol Regulator_Switching:LM2596S-ADJ
- added C? (x2): GRM188R61H225ME11D, eval-board-1_buck-regulator:CAPACITOR_0603N, symbol Device:C
- added D14: Red LED, LED_SMD:LED_0603_1608Metric, symbol Device:LED
- added FB1: 74279221100, Inductor_SMD:L_1206_3216Metric_Pad1.22x1.90mm_HandSolder, symbol Device:Ferrite_Bead
- added R58: 1k, Resistor_SMD:R_0402_1005Metric, symbol Device:R_US
- FB2: renamed from FB?; footprint eval-board-1_buck-regulator:CAPACITOR_1206N -> Inductor_SMD:L_1206_3216Metric_Pad1.22x1.90mm_HandSolder
- R59, R60, R62, R63, R68: renamed from R?; footprint eval-board-1_buck-regulator:CAPACITOR_0402N -> Resistor_SMD:R_0402_1005Metric
- R64: value 270 -> 1k
- R69: value 10k -> 1k
- gave numbers to parts that had none: 24
Connections:
- net +5V is gone; now on net BUCK~: C25.1, C26.1, C27.1, C28.1, L2.2
- net EN_D~ is gone; now on net BUCK_A~: J5.8 (Pin_8)
- net 12V~: now also R64.2, C?.1, C?.1, FB1.1
- net EN_A~: no longer J5.5 (Pin_5)
- net GND: now also R58.2; no longer C1.2, C13.2, C14.2, C16.2, C17.2, C18.2, C19.2, C2.2, C20.2, C21.2, C25.2, C26.2, C27.2, C28.2, C3.2, C4.2, C5.2, C6.2, C9.2, D13.2 (A), D17.2 (A2), D22.1 (K), D23.2 (A), D24.2 (A), J4.1 (Pin_1), J4.2 (Pin_2), J4.3 (Pin_3), J4.4 (Pin_4), JP1.1, R57.1, R60.2, R61.1, R62.2, R64.1, R65.2, R74.2, U2.3 (GND), U3.16 (AGND), U3.32 (PGND), U3.33 (PGND), U3.7 (AGND), U6.2 (GND)
- net GND~: now reaches U3.11 (VSEN-)
- net GND~: now also C1.2, C13.2, C14.2, C16.2, C17.2, C18.2, C19.2, C2.2, C20.2, C21.2, C25.2, C26.2, C27.2, C28.2, C3.2, C4.2, C5.2, C6.2, C9.2, D13.2 (A), D17.2 (A2), D22.1 (K), D23.2 (A), D24.2 (A), J4.1 (Pin_1), J4.2 (Pin_2), J4.3 (Pin_3), J4.4 (Pin_4), JP1.1, R57.1, R60.2, R61.1, R62.2, R65.2, R74.2, U2.3 (GND), U3.16 (AGND), U3.32 (PGND), U3.33 (PGND), U3.7 (AGND), U6.2 (GND), C?.2, C?.2, D14.1 (K)
- net BUCK~: now reaches U3.12 (VSEN+)
- net BUCK~: now also R69.2
- net VSET: now reaches U3.15 (VSET)
- net VSET: now also RV2.2
- net at RV2.1: now also R58.1
- net +12V: no longer names the net of C2.1, FB2.1
- net +12V: now also FB1.2
- removed net BUCK_B~: J5.2 (Pin_2), RV2.2, RV2.3
- net BUCK_C~: no longer names the net of J5.3 (Pin_3)
- net BUCK_D~: no longer names the net of J5.4 (Pin_4)
- net BUCK_D~: no longer R69.2
- net EN_B~: no longer names the net of J5.6 (Pin_6)
- net EN_C~: no longer names the net of J5.7 (Pin_7)
- new net: D14.2 (A), R64.1
Other:
- moved on the sheet: C1, C10, C11, C12, C13, C14, C15, C16, C17, C18, C19, C2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
