File: FIC Board/FIC Board/FIC Board.kicad_pcb (KiCad board)
At the start: 2 copper layers, 184 x 94 mm, 186 parts, among them J1 superseal_connector, J2 Conn_01x12_Female, J3 Conn_01x08_Female, J4 Conn_01x12_Male, J5 Conn_01x08_Male, Q1 IRLR7843, Q10 MMBT3904, Q11 IRLR7843, Q12 IRLR7843, Q13 IRLR7843, Q14 IRLR7843, Q15 IRLR7843, Q16 IRLR7843, Q17 IRLR7843, Q18 IRLR7843, Q19 IRLR7843, Q2 IRLR7843, Q20 IRLR7843, Q21 IRLR7843, Q22 IRLR7843, Q23 IRLR7843, Q24 IRLR7843, Q25 IRLR7843, Q26 MMBT3904, Q27 MMBT3904, Q28 MMBT3904, Q29 MMBT3904, Q3 IRLR7843, Q30 MMBT3904, Q31 IRLR7843, Q32 IRLR7843, Q33 IRLR7843, Q34 IRLR7843, Q35 IRLR7843, Q36 IRLR7843, Q37 IRLR7843, Q38 IRLR7843, Q39 IRLR7843, Q4 IRLR7843, Q40 IRLR7843, Q41 IRF4905, Q42 BC327, Q43 BC337, Q44 IRF4905, Q5 IRLR7843, Q6 MMBT3904, Q7 MMBT3904, Q8 MMBT3904, Q9 MMBT3904, SW1 SW_DIP_x04, U1 MEGA_PRO_EMBED_CH340G_{slash}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, U2 LM2596S-ADJ, U3 LM2596S-ADJ, U4 LM2596S-ADJ, U5 LM2596S-ADJ, U6 L7805

Commit message: recent updates
Other:
- outline, holes or cut-outs redrawn
Changed lines of the file:
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@@
   (gr_line (start 125.074006 111.555993) (end 125.074006 72.306008) (layer "Cmts.User") (width 0.1))
   (gr_line (start 70.324002 72.306008) (end 70.324002 33.806009) (layer "Cmts.User") (width 0.1))
+  (gr_line (start 59.824 104.038763) (end 52.324012 104.038763) (layer "Cmts.User") (width 0.15))
+  (gr_line (start 59.824 104.038763) (end 59.812315 111.555993) (layer "Cmts.User") (width 0.15))
   (gr_line (start 70.324002 33.806009) (end 52.324012 33.806009) (layer "Cmts.User") (width 0.1))
-  (gr_line (start 52.324012 33.806009) (end 52.324012 111.555993) (layer "Cmts.User") (width 0.1))
-  (gr_line (start 52.324012 111.555993) (end 125.074006 111.555993) (layer "Cmts.User") (width 0.1))
+  (gr_line (start 52.324012 33.806009) (end 52.324012 104.038763) (layer "Cmts.User") (width 0.1))
+  (gr_line (start 59.812315 111.555993) (end 125.074006 111.555993) (layer "Cmts.User") (width 0.1))
   (gr_line (start 125.074006 72.306008) (end 70.324002 72.306008) (layer "Cmts.User") (width 0.1))
+  (gr_line (start 142.324 104.05103) (end 149.824 104.056) (layer "Edge.Cuts") (width 0.1))
   (gr_line (start 215.074 111.556) (end 215.074 72.306) (layer "Edge.Cuts") (width 0.1))
   (gr_line (start 160.324 72.306) (end 160.324 33.806) (layer "Edge.Cuts") (width 0.1))
-  (gr_line (start 142.324 111.556) (end 215.074 111.556) (layer "Edge.Cuts") (width 0.1))
+  (gr_line (start 149.814736 111.556) (end 215.074 111.556) (layer "Edge.Cuts") (width 0.1))
   (gr_line (start 125.054 25.806) (end 125.054 119.786) (layer "Edge.Cuts") (width 0.1))
-  (gr_line (start 142.324 33.806) (end 142.324 111.556) (layer "Edge.Cuts") (width 0.1))
+  (gr_line (start 142.324 33.806) (end 142.324 104.05103) (layer "Edge.Cuts") (width 0.1))
   (gr_line (start 160.324 33.806) (end 142.324 33.806) (layer "Edge.Cuts") (width 0.1))
   (gr_line (start 31.074 25.806) (end 31.074 119.786) (layer "Edge.Cuts") (width 0.1))
+  (gr_line (start 149.824 104.056) (end 149.814736 111.556) (layer "Edge.Cuts") (width 0.1))
   (gr_line (start 125.054 119.786) (end 31.074 119.786) (layer "Edge.Cuts") (width 0.1))
   (gr_line (start 215.074 72.306) (end 160.324 72.306) (layer "Edge.Cuts") (width 0.1))

Commit message: recent
Parts:
- removed D21, D22: Red LED, LED_SMD:LED_0603_1608Metric
- removed D23, D24: 1N4746A, Diode_THT:D_DO-41_SOD81_P10.16mm_Horizontal
- removed D25, D26: 1N4007, Diode_THT:D_DO-41_SOD81_P10.16mm_Horizontal
- removed D5: GRN LED, LED_SMD:LED_0603_1608Metric
- removed L2, L3, L4: 47u, FIC Board-footprints:L_12x12mm_H8mm
- removed Q43: BC337, Package_TO_SOT_THT:TO-92_Inline
- removed Q44: IRF4905, Package_TO_SOT_THT:TO-220-3_Vertical
- removed R74: 10k, Resistor_SMD:R_1206_3216Metric
- removed RV4: 10k, Potentiometer_THT:Potentiometer_Bourns_3296X_Horizontal
- removed U5: LM2596S-ADJ, Package_TO_SOT_SMD:TO-263-5_TabPin3
- removed U6: L7805, Package_TO_SOT_THT:TO-220-3_Horizontal_TabDown
- added C22: 47uF 50V, Capacitor_SMD:CP_Elec_6.3x5.9, F.Cu at (201.5, 98.1)
- added C23: 47uF 50V, Capacitor_SMD:CP_Elec_6.3x5.9, F.Cu at (209.0, 98.1)
- added C24: 47uF 50V, Capacitor_SMD:CP_Elec_6.3x5.9, F.Cu at (216.6, 98.1)
- added C25: 4.7u, Capacitor_SMD:C_0603_1608Metric, F.Cu at (200.9, 121.2)
- added C26: 1uF 25V, Capacitor_SMD:C_0603_1608Metric, F.Cu at (197.9, 119.8)
- added FB1: 74279221100, Inductor_SMD:L_1206_3216Metric_Pad1.22x1.90mm_HandSolder, F.Cu at (179.5, 100.5)
- added FB2: 74279221100, FIC Board-footprints:Wurth 742792903 L_12x12mm_H8mm, F.Cu at (190.1, 99.5)
- added H1: MountingHole_Pad, MountingHole:MountingHole_2.7mm_M2.5_Pad_TopBottom, F.Cu at (166.5, 57.8)
- added H10: MountingHole_Pad, MountingHole:MountingHole_2.2mm_M2_DIN965_Pad_TopOnly, F.Cu at (90.5, 136.6)
- added H11: MountingHole_Pad, MountingHole:MountingHole_2.2mm_M2_DIN965_Pad_TopOnly, F.Cu at (114.7, 136.6)
- added H2: MountingHole_Pad, MountingHole:MountingHole_2.7mm_M2.5_Pad_TopBottom, F.Cu at (76.5, 57.8)
- added H3: MountingHole_Pad, MountingHole:MountingHole_2.7mm_M2.5_Pad_TopBottom, F.Cu at (226.1, 127.8)
- added H4: MountingHole_Pad, MountingHole:MountingHole_2.7mm_M2.5_Pad_TopBottom, F.Cu at (136.1, 127.8)
- added H5: MountingHole, MountingHole:MountingHole_2.7mm_M2.5, F.Cu at (125.4, 82.9)
- added H6: MountingHole_Pad, MountingHole:MountingHole_2.2mm_M2_DIN965_Pad_TopOnly, F.Cu at (66.4, 49.0)
- added H7: MountingHole_Pad, MountingHole:MountingHole_2.2mm_M2_DIN965_Pad_TopOnly, F.Cu at (90.5, 49.0)
- added H8: MountingHole_Pad, MountingHole:MountingHole_2.2mm_M2_DIN965_Pad_TopOnly, F.Cu at (114.7, 49.0)
- added H9: MountingHole_Pad, MountingHole:MountingHole_2.2mm_M2_DIN965_Pad_TopOnly, F.Cu at (66.4, 136.6)
- added J6: Conn_02x02_Odd_Even, FIC Board-footprints:Male_2x2_Conn, F.Cu at (194.2, 124.8)
- added J7: Conn_02x03_Odd_Even, FIC Board-footprints:Female_3x2_Conn, F.Cu at (135.8, 106.3)
- added JP1: Jumper_2_Bridged, FIC Board-footprints:MaleHeader_1x2_conn, F.Cu at (200.8, 126.6)
- added TP1: TestPoint, TestPoint:TestPoint_Pad_1.0x1.0mm, F.Cu at (195.0, 108.9)
- added TP2: TestPoint, TestPoint:TestPoint_Pad_1.0x1.0mm, F.Cu at (202.4, 123.8)
- C1: value 100u -> 0.1u 50V; footprint Capacitor_SMD:CP_Elec_8x10 -> Capacitor_THT:C_Disc_D4.7mm_W2.5mm_P5.00mm
- C10, C11, C12, C20, C7, C8, C9: value 100n -> 22uF 25V; footprint Capacitor_SMD:C_0603_1608Metric -> Capacitor_SMD:C_1210_3225Metric
- C13, C14: value 220u -> 2.2uF 50V; footprint Capacitor_SMD:CP_Elec_8x10 -> Capacitor_SMD:C_0603_1608Metric
- C15, C16: value 220u -> 22uF 25V; footprint Capacitor_SMD:CP_Elec_8x10 -> Capacitor_SMD:C_1210_3225Metric
- C17: value 0.1u 50V -> 22uF 25V; footprint Capacitor_THT:C_Disc_D4.7mm_W2.5mm_P5.00mm -> Capacitor_SMD:C_1210_3225Metric
- C18: value 47u 50V -> 47uF 50V; footprint Capacitor_THT:CP_Radial_D6.3mm_P2.50mm -> Capacitor_SMD:CP_Elec_6.3x5.9
- C19: value 10u 25V -> 2.2uF 50V; footprint Capacitor_THT:CP_Radial_D4.0mm_P2.00mm -> Capacitor_SMD:C_0603_1608Metric
- C2, C3: value 100u -> 47uF 50V; footprint Capacitor_SMD:CP_Elec_8x10 -> Capacitor_SMD:CP_Elec_6.3x5.9
- C21: value 100n -> 2.2uF 50V
- C4: value 100u -> KGM15BR51E224KT; footprint Capacitor_SMD:CP_Elec_8x10 -> Capacitor_SMD:C_0603_1608Metric; moved to B.Cu
- C5: value 100n -> CL10B104KO8NNNC; moved to B.Cu
- C6: value 100n -> 0.1uF
- D1: value LL34 5.1V -> Diode_SMD:D_MiniMELF
- D10: value LL34 5.1V -> 2.0V 20mA GRN 0603; footprint Diode_SMD:D_MiniMELF -> LED_SMD:LED_0603_1608Metric
- D11: value RED LED -> 2.1V 20mA YLW 0603
- D12: value RED LED -> 2.0V 20mA GRN 0603
- D13: value SS34 -> 2.0V 20mA RED 0603; footprint Diode_SMD:D_SMA -> LED_SMD:LED_0603_1608Metric
- D14: value SS34 -> 10V Zener SOD-80; footprint Diode_SMD:D_SMA -> Diode_SMD:D_MiniMELF; moved to B.Cu
- D15, D16: value SS34 -> ~; footprint Diode_SMD:D_SMA -> LED_SMD:LED_0603_1608Metric
- D18: value 1N47xxA -> 1N4148W-13-F; footprint Diode_THT:D_DO-41_SOD81_P10.16mm_Horizontal -> Diode_SMD:D_SOD-123
- D19: value Red LED -> 2.4V Zener SOD-80; footprint LED_SMD:LED_0603_1608Metric -> Diode_SMD:D_MiniMELF
- D2: value LL34 5.1V -> 4.7V Zener SOD-80
- D20: value Red LED -> 1N4148W-13-F; footprint LED_SMD:LED_0603_1608Metric -> Diode_SMD:D_SOD-123
- D3: value GRN LED -> 4.7V Zener SOD-80; footprint LED_SMD:LED_0603_1608Metric -> Diode_SMD:D_MiniMELF
- D4: value YLW LED -> 4.7V Zener SOD-80; footprint LED_SMD:LED_0603_1608Metric -> Diode_SMD:D_MiniMELF
- D6, D8: value YLW LED -> 2.1V 20mA YLW 0603
- D7: value GRN LED -> 2.0V 20mA GRN 0603
- D9: value LL34 5.1V -> 2.0V 20mA RED 0603; footprint Diode_SMD:D_MiniMELF -> LED_SMD:LED_0603_1608Metric
- F1: value 10A Fuse -> 3557-2; footprint afootprints:Univ_AUTO_Fuse -> FIC Board-footprints:Univ_AUTO_Fuse
- J1: value superseal_connector -> 6437288-3
- J2: value Conn_01x12_Female -> Conn_02x03_Odd_Even; footprint Connector_PinSocket_2.54mm:PinSocket_1x12_P2.54mm_Vertical -> FIC Board-footprints:Male_3x2_Conn
- J3: value Conn_01x08_Female -> Conn_02x03_Odd_Even; footprint Connector_PinSocket_2.54mm:PinSocket_1x08_P2.54mm_Vertical -> FIC Board-footprints:Male_3x2_Conn
- J4: value Conn_01x12_Male -> ~; footprint Connector_PinHeader_2.54mm:PinHeader_1x12_P2.54mm_Vertical -> FIC Board-footprints:Female_3x2_Conn
- J5: value Conn_01x08_Male -> Conn_02x02_Odd_Even; footprint Connector_PinHeader_2.54mm:PinHeader_1x08_P2.54mm_Vertical -> FIC Board-footprints:Female_2x2_Conn
- L1: value 47u -> SRP1265C-1R0M; footprint FIC Board-footprints:L_12x12mm_H8mm -> FIC Board-footprints:INDPM135126X650N
- Q1, Q11, Q13, Q15, Q17, Q18, Q19, Q2, Q20, Q21, Q23, Q25, Q3, Q33, Q4, Q5: footprint afootprints:IRLR7843 -> Package_TO_SOT_SMD:TO-252-2
- Q10: footprint afootprints:2N3904SMD -> Package_TO_SOT_SMD:SOT-23
- Q12, Q14, Q16, Q22, Q24, Q34: value IRLR7843 -> MMBT3904; footprint afootprints:IRLR7843 -> Package_TO_SOT_SMD:SOT-23
- Q26, Q7, Q8, Q9: value MMBT3904 -> IRLR7843; footprint afootprints:2N3904SMD -> Package_TO_SOT_SMD:TO-252-2
- Q27, Q28, Q29, Q30: value MMBT3904 -> IRLR7843; footprint afootprints:2N3904SMD -> Package_TO_SOT_SMD:TO-252-2; moved to B.Cu
- Q31, Q32, Q35, Q37, Q39: footprint afootprints:IRLR7843 -> Package_TO_SOT_SMD:TO-252-2; moved to B.Cu
- Q36, Q38, Q40: value IRLR7843 -> MMBT3904; footprint afootprints:IRLR7843 -> Package_TO_SOT_SMD:SOT-23; moved to B.Cu
- Q41: footprint Package_TO_SOT_THT:TO-220-3_Vertical -> Package_TO_SOT_SMD:TO-263-2; moved to B.Cu
- Q42: value BC327 -> IRF4905; footprint Package_TO_SOT_THT:TO-92_Inline -> Package_TO_SOT_SMD:TO-263-2
- Q6: value MMBT3904 -> IRLR7843; footprint Package_TO_SOT_SMD:SOT-23 -> Package_TO_SOT_SMD:TO-252-2
- R1, R11, R12, R13, R14, R15, R16, R17, R18, R19, R2, R20, R27, R3, R34, R4, R5, R6: value 10k -> 1KΩ 0603; footprint Resistor_SMD:R_1206_3216Metric -> Resistor_SMD:R_0603_1608Metric
- R10, R39, R44, R7, R8, R9: value 10k -> 10KΩ 0603; footprint Resistor_SMD:R_1206_3216Metric -> Resistor_SMD:R_0603_1608Metric
- R21, R22, R23, R24, R29, R33, R37, R38, R40, R41, R42, R43, R45, R46, R47, R50, R73: value 1k -> 10KΩ 0603; footprint Resistor_SMD:R_1206_3216Metric -> Resistor_SMD:R_0603_1608Metric
- R25, R26, R28, R30, R31, R32, R35, R36, R72: value 1k -> 1KΩ 0603; footprint Resistor_SMD:R_1206_3216Metric -> Resistor_SMD:R_0603_1608Metric
- R48, R49, R58, R67, R69: value 10k -> 10KΩ 0603
- R51: value 1k -> 10KΩ 0603
- R52, R53, R54, R55: value 1k -> 10KΩ 0603; moved to B.Cu
- R56: value 1k -> 8.87K; moved to B.Cu
- R57: value 10k -> 10KΩ 0603; moved to B.Cu
- R59, R60: value 10k -> 5.11KΩ
- R61, R64: value 270 -> 1KΩ 0603
- R62: value 270 -> 10K
- R63: value 270 -> 10KΩ 0603; moved to B.Cu
- R65: value 10k -> 100KΩ 0603; footprint Resistor_SMD:R_1206_3216Metric -> Resistor_SMD:R_0603_1608Metric
- R66: value 10k -> 100KΩ 0603
- R68: value 10k -> 2.2Ω
- R70, R71: value 1k -> 8.87KΩ; footprint Resistor_SMD:R_1206_3216Metric -> Resistor_SMD:R_0603_1608Metric
- SW1: value SW_DIP_x04 -> SW_DIP_04
- U1: footprint afootprints:MODULE_MEGA_PRO_EMBED_CH340G___ATMEGA2560 -> FIC Board-footprints:MODULE_MEGA_PRO_EMBED_CH340G___ATMEGA2560
- U2: value LM2596S-ADJ -> LM393DR; footprint Package_TO_SOT_SMD:TO-263-5_TabPin3 -> Package_SO:SOIC-8_3.9x4.9mm_P1.27mm; moved to F.Cu
- U3: value LM2596S-ADJ -> L7805CV; footprint Package_TO_SOT_SMD:TO-263-5_TabPin3 -> Package_TO_SOT_THT:TO-220-3_Horizontal_TabDown; moved to F.Cu
- U4: value LM2596S-ADJ -> SIC453ED-T1-GE3; footprint Package_TO_SOT_SMD:TO-263-5_TabPin3 -> FIC Board-footprints:SiC45X; moved to F.Cu
- moved D9 379.6 mm to (167.4, 110.7), turned to 180 degrees
- moved R37 362.2 mm to (227.0, 116.5)
- moved Q11 323.6 mm to (112.0, 126.8), turned to 180 degrees
- moved Q24 309.4 mm to (88.2, 118.6)
- moved Q1 305.9 mm to (125.4, 95.9)
- moved R33 305.1 mm to (164.0, 110.7)
- moved Q12 300.7 mm to (116.8, 121.5)
- moved Q36 296.6 mm to (118.6, 103.1), turned to 180 degrees
- moved Q38 295.3 mm to (86.4, 124.4), turned to 180 degrees
- moved Q13 293.5 mm to (94.8, 125.2), turned to 90 degrees
- moved Q16 292.3 mm to (114.9, 112.9)
- moved Q3 292.1 mm to (125.3, 118.1)
- moved R25 291.8 mm to (115.5, 61.1), turned to 90 degrees
- moved Q4 291.7 mm to (125.3, 125.4)
- moved Q35 291.7 mm to (113.1, 103.5), turned to 90 degrees
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Connections:
- C1 pad 1: 12V~ -> Net-(D14-K)
- C10 pad 1: BUCK_B~ -> /POWER/VIN
- C11 pad 1: BUCK_C~ -> /POWER/VIN
- C12 pad 1: BUCK_D~ -> /POWER/VIN
- C13 pad 1: BUCK_A~ -> /POWER/VIN
- C14 pad 1: BUCK_B~ -> /POWER/VIN
- C15 pad 1: BUCK_C~ -> BUCK~
- C16 pad 1: BUCK_D~ -> BUCK~
- C17 pad 1: Net-(C17-Pad1) -> BUCK~
- C18 pad 1: Net-(C17-Pad1) -> BUCK~
- C19 pad 1: 12V~ -> FIL12V~
- C2 pad 1: 12V~ -> Net-(D14-K)
- C20 pad 1: 12V~ -> Net-(C20-Pad1)
- C21 pad 1: 5V~ -> /POWER/VIN
- C3 pad 1: 12V~ -> Net-(D14-K)
- C4 pad 1: 12V~ -> BATGND
- C4 pad 2: GND~ -> LET_C1
- C5 pad 1: 12V~ -> BATGND
- C5 pad 2: GND~ -> LGHT_P
- C6 pad 1: 12V~ -> Net-(U4-BOOT)
- C6 pad 2: GND~ -> Net-(C6-Pad2)
- C7 pad 1: 12V~ -> /POWER/VIN
- C8 pad 1: 12V~ -> /POWER/VIN
- C9 pad 1: BUCK_A~ -> /POWER/VIN
- D10 pad 1: MISC_2_FIL -> RX_2
- D10 pad 2: BATGND -> Net-(D10-A)
- D11 pad 1: BATGND -> TX_3
- D11 pad 2: Net-(D11-Pad2) -> Net-(D11-A)
- D12 pad 1: BATGND -> RX_3
- D12 pad 2: Net-(D12-Pad2) -> Net-(D12-A)
- D13 pad 1: Net-(D13-Pad1) -> GND~
- D13 pad 2: GND~ -> Net-(D13-A)
- D14 pad 1: Net-(D14-Pad1) -> Net-(D14-K)
- D14 pad 2: GND~ -> Net-(D14-A)
- D15 pad 1: Net-(D15-Pad1) -> Net-(D15-K)
- D15 pad 2: GND~ -> Net-(D15-A)
- D16 pad 1: Net-(D16-Pad1) -> Net-(D16-K)
- D16 pad 2: GND~ -> Net-(D16-A)
- D17 pad 1: VCC~ -> FUS12V~
- D18 pad 1: Net-(C17-Pad1) -> Net-(D18-K)
- D18 pad 2: Net-(D18-Pad2) -> Net-(D15-K)
- D19 pad 1: GND~ -> Net-(D19-K)
- D19 pad 2: Net-(D19-Pad2) -> GND~
- D20 pad 1: GND~ -> Net-(D18-K)
- D20 pad 2: Net-(D20-Pad2) -> Net-(D16-K)
- D3 pad 1: Net-(D3-Pad1) -> MISC_1_FIL
- D3 pad 2: +5V -> BATGND
- D4 pad 1: Net-(D4-Pad1) -> MISC_2_FIL
- D4 pad 2: +5V -> BATGND
- D6 pad 1: Net-(D6-Pad1) -> TX_1
- D6 pad 2: +5V -> Net-(D6-A)
- D7 pad 1: Net-(D7-Pad1) -> RX_1
- D7 pad 2: +5V -> Net-(D7-A)
- D8 pad 1: Net-(D8-Pad1) -> TX_2
- D8 pad 2: +5V -> Net-(D8-A)
- D9 pad 1: MISC_1_FIL -> GND~
- D9 pad 2: BATGND -> Net-(D9-A)
- F1 pad 1: BATGND -> RLY87
- F1 pad 2: VCC -> FUS12V
- J1 pad 10: RAP_A1 -> LET_W1
- J1 pad 11: RAP_W1 -> LET_W2
- J1 pad 12: BUCK_D -> LET_W3
- J1 pad 13: LGHT_P -> LET_W4
- J1 pad 14: LGHT_N -> LET_W5
- J1 pad 15: RAP_A2 -> LET_W6
- J1 pad 16: RAP_W2 -> RAP_W1
- J1 pad 17: BUCK_D -> RAP_W2
- J1 pad 18: RAP_A3 -> RAP_W3
- J1 pad 19: RAP_W3 -> RAP_W4
- J1 pad 2: LET_W1 -> LET_A2
- J1 pad 20: BUCK_D -> RAP_A4
- J1 pad 21: LGHT_S -> LET_C1
- J1 pad 23: RAP_A4 -> BATGND
- J1 pad 24: RAP_W4 -> LGHT_P
- J1 pad 25: BUCK_D -> LGHT_S
- J1 pad 26: LET_A4 -> LET_C1
- J1 pad 27: LET_W4 -> LET_C1
- J1 pad 28: BUCK_B -> LET_C1
- J1 pad 29: LET_A5 -> LET_C1
- J1 pad 3: BUCK_A -> LET_A3
- J1 pad 30: LET_W5 -> LET_C1
- J1 pad 31: BUCK_C -> LET_C1
- J1 pad 32: LET_A6 -> LET_C1
- J1 pad 33: BUCK_C -> LET_C1
- J1 pad 34: LET_W6 -> LET_C1
- J1 pad 35: BAT12V -> TURN_D
- J1 pad 36: BATGND -> RX_1
- J1 pad 37: HEDRLY -> TX_1
- J1 pad 38: HEDRLY -> TX_2
- J1 pad 39: RLY87 -> RX_2
- J1 pad 4: LET_A2 -> LET_A4
- J1 pad 40: TX_1 -> FIL12V
- J1 pad 41: RX_1 -> BATGND
- J1 pad 42: BAT12V -> TURN_P
- J1 pad 43: BATGND -> unconnected-(J1-Pad43)
- J1 pad 44: RLY87A -> TX_3
- J1 pad 45: unconnected-(J1-Pad45) -> RX_3
- J1 pad 46: unconnected-(J1-Pad46) -> FIL12V
- J1 pad 47: unconnected-(J1-Pad47) -> BATGND
- J1 pad 48: TURN_D -> MISC_1
- J1 pad 49: TURN_P -> SDA
- J1 pad 5: LET_W2 -> LET_A5
- J1 pad 50: MISC_1 -> SCL
- J1 pad 51: MISC_2 -> HEDRLY
- J1 pad 52: unconnected-(J1-Pad52) -> BAT12V
- J1 pad 53: RX_3 -> BATGND
- J1 pad 54: 12V -> MISC_2
- J1 pad 55: BATGND -> unconnected-(J1-Pad55)
- J1 pad 56: TX_2 -> RLY87A
- J1 pad 57: RX_2 -> HEDRLY
- J1 pad 58: 12V -> BAT12V
- J1 pad 6: BUCK_A -> LET_A6
- J1 pad 60: TX_3 -> RLY87
- J1 pad 7: LET_A3 -> RAP_A1
- J1 pad 8: LET_W3 -> RAP_A2
- J1 pad 9: BUCK_B -> RAP_A3
- J2 pad 1: BATGND -> FUS12V~
- J2 pad 2: BATGND -> FIL12V~
- J2 pad 3: BATGND -> FUS12V~
- J2 pad 4: BATGND -> FIL12V~
- J2 pad 5: VCC -> FUS12V~
- J2 pad 6: VCC -> FIL12V~
- J3 pad 1: BUCK_A -> GND~
- J3 pad 2: BUCK_B -> BUCK~
- J3 pad 3: BUCK_C -> GND~
- J3 pad 4: BUCK_D -> BUCK~
- J3 pad 5: EN_A -> GND~
- J3 pad 6: EN_B -> BUCK~
- J4 pad 1: GND~ -> FUS12V
- J4 pad 2: GND~ -> FIL12V
- J4 pad 3: GND~ -> FUS12V
- J4 pad 4: GND~ -> FIL12V
- J4 pad 5: VCC~ -> FUS12V
- J4 pad 6: VCC~ -> FIL12V
- J5 pad 1: BUCK_A~ -> SDA
- J5 pad 2: BUCK_B~ -> PGOOD
- J5 pad 3: BUCK_C~ -> SCL
- J5 pad 4: BUCK_D~ -> SALRT
- L1 pad 1: Net-(D13-Pad1) -> /POWER/SW
- L1 pad 2: BUCK_A~ -> BUCK~
- Q1 pad 1: Net-(Q1-Pad1) -> LET_COLOR1
- Q1 pad 2: LET_A1 -> LET_W1
- Q1 pad 3: Net-(Q1-Pad3) -> Net-(Q1-S)
- Q10 pad 1: Net-(Q10-Pad1) -> Net-(Q10-B)
- Q10 pad 3: Net-(Q10-Pad3) -> Net-(Q10-C)
- Q11 pad 1: LET_POWER1 -> LET_POWER2
- Q11 pad 2: Net-(Q1-Pad3) -> Net-(Q11-D)
- Q12 pad 1: LET_POWER2 -> Net-(Q12-B)
- Q12 pad 2: Net-(Q12-Pad2) -> BATGND
- Q12 pad 3: BATGND -> Net-(Q12-C)
- Q13 pad 2: Net-(Q13-Pad2) -> Net-(Q13-D)
- Q14 pad 1: LET_POWER4 -> Net-(Q14-B)
- Q14 pad 2: Net-(Q14-Pad2) -> BATGND
- Q14 pad 3: BATGND -> Net-(Q14-C)
- Q15 pad 1: LET_POWER5 -> LET_POWER4
- Q15 pad 2: Net-(Q15-Pad2) -> Net-(Q15-D)
- Q16 pad 1: LET_COLOR1 -> Net-(Q16-B)
- Q16 pad 2: LET_W1 -> BATGND
- Q16 pad 3: Net-(Q1-Pad3) -> Net-(Q16-C)
- Q17 pad 1: LET_COLOR2 -> LET_COLOR5
- Q17 pad 2: LET_W2 -> LET_W5
- Q17 pad 3: Net-(Q12-Pad2) -> Net-(Q17-S)
- Q18 pad 1: LET_COLOR3 -> Net-(Q18-G)
- Q18 pad 2: LET_W3 -> LET_A5
- Q18 pad 3: Net-(Q13-Pad2) -> Net-(Q17-S)
- Q19 pad 1: LET_COLOR4 -> LET_COLOR6
- Q19 pad 2: LET_W4 -> LET_W6
- Q19 pad 3: Net-(Q14-Pad2) -> Net-(Q19-S)
- Q2 pad 1: Net-(Q2-Pad1) -> Net-(Q10-C)
- Q2 pad 2: LET_A2 -> LET_A1
- Q2 pad 3: Net-(Q12-Pad2) -> Net-(Q1-S)
- Q20 pad 1: LET_COLOR5 -> Net-(Q20-G)
- Q20 pad 2: LET_W5 -> LET_A6
- Q20 pad 3: Net-(Q15-Pad2) -> Net-(Q19-S)
- Q21 pad 1: Net-(Q21-Pad1) -> LET_POWER5
- Q21 pad 2: LET_A6 -> Net-(Q17-S)
- Q21 pad 3: Net-(Q21-Pad3) -> BATGND
- Q22 pad 1: Net-(Q22-Pad1) -> Net-(Q22-B)
- Q22 pad 2: RAP_A1 -> BATGND
- Q22 pad 3: Net-(Q22-Pad3) -> Net-(Q18-G)
- Q23 pad 1: Net-(Q23-Pad1) -> LET_POWER6
- Q23 pad 2: RAP_A2 -> Net-(Q19-S)
- Q23 pad 3: Net-(Q23-Pad3) -> BATGND
- Q24 pad 1: Net-(Q24-Pad1) -> Net-(Q24-B)
- Q24 pad 2: RAP_A3 -> BATGND
- Q24 pad 3: Net-(Q24-Pad3) -> Net-(Q20-G)
- Q25 pad 1: Net-(Q25-Pad1) -> RAP_COLOR1
- Q25 pad 2: RAP_A4 -> RAP_W1
- Q25 pad 3: Net-(Q25-Pad3) -> Net-(Q25-S)
- Q26 pad 1: Net-(Q26-Pad1) -> Net-(Q26-G)
- Q26 pad 2: BATGND -> RAP_A1
- Q26 pad 3: Net-(Q21-Pad1) -> Net-(Q25-S)
- Q27 pad 1: Net-(Q27-Pad1) -> RAP_COLOR2
- Q27 pad 2: BATGND -> RAP_W2
- Q27 pad 3: Net-(Q22-Pad1) -> Net-(Q27-S)
- Q28 pad 1: Net-(Q28-Pad1) -> Net-(Q28-G)
- Q28 pad 2: BATGND -> RAP_A2
- Q28 pad 3: Net-(Q23-Pad1) -> Net-(Q27-S)
- Q29 pad 1: Net-(Q29-Pad1) -> RAP_COLOR3
- Q29 pad 2: BATGND -> RAP_W3
- Q29 pad 3: Net-(Q24-Pad1) -> Net-(Q29-S)
- Q3 pad 1: Net-(Q3-Pad1) -> LET_COLOR2
- Q3 pad 2: LET_A3 -> LET_W2
- Q3 pad 3: Net-(Q13-Pad2) -> Net-(Q11-D)
- Q30 pad 1: Net-(Q30-Pad1) -> Net-(Q30-G)
- Q30 pad 2: BATGND -> RAP_A3
- Q30 pad 3: Net-(Q25-Pad1) -> Net-(Q29-S)
- Q31 pad 1: LET_POWER6 -> RAP_COLOR4
- Q31 pad 2: Net-(Q21-Pad3) -> RAP_W4
- Q31 pad 3: BATGND -> Net-(Q31-S)
- Q32 pad 1: RAP_POWER1 -> Net-(Q32-G)
- Q32 pad 2: Net-(Q22-Pad3) -> RAP_A4
- Q32 pad 3: BATGND -> Net-(Q31-S)
- Q33 pad 1: RAP_POWER2 -> RAP_POWER1
- Q33 pad 2: Net-(Q23-Pad3) -> Net-(Q25-S)
- Q34 pad 1: RAP_POWER3 -> Net-(Q34-B)
- Q34 pad 2: Net-(Q24-Pad3) -> BATGND
- Q34 pad 3: BATGND -> Net-(Q26-G)
- Q35 pad 1: RAP_POWER4 -> RAP_POWER2
- Q35 pad 2: Net-(Q25-Pad3) -> Net-(Q27-S)
- Q36 pad 1: LET_COLOR6 -> Net-(Q36-B)
- Q36 pad 2: LET_W6 -> BATGND
- Q36 pad 3: Net-(Q21-Pad3) -> Net-(Q28-G)
- Q37 pad 1: RAP_COLOR1 -> RAP_POWER3
- Q37 pad 2: RAP_W1 -> Net-(Q29-S)
- Q37 pad 3: Net-(Q22-Pad3) -> BATGND
- Q38 pad 1: RAP_COLOR2 -> Net-(Q38-B)
- Q38 pad 2: RAP_W2 -> BATGND
- Q38 pad 3: Net-(Q23-Pad3) -> Net-(Q30-G)
- Q39 pad 1: RAP_COLOR3 -> RAP_POWER4
- Q39 pad 2: RAP_W3 -> Net-(Q31-S)
- Q39 pad 3: Net-(Q24-Pad3) -> BATGND
- Q4 pad 1: Net-(Q4-Pad1) -> Net-(Q12-C)
- Q4 pad 2: LET_A4 -> LET_A2
- Q4 pad 3: Net-(Q14-Pad2) -> Net-(Q11-D)
- Q40 pad 1: RAP_COLOR4 -> Net-(Q40-B)
- Q40 pad 2: RAP_W4 -> BATGND
- Q40 pad 3: Net-(Q25-Pad3) -> Net-(Q32-G)
- Q41 pad 1: Net-(D18-Pad2) -> Net-(D14-A)
- Q41 pad 2: VCC~ -> FUS12V~
- Q41 pad 3: Net-(C17-Pad1) -> Net-(D14-K)
- Q42 pad 1: Net-(D26-Pad2) -> Net-(D18-K)
- Q42 pad 2: Net-(Q42-Pad2) -> FIL12V~
- Q42 pad 3: Net-(C17-Pad1) -> Net-(D14-K)
- Q5 pad 1: Net-(Q10-Pad3) -> LET_COLOR3
- Q5 pad 2: LET_A5 -> LET_W3
- Q5 pad 3: Net-(Q15-Pad2) -> Net-(Q13-D)
- Q6 pad 1: Net-(Q6-Pad1) -> Net-(Q14-C)
- Q6 pad 2: BATGND -> LET_A3
- Q6 pad 3: Net-(Q1-Pad1) -> Net-(Q13-D)
- Q7 pad 1: Net-(Q7-Pad1) -> LET_COLOR4
- Q7 pad 2: BATGND -> LET_W4
- Q7 pad 3: Net-(Q2-Pad1) -> Net-(Q15-D)
- Q8 pad 1: Net-(Q8-Pad1) -> Net-(Q16-C)
- Q8 pad 2: BATGND -> LET_A4
- Q8 pad 3: Net-(Q3-Pad1) -> Net-(Q15-D)
- Q9 pad 1: Net-(Q9-Pad1) -> LET_POWER1
- Q9 pad 2: BATGND -> Net-(Q1-S)
- Q9 pad 3: Net-(Q4-Pad1) -> BATGND
- R1 pad 1: Net-(Q1-Pad1) -> Net-(R1-Pad1)
- R1 pad 2: BUCK_A -> LET_COLOR1
- R10 pad 1: LET_COLOR5 -> MISC_2
- R10 pad 2: Net-(Q10-Pad1) -> MISC_2_FIL
- R11 pad 1: Net-(Q21-Pad1) -> Net-(R1-Pad1)
- R11 pad 2: BUCK_C -> LET_COLOR4
- R12 pad 1: Net-(Q22-Pad1) -> Net-(R12-Pad1)
- R12 pad 2: BUCK_D -> RAP_COLOR4
- R13 pad 1: Net-(Q23-Pad1) -> Net-(R1-Pad1)
- R13 pad 2: BUCK_D -> LET_COLOR5
- R14 pad 1: Net-(Q24-Pad1) -> Net-(R1-Pad1)
- R14 pad 2: BUCK_D -> LET_COLOR6
- R15 pad 1: Net-(Q25-Pad1) -> Net-(R15-Pad1)
- R15 pad 2: BUCK_D -> LET_POWER1
- R16 pad 1: LET_COLOR6 -> Net-(R16-Pad1)
- R16 pad 2: Net-(Q26-Pad1) -> RAP_POWER1
- R17 pad 1: RAP_COLOR1 -> Net-(R15-Pad1)
- R17 pad 2: Net-(Q27-Pad1) -> LET_POWER2
- R18 pad 1: RAP_COLOR2 -> Net-(R16-Pad1)
- R18 pad 2: Net-(Q28-Pad1) -> RAP_POWER2
- R19 pad 1: RAP_COLOR3 -> Net-(R15-Pad1)
- R19 pad 2: Net-(Q29-Pad1) -> LET_POWER3
- R2 pad 1: Net-(Q2-Pad1) -> Net-(R12-Pad1)
- R2 pad 2: BUCK_A -> RAP_COLOR1
- R20 pad 1: RAP_COLOR4 -> Net-(R16-Pad1)
- R20 pad 2: Net-(Q30-Pad1) -> RAP_POWER3
- R21 pad 1: Net-(R21-Pad1) -> Net-(R15-Pad1)
- R21 pad 2: LET_COLOR1 -> BATGND
- R22 pad 1: Net-(R21-Pad1) -> Net-(R16-Pad1)
- R22 pad 2: LET_COLOR2 -> BATGND
- R23 pad 1: Net-(R21-Pad1) -> Net-(R12-Pad1)
- R23 pad 2: LET_COLOR3 -> BATGND
- R24 pad 1: Net-(R21-Pad1) -> Net-(R1-Pad1)
- R24 pad 2: LET_COLOR4 -> BATGND
- R25 pad 1: Net-(R21-Pad1) -> Net-(R15-Pad1)
- R25 pad 2: LET_COLOR5 -> LET_POWER4
- R26 pad 1: Net-(R21-Pad1) -> Net-(R16-Pad1)
- R26 pad 2: LET_COLOR6 -> RAP_POWER4
- R27 pad 1: Net-(R21-Pad1) -> Net-(R15-Pad1)
- R27 pad 2: BATGND -> LET_POWER5
- R28 pad 1: Net-(R28-Pad1) -> Net-(R15-Pad1)
- R28 pad 2: LET_POWER1 -> LET_POWER6
- R29 pad 1: Net-(R28-Pad1) -> LGHT_P
- R29 pad 2: LET_POWER2 -> SDA
- R3 pad 1: Net-(Q3-Pad1) -> Net-(R1-Pad1)
- R3 pad 2: BUCK_B -> LET_COLOR2
- R30 pad 1: Net-(R28-Pad1) -> LGHT_P
- R30 pad 2: LET_POWER3 -> Net-(D6-A)
- R31 pad 1: Net-(R28-Pad1) -> LGHT_P
- R31 pad 2: LET_POWER4 -> Net-(D7-A)
- R32 pad 1: Net-(R28-Pad1) -> LGHT_P
- R32 pad 2: LET_POWER5 -> Net-(D8-A)
- R33 pad 1: Net-(R28-Pad1) -> FUS12V~
- R33 pad 2: LET_POWER6 -> Net-(D9-A)
- R34 pad 1: Net-(R28-Pad1) -> LGHT_P
- R34 pad 2: BATGND -> Net-(D10-A)
- R35 pad 1: Net-(R35-Pad1) -> LGHT_P
- R35 pad 2: RAP_COLOR1 -> Net-(D11-A)
- R36 pad 1: Net-(R35-Pad1) -> LGHT_P
- R36 pad 2: RAP_COLOR2 -> Net-(D12-A)
- R37 pad 1: Net-(R35-Pad1) -> BUCK~
- R37 pad 2: RAP_COLOR3 -> Net-(D13-A)
- R38 pad 1: Net-(R35-Pad1) -> LET_COLOR1
- R38 pad 2: RAP_COLOR4 -> Net-(Q10-B)
- R39 pad 1: Net-(R35-Pad1) -> LET_C1
- R39 pad 2: BATGND -> Net-(Q10-C)
- R4 pad 1: Net-(Q4-Pad1) -> Net-(R12-Pad1)
- R4 pad 2: BUCK_B -> RAP_COLOR2
- R40 pad 1: Net-(R40-Pad1) -> LET_COLOR2
- R40 pad 2: RAP_POWER1 -> Net-(Q12-B)
- R41 pad 1: Net-(R40-Pad1) -> LET_C1
- R41 pad 2: RAP_POWER2 -> Net-(Q12-C)
- R42 pad 1: Net-(R40-Pad1) -> LET_COLOR3
- R42 pad 2: RAP_POWER3 -> Net-(Q14-B)
- R43 pad 1: Net-(R40-Pad1) -> LET_C1
- R43 pad 2: RAP_POWER4 -> Net-(Q14-C)
- R44 pad 1: Net-(R40-Pad1) -> LET_COLOR4
- R44 pad 2: BATGND -> Net-(Q16-B)
- R45 pad 1: TURN_D_FIL -> LET_C1
- R45 pad 2: TURN_D -> Net-(Q16-C)
- R46 pad 1: TURN_P_FIL -> LET_COLOR5
- R46 pad 2: TURN_P -> Net-(Q22-B)
- R47 pad 1: MISC_1_FIL -> LET_C1
- R47 pad 2: MISC_1 -> Net-(Q18-G)
- R48 pad 1: BAT12V -> LET_COLOR6
- R48 pad 2: Net-(D11-Pad2) -> Net-(Q24-B)
- R49 pad 1: 12V -> LET_C1
- R49 pad 2: Net-(D12-Pad2) -> Net-(Q20-G)
- R5 pad 1: Net-(Q10-Pad3) -> Net-(R1-Pad1)
- R5 pad 2: BUCK_C -> LET_COLOR3
- R50 pad 1: MISC_2_FIL -> RAP_COLOR1
- R50 pad 2: MISC_2 -> Net-(Q34-B)
- R51 pad 1: Net-(D3-Pad1) -> LET_C1
- R51 pad 2: TX_1 -> Net-(Q26-G)
- R52 pad 1: Net-(D4-Pad1) -> RAP_COLOR2
- R52 pad 2: RX_1 -> Net-(Q36-B)
- R53 pad 1: Net-(D5-Pad1) -> LET_C1
- R53 pad 2: TX_2 -> Net-(Q28-G)
- R54 pad 1: Net-(D6-Pad1) -> RAP_COLOR3
- R54 pad 2: RX_2 -> Net-(Q38-B)
- R55 pad 1: Net-(D7-Pad1) -> LET_C1
- R55 pad 2: TX_3 -> Net-(Q30-G)
- R56 pad 1: Net-(D8-Pad1) -> Net-(Q40-B)
- R56 pad 2: RX_3 -> RAP_COLOR4
- R57 pad 1: GND~ -> LET_C1
- R57 pad 2: EN_A~ -> Net-(Q32-G)
- R58 pad 1: GND~ -> Net-(D14-K)
- R58 pad 2: EN_B~ -> Net-(D19-K)
- R59 pad 1: GND~ -> Net-(D14-K)
- R59 pad 2: EN_C~ -> Net-(D15-A)
- R6 pad 1: LET_COLOR1 -> Net-(R12-Pad1)
- R6 pad 2: Net-(Q6-Pad1) -> RAP_COLOR3
- R60 pad 1: GND~ -> Net-(D14-K)
- R60 pad 2: EN_D~ -> Net-(D16-A)
- R61 pad 1: GND~ -> Net-(D19-K)
- R61 pad 2: Net-(R61-Pad2) -> Net-(U2A-+)
- R62 pad 1: GND~ -> Net-(U2A-+)
- R62 pad 2: Net-(R62-Pad2) -> Net-(D15-K)
- R63 pad 1: GND~ -> Net-(D14-A)
- R63 pad 2: Net-(R63-Pad2) -> GND~
- R64 pad 1: GND~ -> Net-(R64-Pad1)
- R64 pad 2: Net-(R64-Pad2) -> Net-(U2B-+)
- R65 pad 1: Net-(D18-Pad2) -> Net-(D18-K)
- R66 pad 1: Net-(D19-Pad2) -> Net-(U2B-+)
- R66 pad 2: BUCK_A~ -> Net-(D16-K)
- R67 pad 1: Net-(D20-Pad2) -> /POWER/VDD
- R67 pad 2: BUCK_B~ -> PGOOD~
- R68 pad 1: Net-(D21-Pad2) -> Net-(C6-Pad2)
- R68 pad 2: BUCK_C~ -> Net-(U4-PH)
- R69 pad 1: Net-(D22-Pad2) -> /POWER/VDD
- R69 pad 2: BUCK_D~ -> Net-(JP1-B)
- R7 pad 1: LET_COLOR2 -> TURN_D
- R7 pad 2: Net-(Q7-Pad1) -> TURN_D_FIL
- R70 pad 1: Net-(C17-Pad1) -> Net-(U4-ADDR)
- R70 pad 2: Net-(D23-Pad1) -> GND~
- R71 pad 1: Net-(Q42-Pad2) -> Net-(U4-RT/SYNC)
- R71 pad 2: Net-(D23-Pad1) -> GND~
- R72 pad 1: Net-(C17-Pad1) -> GND~
- R72 pad 2: Net-(D24-Pad1) -> Net-(R72-Pad2)
- R73 pad 1: Net-(Q43-Pad2) -> LGHT_P
- R73 pad 2: Net-(D24-Pad1) -> SCL
- R8 pad 1: LET_COLOR3 -> TURN_P
- R8 pad 2: Net-(Q8-Pad1) -> TURN_P_FIL
- R9 pad 1: LET_COLOR4 -> MISC_1
- R9 pad 2: Net-(Q9-Pad1) -> MISC_1_FIL
- RV1 pad 1: Net-(R61-Pad2) -> Net-(D14-K)
- RV1 pad 2: BUCK_A~ -> Net-(U2A--)
- RV1 pad 3: BUCK_A~ -> GND~
- RV2 pad 1: Net-(R62-Pad2) -> Net-(D14-K)
- RV2 pad 2: BUCK_B~ -> Net-(R64-Pad1)
- RV2 pad 3: BUCK_B~ -> GND~
- RV3 pad 1: Net-(R63-Pad2) -> Net-(R72-Pad2)
- RV3 pad 2: BUCK_C~ -> Net-(U4-VSET)
- RV3 pad 3: BUCK_C~ -> unconnected-(RV3-Pad3)
- SW1 pad 1: +5V -> LGHT_P
- SW1 pad 2: +5V -> LGHT_P
- SW1 pad 3: +5V -> LGHT_P
- SW1 pad 4: +5V -> LGHT_P
- SW1 pad 5: Net-(R40-Pad1) -> Net-(R15-Pad1)
- SW1 pad 6: Net-(R35-Pad1) -> Net-(R16-Pad1)
- SW1 pad 7: Net-(R28-Pad1) -> Net-(R12-Pad1)
- SW1 pad 8: Net-(R21-Pad1) -> Net-(R1-Pad1)
- U1 pad 3V3_1: Net-(U1-Pad3V3_1) -> unconnected-(U1-3V3-Pad3V3_1)
- U1 pad 3V3_2: Net-(U1-Pad3V3_1) -> unconnected-(U1-3V3-Pad3V3_1)
- U1 pad 5V_1: +5V -> LGHT_P
- U1 pad 5V_2: +5V -> LGHT_P
- U1 pad A4: unconnected-(U1-PadA4) -> LGHT_S
- U1 pad D20: unconnected-(U1-PadD20) -> SDA
- U1 pad D21: unconnected-(U1-PadD21) -> SCL
- U1 pad D32: unconnected-(U1-PadD32) -> PGOOD
- U1 pad D33: unconnected-(U1-PadD33) -> SALRT
- U1 pad VIN_1: Net-(U1-PadVIN_1) -> unconnected-(U1-VIN-PadVIN_1)
- U1 pad VIN_2: Net-(U1-PadVIN_1) -> unconnected-(U1-VIN-PadVIN_1)
- U2 pad 1: 12V~ -> Net-(D15-K)
- U2 pad 2: Net-(D13-Pad1) -> Net-(U2A--)
- U2 pad 3: GND~ -> Net-(U2A-+)
- U2 pad 4: Net-(R61-Pad2) -> GND~
- U2 pad 5: EN_A~ -> Net-(U2B-+)
- U3 pad 1: 12V~ -> LET_C1
- U3 pad 2: Net-(D14-Pad1) -> BATGND
- U3 pad 3: GND~ -> LGHT_P
- U4 pad 1: 12V~ -> /POWER/VIN
- U4 pad 2: Net-(D15-Pad1) -> /POWER/VIN
- U4 pad 3: GND~ -> /POWER/VIN
- U4 pad 4: Net-(R63-Pad2) -> Net-(U4-PH)
- U4 pad 5: EN_C~ -> Net-(U4-GH)
Routing:
- net BATGND: track 0.00 -> 406.6 mm, vias 0 -> 26
- net SCL: track 0.00 -> 242.9 mm, vias 0 -> 1
- net LET_C1: track 0.00 -> 239.5 mm, vias 0 -> 10
- net SDA: track 0.00 -> 231.5 mm, vias 0 -> 1
- net LGHT_P: track 0.00 -> 196.0 mm, vias 0 -> 5
- net LET_COLOR3: track 0.00 -> 176.4 mm, vias 0 -> 1
- net LGHT_S: track 0.00 -> 152.3 mm, vias 0 -> 1
- net RAP_POWER3: track 0.00 -> 149.0 mm, vias 0 -> 4
- net RAP_POWER4: track 0.00 -> 146.2 mm, vias 0 -> 4
- net RX_3: track 0.00 -> 146.1 mm, vias 0 -> 2
- net LET_POWER3: track 0.00 -> 144.8 mm, vias 0 -> 3
- net TX_3: track 0.00 -> 143.7 mm, vias 0 -> 2
- net RX_2: track 0.00 -> 137.2 mm, vias 0 -> 1
- net TX_2: track 0.00 -> 134.7 mm, vias 0 -> 1
- net RAP_POWER2: track 0.00 -> 134.6 mm, vias 0 -> 2
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- added copper zone on F.Cu, net /POWER/SW
- added copper zone on F.Cu, net /POWER/VIN
- added copper zone on B.Cu, net BUCK~
- added copper zone on F.Cu, net BUCK~
- added copper zone on B.Cu, net FIL12V~
- added copper zone on F.Cu, net FIL12V~
- added copper zone on B.Cu, net FUS12V
- added copper zone on F.Cu, net FUS12V
- added copper zone on B.Cu, net FUS12V~
- added copper zone on F.Cu, net FUS12V~
- added copper zone on B.Cu, net GND~
- added copper zone on F.Cu, net GND~
- added copper zone on B.Cu, net LET_C1
- added copper zone on F.Cu, net Net-(C20-Pad1)
- added copper zone on B.Cu, net Net-(D14-K)
- added copper zone on F.Cu, net Net-(D14-K)
Other:
- outline, holes or cut-outs redrawn
- board text added: "BUCK"
- board text added: "BUCK VOLTAGE"
- board text added: "Brethren, I count not myself to have apprehended: but this one thing I do, forgetting those things which are behind, and reaching forth unto those things which are before, I press toward the mark for the prize of the high calling of God in Christ Jesus."
- board text added: "Daniel Hoefer 2023"
- board text added: "ENABLE"
- board text added: "FILTERED 12V"
- board text added: "FUSE"
- board text added: "FUSE 12V"
- board text added: "GND"
- board text added: "OVER"
- board text added: "PWA, DEV-T4R1002"
- board text added: "PWA, DEV-T4R1005"
- board text added: "PWB, DEV-T4R1003"
- board text added: "PWB, DEV-T4R1006"
- board text added: "Philippians 3:13-14"
- board text added: "REV"
- board text added: "RX_1"
- board text added: "RX_3"
- board text added: "SDA SCL PGOOD SLART"
- board text added: "TX_1"
- board text added: "TX_2"
- board text added: "TX_3"
- board text added: "UNDER"
